File: tracker/low_voltage_psu.kicad_sch (KiCad schematic)
At the start: 6 parts, among them U7 AP61100Z6

Commit message: save
Parts:
- added R14: 200K, Resistor_SMD:R_0402_1005Metric, symbol Device:R_Small
Connections:
- net +VSYS: now also R14.2; no longer U7.5 (EN)
- new net LV_PSU_EN: R14.1, U7.5 (EN)
Other:
- moved on the sheet: C29
Changed lines of the file:
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@@
-	)
-	(junction
-		(at 116.84 63.5)
-		(diameter 0)
-		(color 0 0 0 0)
 	)
 	(junction
@@
 	)
 	(junction
+		(at 114.3 63.5)
+		(diameter 0)
+		(color 0 0 0 0)
+	)
+	(junction
+		(at 124.46 68.58)
+		(diameter 0)
+		(color 0 0 0 0)
+	)
+	(junction
 		(at 157.48 73.66)
 		(diameter 0)
@@
 	(wire
 		(pts
-			(xy 128.27 63.5) (xy 124.46 63.5)
-		)
-		(stroke
-			(width 0)
-			(type default)
-		)
-	)
-	(wire
-		(pts
-			(xy 124.46 68.58) (xy 124.46 63.5)
+			(xy 114.3 63.5) (xy 124.46 63.5)
 		)
 		(stroke
@@
 	(wire
 		(pts
-			(xy 116.84 63.5) (xy 116.84 64.77)
+			(xy 114.3 63.5) (xy 114.3 64.77)
+		)
+		(stroke
+			(width 0)
+			(type default)
+		)
+	)
+	(wire
+		(pts
+			(xy 104.14 81.28) (xy 124.46 81.28)
 		)
 		(stroke
@@
 	(wire
 		(pts
-			(xy 106.68 63.5) (xy 116.84 63.5)
-		)
-		(stroke
-			(width 0)
-			(type default)
-		)
-	)
-	(wire
-		(pts
-			(xy 124.46 63.5) (xy 116.84 63.5)
+			(xy 104.14 63.5) (xy 114.3 63.5)
+		)
+		(stroke
+			(width 0)
+			(type default)
+		)
+	)
+	(wire
+		(pts
+			(xy 124.46 63.5) (xy 128.27 63.5)
+		)
+		(stroke
+			(width 0)
+			(type default)
+		)
+	)
+	(wire
+		(pts
+			(xy 124.46 68.58) (xy 124.46 81.28)
 		)
 		(stroke
@@
 	(hierarchical_label "+VSYS"
 		(shape input)
-		(at 106.68 63.5 180)
+		(at 104.14 63.5 180)
+		(effects
+			(font
+				(size 1.27 1.27)
+			)
+			(justify right)
+		)
+	)
+	(hierarchical_label "LV_PSU_EN"
+		(shape input)
+		(at 104.14 81.28 180)
 		(effects
 			(font
@@
 	(symbol
 		(lib_id "Device:C_Small")
-		(at 116.84 67.31 0)
+		(at 114.3 67.31 0)
 		(mirror y)
 		(unit 1)
@@
 		(dnp no)
 		(property "Reference" "C29"
-			(at 114.3 66.0462 0)
+			(at 111.76 66.0462 0)
 			(effects
 				(font
@@
 		)
 		(property "Value" "10u"
-			(at 114.3 68.5862 0)
+			(at 111.76 68.5862 0)
 			(effects
 				(font
@@
 		)
 		(property "Footprint" "Capacitor_SMD:C_0805_2012Metric"
-			(at 116.84 67.31 0)
+			(at 114.3 67.31 0)
 			(effects
 				(font
@@
 		)
 		(property "Datasheet" "~"
-			(at 116.84 67.31 0)
+			(at 114.3 67.31 0)
 			(effects
 				(font
@@
 		)
 		(property "Description" "Unpolarized capacitor, small symbol"
-			(at 116.84 67.31 0)
+			(at 114.3 67.31 0)
 			(effects
 				(font
@@
 	(symbol
 		(lib_id "Device:R_Small")
+		(at 124.46 66.04 180)
+		(unit 1)
+		(exclude_from_sim no)
+		(in_bom yes)
+		(on_board yes)
+		(dnp no)
+		(property "Reference" "R14"
+			(at 121.158 65.024 0)
+			(effects
+				(font
+					(size 1.27 1.27)
+				)
+			)
+		)
+		(property "Value" "200K"
+			(at 120.65 67.31 0)
+			(effects
+				(font
+					(size 1.27 1.27)
+				)
+			)
+		)
+		(property "Footprint" "Resistor_SMD:R_0402_1005Metric"
+			(at 124.46 66.04 0)
+			(effects
+				(font
+					(size 1.27 1.27)
+				)
+				(hide yes)
+			)
+		)
+		(property "Datasheet" "~"
+			(at 124.46 66.04 0)
+			(effects
+				(font
+					(size 1.27 1.27)
+				)
+				(hide yes)
+			)
+		)
+		(property "Description" "Resistor, small symbol"
+			(at 124.46 66.04 0)
+			(effects
+				(font
+					(size 1.27 1.27)
+				)
+				(hide yes)
+			)
+		)
+		(pin "1"
+		)
+		(pin "2"
+		)
+		(instances
+			(project "tracker"
+				(path "/4f1d18f5-7d2b-4d0b-8633-b1619d53124c/1b416177-91af-4d12-8e72-813a2e7f8715"
+					(reference "R14")
+					(unit 1)
+				)
+			)
+		)
+	)
+	(symbol
+		(lib_id "Device:R_Small")
 		(at 157.48 71.12 0)
 		(mirror x)
@@
 	(symbol
 		(lib_id "power:GND")
-		(at 116.84 69.85 0)
+		(at 114.3 69.85 0)
 		(unit 1)
 		(exclude_from_sim no)
@@
 		(dnp no)
 		(property "Reference" "#PWR048"
-			(at 116.84 76.2 0)
+			(at 114.3 76.2 0)
 			(effects
 				(font
@@
 		)
 		(property "Value" "GND"
-			(at 116.84 73.914 0)
+			(at 114.3 73.914 0)
 			(effects
 				(font
@@
 		)
 		(property "Footprint" ""
-			(at 116.84 69.85 0)
+			(at 114.3 69.85 0)
 			(effects
 				(font
@@
 		)
 		(property "Datasheet" ""
-			(at 116.84 69.85 0)
+			(at 114.3 69.85 0)
 			(effects
 				(font
@@
 		)
 		(property "Description" "Power symbol creates a global label with name \"GND\" , ground"
-			(at 116.84 69.85 0)
-			(effects
-				(font
+			(at 114.3 69.85 0)
+			(effects
+				(font

Commit message: save
Parts:
- renumbered C29 to C30, C30 to C31, R14 to R12, R9 to R13, R10 to R14, U7 to U9
Changed lines of the file:
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@@
 		(on_board yes)
 		(dnp no)
-		(property "Reference" "C29"
+		(property "Reference" "C30"
 			(at 111.76 66.0462 0)
 			(effects
@@
 			(project "BK4000TG_V3"
 				(path "/4f1d18f5-7d2b-4d0b-8633-b1619d53124c/1b416177-91af-4d12-8e72-813a2e7f8715"
-					(reference "C29")
+					(reference "C30")
 					(unit 1)
 				)
@@
 		(on_board yes)
 		(dnp no)
-		(property "Reference" "#PWR050"
+		(property "Reference" "#PWR066"
 			(at 157.48 87.63 0)
 			(effects
@@
 			(project "BK4000TG_V3"
 				(path "/4f1d18f5-7d2b-4d0b-8633-b1619d53124c/1b416177-91af-4d12-8e72-813a2e7f8715"
-					(reference "#PWR050")
+					(reference "#PWR066")
 					(unit 1)
 				)
@@
 		(dnp no)
 		(fields_autoplaced yes)
-		(property "Reference" "U7"
+		(property "Reference" "U9"
 			(at 135.89 55.88 0)
 			(effects
@@
 			(project ""
 				(path "/4f1d18f5-7d2b-4d0b-8633-b1619d53124c/1b416177-91af-4d12-8e72-813a2e7f8715"
-					(reference "U7")
+					(reference "U9")
 					(unit 1)
 				)
@@
 		(on_board yes)
 		(dnp no)
-		(property "Reference" "R10"
+		(property "Reference" "R14"
 			(at 160.782 75.438 0)
 			(effects
@@
 			(project "BK4000TG_V3"
 				(path "/4f1d18f5-7d2b-4d0b-8633-b1619d53124c/1b416177-91af-4d12-8e72-813a2e7f8715"
-					(reference "R10")
+					(reference "R14")
 					(unit 1)
 				)
@@
 		(on_board yes)
 		(dnp no)
-		(property "Reference" "C30"
+		(property "Reference" "C31"
 			(at 171.45 69.8562 0)
 			(effects
@@
 			(project "BK4000TG_V3"
 				(path "/4f1d18f5-7d2b-4d0b-8633-b1619d53124c/1b416177-91af-4d12-8e72-813a2e7f8715"
-					(reference "C30")
+					(reference "C31")
 					(unit 1)
 				)
@@
 		(on_board yes)
 		(dnp no)
-		(property "Reference" "#PWR049"
+		(property "Reference" "#PWR065"
 			(at 135.89 87.63 0)
 			(effects
@@
 			(project ""
 				(path "/4f1d18f5-7d2b-4d0b-8633-b1619d53124c/1b416177-91af-4d12-8e72-813a2e7f8715"
-					(reference "#PWR049")
+					(reference "#PWR065")
 					(unit 1)
 				)
@@
 		(on_board yes)
 		(dnp no)
-		(property "Reference" "R14"
+		(property "Reference" "R12"
 			(at 121.158 65.024 0)
 			(effects
@@
 			(project "tracker"
 				(path "/4f1d18f5-7d2b-4d0b-8633-b1619d53124c/1b416177-91af-4d12-8e72-813a2e7f8715"
-					(reference "R14")
+					(reference "R12")
 					(unit 1)
 				)
@@
 		(on_board yes)
 		(dnp no)
-		(property "Reference" "R9"
+		(property "Reference" "R13"
 			(at 160.782 70.104 0)
 			(effects
@@
 			(project "BK4000TG_V3"
 				(path "/4f1d18f5-7d2b-4d0b-8633-b1619d53124c/1b416177-91af-4d12-8e72-813a2e7f8715"
-					(reference "R9")
+					(reference "R13")
 					(unit 1)
 				)
@@
 		(on_board yes)
 		(dnp no)
-		(property "Reference" "#PWR051"
+		(property "Reference" "#PWR067"
 			(at 168.91 87.63 0)
 			(effects
@@
 			(project "BK4000TG_V3"
 				(path "/4f1d18f5-7d2b-4d0b-8633-b1619d53124c/1b416177-91af-4d12-8e72-813a2e7f8715"
-					(reference "#PWR051")
+					(reference "#PWR067")
 					(unit 1)
 				)
@@
 		(on_board yes)
 		(dnp no)
-		(property "Reference" "#PWR048"
+		(property "Reference" "#PWR064"
 			(at 114.3 76.2 0)
 			(effects
@@
 			(project "BK4000TG_V3"
 				(path "/4f1d18f5-7d2b-4d0b-8633-b1619d53124c/1b416177-91af-4d12-8e72-813a2e7f8715"
-					(reference "#PWR048")
-					(unit 1)
-				)
+					(reference "#PWR064")
+					(unit 1)
+				)
