File: tracker/tracker.kicad_pcb (KiCad board)
At the start: 2 copper layers, 50.5 x 56.9 mm, 76 parts, among them J1 Conn_01x10, J2 SIM_Card, M1 BG96, Q1 SSM6N7002KFU, Q2 SSM6N7002KFU, Q3 SSM6N7002KFU, U1 STM32U545CEUx, U2 GD25QxxxEY, U3 74LVC244APW,118, U4 AP22800HB-7, U5 DF5A6.8JE,LM, U6 LMR51430, U7 AP61100Z6, U8 BQ25601, Y1 32.768KHz, Y2 8MHz

Commit message: save
Parts:
- removed C34: 10u, Capacitor_SMD:C_0805_2012Metric
- removed Q3: SSM6N7002KFU, Package_TO_SOT_SMD:SOT-363_SC-70-6
- removed Y1: 32.768KHz, Crystal:Crystal_SMD_SeikoEpson_MC146-4Pin_6.7x1.5mm
- added C41: 10u, Capacitor_SMD:C_0805_2012Metric, B.Cu at (152.9, 87.2)
- added C42: 0.1u, Capacitor_SMD:C_0603_1608Metric, B.Cu at (152.7, 89.1)
- added D1: 12V, Diode_SMD:D_SOD-323, F.Cu at (165.2, 95.3)
- added J3: Conn_01x01, My Footprints:pad_smd_1.5x3, F.Cu at (168.4, 93.3)
- added J4: Conn_01x01, My Footprints:pad_smd_1.5x3, F.Cu at (171.1, 93.3)
- added J5: Conn_Coaxial, Connector_Coaxial:U.FL_Molex_MCRF_73412-0110_Vertical, B.Cu at (164.0, 46.4)
- added J6: Conn_01x02, Connector_JST:JST_XH_B2B-XH-A_1x02_P2.50mm_Vertical, B.Cu at (129.0, 92.6)
- added R15: TBD, Resistor_SMD:R_0402_1005Metric, B.Cu at (147.2, 94.0)
- added U10: PUMH10,115, Package_TO_SOT_SMD:SOT-363_SC-70-6, F.Cu at (162.7, 80.6)
- added U9: ~, My Footprints:BQ25622E, B.Cu at (148.1, 89.8)
- added Y3: 32.768KHz, Crystal:Crystal_SMD_SeikoEpson_MC146-4Pin_6.7x1.5mm, F.Cu at (148.6, 83.3)
- C29, C30, C31, C32, C36, C37, C38, C39, C40, L3, L4, R10, R11, R12, R9, U7: moved to B.Cu
- J1: value Conn_01x10 -> Conn_01x05; footprint Connector:Tag-Connect_TC2050-IDC-NL_2x05_P1.27mm_Vertical -> Connector_JST:JST_PH_B5B-PH-SM4-TB_1x05-1MP_P2.00mm_Vertical
- Q2: value SSM6N7002KFU -> DMP2008UFG; footprint Package_TO_SOT_SMD:SOT-363_SC-70-6 -> Package_SON:Diodes_PowerDI3333-8
- R13: value 37K -> 10K; footprint Resistor_SMD:R_0402_1005Metric -> Resistor_SMD:R_0603_1608Metric
- R14: value 100K -> 200K; moved to B.Cu
- R4: value 200K -> 220K; footprint Resistor_SMD:R_0402_1005Metric -> Resistor_SMD:R_0603_1608Metric
- U2: moved to F.Cu
- U8: value BQ25601 -> PUMH10,115; footprint Package_DFN_QFN:Texas_RTW_WQFN-24-1EP_4x4mm_P0.5mm_EP2.7x2.7mm_ThermalVias -> Package_TO_SOT_SMD:SOT-363_SC-70-6; moved to F.Cu
- moved C28 69.5 mm to (157.0, 89.5)
- moved C12 66.8 mm to (163.1, 77.8)
- moved C22 55.1 mm to (151.2, 61.8), turned to 180 degrees
- moved C4 54.0 mm to (144.4, 74.4), turned to -90 degrees
- moved R14 52.0 mm to (138.4, 90.2), turned to 90 degrees
- moved C2 51.8 mm to (145.9, 81.4)
- moved C3 51.4 mm to (144.4, 79.6), turned to 90 degrees
- moved C1 50.7 mm to (145.9, 85.1), turned to 180 degrees
- moved C40 49.4 mm to (140.1, 87.2), turned to 90 degrees
- moved L4 49.0 mm to (149.7, 85.7), turned to 90 degrees
- moved C39 46.5 mm to (142.2, 87.2), turned to 90 degrees
- moved C36 45.1 mm to (148.6, 93.9), turned to -90 degrees
- moved R12 44.4 mm to (145.9, 94.0), turned to -90 degrees
- moved R11 44.0 mm to (146.4, 92.4), turned to 180 degrees
- moved C38 43.6 mm to (144.3, 87.2), turned to 90 degrees
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Connections:
- net Net-(AE1-A) renamed /gsm/ANT_GNSS
- C10 pad 1: Net-(U2-VCC) -> +3V3
- C23 pad 1: /psu/+VIN -> /psu/+VIN_PROTECTED
- C24 pad 1: /psu/+VIN -> /psu/+VIN_PROTECTED
- C29 pad 1: /low_voltage_psu/+VSYS -> +VSYS
- C30 pad 1: /low_voltage_psu/+3V3 -> +3V3
- C35 pad 2: Net-(U8-BTST) -> Net-(U9-BTST)
- C36 pad 1: Net-(U8-REGN) -> Net-(U9-REGN)
- C37 pad 1: Net-(C37-Pad1) -> /battery charger/+BAT
- C38 pad 1: /battery charger/+VSYS -> +VSYS
- C39 pad 1: /battery charger/+VSYS -> +VSYS
- C40 pad 1: /battery charger/+VSYS -> +VSYS
- J1 pad 5: unconnected-(J1-Pin_5-Pad5) -> GND
- L3 pad 2: /low_voltage_psu/+3V3 -> +3V3
- L4 pad 2: /battery charger/+VSYS -> +VSYS
- M1 pad 60: unconnected-(M1-ANT_MAIN-Pad60) -> /gsm/ANT_MAIN
- Q2 pad 1: /mcu/PSU_CTRL -> /psu/+VIN_PROTECTED
- Q2 pad 2: +3V3 -> /psu/+VIN_PROTECTED
- Q2 pad 3: unconnected-(Q2B-D-Pad3) -> /psu/+VIN_PROTECTED
- Q2 pad 4: unconnected-(Q2B-S-Pad4) -> Net-(D1-A)
- Q2 pad 5: unconnected-(Q2B-G-Pad5) -> /+VIN
- R11 pad 1: Net-(U8-REGN) -> Net-(U9-TS_BIAS)
- R11 pad 2: Net-(U8-TS) -> Net-(U9-TS)
- R12 pad 1: Net-(U8-TS) -> Net-(U9-TS)
- R13 pad 1: Net-(C37-Pad1) -> Net-(D1-A)
- R13 pad 2: /battery charger/BAT_LEVEL -> GND
- R14 pad 1: /battery charger/BAT_LEVEL -> /battery charger/CHARGER_PG
- R14 pad 2: GND -> +VSYS
- R4 pad 1: +3V3 -> /psu/+VIN_PROTECTED
- R4 pad 2: /mcu/PSU_CTRL -> Net-(D1-A)
- R5 pad 1: /psu/+VIN -> /psu/+VIN_PROTECTED
- R5 pad 2: Net-(Q2A-D) -> Net-(U6-EN)
- R6 pad 2: Net-(Q2A-D) -> Net-(U6-EN)
- R9 pad 2: /low_voltage_psu/+3V3 -> +3V3
- RN1 pad 1: /gsm/SIM_CLK -> /gsm/SIM_RST
- RN1 pad 3: /gsm/SIM_RST -> /gsm/SIM_CLK
- RN1 pad 6: Net-(J2-RST) -> Net-(J2-CLK)
- RN1 pad 8: Net-(J2-CLK) -> Net-(J2-RST)
- U1 pad 14: /mcu/OCTOSPI1_NCS -> unconnected-(U1-PA4-Pad14)
- U1 pad 20: unconnected-(U1-PB2-Pad20) -> /gsm/GSM_RESET
- U1 pad 21: unconnected-(U1-PB10-Pad21) -> /gsm/GSM_PWRKEY
- U1 pad 29: /gsm/GSM_STATUS -> unconnected-(U1-PA8-Pad29)
- U1 pad 33: unconnected-(U1-PA12-Pad33) -> /mcu/OCTOSPI1_NCS
- U1 pad 34: unconnected-(U1-PA13-Pad34) -> /mcu/SWDIO
- U1 pad 37: unconnected-(U1-PA14-Pad37) -> /mcu/SWCLK
- U1 pad 42: unconnected-(U1-PB6-Pad42) -> /mcu/I2C_SCL
- U1 pad 43: unconnected-(U1-PB7-Pad43) -> /mcu/I2C_SDA
- U1 pad 44: unconnected-(U1-PH3-Pad44) -> /gsm/GSM_LINE_BUF_EN
- U1 pad 45: unconnected-(U1-PB8-Pad45) -> /gsm/GSM_AP_READY
- U1 pad 46: unconnected-(U1-PB9-Pad46) -> /gsm/GSM_STATUS
- U2 pad 8: Net-(U2-VCC) -> +3V3
- U3 pad 1: (no net) -> /gsm/GSM_LINE_BUF_EN
- U6 pad 3: /psu/+VIN -> /psu/+VIN_PROTECTED
- U6 pad 5: Net-(Q2A-D) -> Net-(U6-EN)
- U7 pad 3: /low_voltage_psu/+VSYS -> +VSYS
- U7 pad 5: /low_voltage_psu/+VSYS -> /battery charger/CHARGER_PG
- U7 pad 6: /low_voltage_psu/+3V3 -> +3V3
- U8 pad 1: +5V -> /mcu/PSU_CTRL
- U8 pad 2: GND -> +3V3
- U8 pad 3: /battery charger/CHARGER_PG -> unconnected-(U8-Pad3)
- U8 pad 4: /battery charger/CHARGER_STAT -> unconnected-(U8-Pad4)
- U8 pad 5: /battery charger/CHARGER_SCL -> unconnected-(U8-Pad5)
- U8 pad 6: /battery charger/CHARGER_SDA -> Net-(U6-EN)
Routing:
- net /gsm/GSM_LINE_BUF_EN: track 0.00 -> 33.5 mm, vias 0 -> 2
- net /gsm/GPS_TX: track 0.00 -> 28.6 mm, vias 0 -> 2
- net /gsm/GPS_RX: track 0.00 -> 27.8 mm, vias 0 -> 2
- net /gsm/GSM_AP_READY: track 0.00 -> 26.6 mm, vias 0 -> 2
- net /gsm/PWRKEY: track 0.00 -> 25.4 mm, vias 0 -> 1
- net /gsm/RESET: track 0.00 -> 25.0 mm, vias 0 -> 1
- net /mcu/OCTOSPI1_IO0: track 0.00 -> 24.3 mm
- net /mcu/OCTOSPI1_IO2: track 0.00 -> 24.1 mm
- net /mcu/OCTOSPI1_IO1: track 0.00 -> 24.1 mm
- net /mcu/OCTOSPI1_IO3: track 0.00 -> 24.1 mm
- net /gsm/GSM_STATUS: track 0.00 -> 23.6 mm, vias 0 -> 2
- net /mcu/OCTOSPI1_CLK: track 0.00 -> 23.4 mm
- net /gsm/GSM_PWRKEY: track 0.00 -> 23.2 mm, vias 0 -> 2
- net /mcu/I2C_SCL: track 0.00 -> 19.1 mm, vias 0 -> 1
- net /gsm/GSM_RESET: track 0.00 -> 18.0 mm, vias 0 -> 2
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- added copper zone on B.Cu, net +3V3
- added copper zone on In1.Cu, net +3V3
- added copper zone on B.Cu, net +5V
- added copper zone on In1.Cu, net +5V
- added copper zone on B.Cu, net +VSYS
- added copper zone on F.Cu, net +VSYS
- added copper zone on In1.Cu, net +VSYS
- added copper zone on B.Cu, net /battery charger/+BAT
- added copper zone on In1.Cu, net /battery charger/+BAT
- added copper zone on B.Cu, net /battery charger/BQ_SW
- added copper zone on B.Cu, net /gsm/+VBAT_GSM
- added copper zone on F.Cu, net /gsm/+VBAT_GSM
- added copper zone on B.Cu, net Net-(U6-SW)
- added copper zone on B.Cu, net Net-(U7-SW)
Other:
- board size 50.5 x 56.9 mm -> 49.9 x 54.9 mm
- copper layers 2 -> 4

Commit message: save project
Parts:
- removed C19: 1u, Capacitor_SMD:C_0402_1005Metric
- added R16: 10K, Resistor_SMD:R_0603_1608Metric, F.Cu at (169.0, 88.5)
- added R17: 150K, Resistor_SMD:R_0603_1608Metric, F.Cu at (169.1, 90.1)
- C10, C12, C5, C6, C7, C8, C9: footprint Capacitor_SMD:C_0402_1005Metric -> Capacitor_SMD:C_0603_1608Metric
- C15, C16: moved to B.Cu
- C17: value 1u -> 4.7u; footprint Capacitor_SMD:C_0402_1005Metric -> Capacitor_SMD:C_0603_1608Metric
- C20, C21: footprint Capacitor_SMD:C_0402_1005Metric -> Capacitor_SMD:C_0603_1608Metric; moved to B.Cu
- moved U10 27.6 mm to (135.9, 87.3), turned to 90 degrees
- moved U8 24.5 mm to (132.9, 87.3)
- moved C17 14.3 mm to (134.8, 72.9), turned to 180 degrees
- moved L1 8.30 mm to (145.4, 61.0), turned to 0 degrees
- moved C16 8.01 mm to (156.8, 45.6)
- moved C14 6.30 mm to (144.6, 62.5), turned to 180 degrees
- moved AE1 4.39 mm to (134.5, 54.0)
- moved C20 3.84 mm to (146.4, 70.7), turned to 90 degrees
- moved C11 3.06 mm to (142.2, 64.2), turned to -90 degrees
- moved C15 2.91 mm to (143.6, 69.6)
- moved U4 2.69 mm to (144.2, 64.3)
- moved R3 2.30 mm to (144.7, 66.1), turned to 180 degrees
- moved C22 2.18 mm to (152.6, 60.1), turned to 90 degrees
- moved R2 1.75 mm to (137.2, 85.0), turned to 180 degrees
- moved C13 1.74 mm to (142.7, 66.1), turned to 180 degrees
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Connections:
- C17 pad 1: /gsm/+VBAT_GSM -> /mcu/VCAP
- U1 pad 20: /gsm/GSM_RESET -> /mcu/VIN_MEAS
- U1 pad 21: /gsm/GSM_PWRKEY -> unconnected-(U1-PB10-Pad21)
- U1 pad 22: unconnected-(U1-VCAP-Pad22) -> /mcu/VCAP
- U1 pad 26: unconnected-(U1-PB13-Pad26) -> /gsm/GSM_RESET
- U1 pad 28: unconnected-(U1-PB15-Pad28) -> /gsm/GSM_PWRKEY
- U1 pad 38: unconnected-(U1-PA15-Pad38) -> /battery charger/CHARGER_INT
Routing:
- net /mcu/VIN_MEAS: track 0.00 -> 45.3 mm, vias 0 -> 2
- net +3V3: track 2.10 -> 36.3 mm, vias 6 -> 8
- net Net-(U6-EN): track 4.91 -> 29.8 mm
- net Net-(U9-~{CE}): track 0.00 -> 16.5 mm, vias 0 -> 1
- net Net-(U9-~{QON}): track 0.00 -> 13.2 mm, vias 0 -> 1
- net /gsm/GSM_RESET: track 18.0 -> 22.4 mm
- net /mcu/VCAP: track 0.00 -> 2.86 mm
- net /gsm/ANT_GNSS: track 18.0 -> 15.3 mm
- net /battery charger/CHARGER_PG: track 0.00 -> 2.18 mm
- net Net-(U7-FB): track 0.00 -> 2.17 mm
- net /gsm/SIM_VCC: track 7.39 -> 9.32 mm
- net Net-(J2-CLK): track 9.52 -> 7.66 mm
- net /gsm/SIM_RST: track 2.41 -> 4.02 mm
- net Net-(J2-RST): track 7.51 -> 5.90 mm
- net /battery charger/CHARGER_INT: track 0.00 -> 1.53 mm, vias 0 -> 1
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- added copper zone on F.Cu, net /gsm/+GSM_SWITCHED

Commit message: save project
Parts:
- removed C38: 10u, Capacitor_SMD:C_0805_2012Metric
- moved U8 29.0 mm to (161.9, 85.4), turned to 0 degrees
- moved R9 5.49 mm to (141.2, 89.2), turned to 90 degrees
- moved C30 4.77 mm to (137.7, 87.9), turned to 0 degrees
- moved C40 4.63 mm to (143.9, 89.1), turned to 180 degrees
- moved U10 3.53 mm to (133.5, 84.7), turned to 180 degrees
- moved L3 3.52 mm to (135.6, 90.3), turned to 90 degrees
- moved R10 3.29 mm to (140.1, 89.2), turned to -90 degrees
- moved R2 2.58 mm to (139.5, 86.2)
- moved R1 2.58 mm to (139.0, 85.2)
- moved R14 2.57 mm to (137.6, 92.6), turned to -90 degrees
- moved J6 2.24 mm to (131.2, 92.0)
- moved C39 2.20 mm to (143.9, 86.7), turned to 180 degrees
- moved R15 1.70 mm to (148.8, 94.5)
- moved U7 1.60 mm to (138.3, 90.2), turned to 180 degrees
- moved C36 1.55 mm to (150.1, 94.2)
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Connections:
- U1 pad 38: /battery charger/CHARGER_INT -> /battery charger/POWER_CYCLE
- U1 pad 39: unconnected-(U1-PB3-Pad39) -> /battery charger/CHARGE_ENABLE
- U1 pad 40: unconnected-(U1-PB4-Pad40) -> /battery charger/CHARGER_INT
Routing:
- net Net-(U6-EN): track 29.8 -> 2.58 mm, vias 1 -> 0
- net /battery charger/CHARGER_INT: track 1.53 -> 17.6 mm, vias 1 -> 3
- net +3V3: track 36.3 -> 48.5 mm, vias 8 -> 12
- net Net-(U9-~{QON}): track 13.2 -> 21.7 mm
- net Net-(U9-~{CE}): track 16.5 -> 23.8 mm
- net /battery charger/CHARGE_ENABLE: track 0.00 -> 5.22 mm
- net /battery charger/POWER_CYCLE: track 0.00 -> 5.17 mm
- net /mcu/I2C_SCL: track 19.2 -> 21.5 mm
- net /mcu/I2C_SDA: track 16.8 -> 18.7 mm
- net /battery charger/CHARGER_PG: track 2.18 -> 3.78 mm, vias 0 -> 1
- net GND: track 0.00 -> 0.91 mm, vias 0 -> 10
- net +VSYS: vias 12 -> 18
- added copper zone on B.Cu, net GND
- added copper zone on F.Cu, net GND
Other:
- board size 49.9 x 54.9 mm -> 49.4 x 53.2 mm

Commit message: save
Parts:
- moved U8 4.24 mm to (158.1, 83.5), turned to -90 degrees
- moved C4 3.92 mm to (148.0, 72.9), turned to 180 degrees
- moved C3 3.92 mm to (148.0, 81.1), turned to 180 degrees
- moved R17 2.35 mm to (169.0, 87.8)
- moved R16 2.35 mm to (169.0, 86.2)
- moved R13 1.53 mm to (161.8, 95.5), turned to 180 degrees
- moved C37 0.88 mm to (143.9, 92.1)
- moved C5 0.78 mm to (134.9, 74.8), turned to 180 degrees
- moved C25 0.63 mm to (161.1, 88.9)
- moved C7 0.59 mm to (139.7, 81.5)
- moved C6 0.49 mm to (135.6, 80.8)
- moved C39 0.29 mm to (143.9, 87.0)
- moved Q2 0.23 mm to (165.2, 90.5)
- moved J3 0.14 mm to (168.2, 93.2)
- moved J4 0.14 mm to (170.7, 93.2)
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Connections:
- U1 pad 41: unconnected-(U1-PB5-Pad41) -> /battery charger/CHARGER_STAT
Routing:
- net /battery charger/CHARGER_STAT: track 0.00 -> 17.5 mm, vias 0 -> 3
- net /battery charger/CHARGER_PG: track 3.78 -> 17.1 mm, vias 1 -> 2
- net Net-(U6-EN): track 2.58 -> 12.1 mm, vias 0 -> 2
- net +3V3: track 48.5 -> 57.3 mm, vias 12 -> 16
- net /psu/+VIN_PROTECTED: track 0.67 -> 9.00 mm
- net Net-(D1-A): track 0.00 -> 7.19 mm
- net /mcu/OSC_OUT: track 8.38 -> 11.7 mm
- net /mcu/OSC_IN: track 4.70 -> 7.80 mm
- net Net-(U4-DIS): track 0.00 -> 2.26 mm
- net /mcu/VIN_MEAS: track 45.3 -> 47.3 mm
- net /mcu/OSC32_OUT: track 6.21 -> 7.57 mm
- net /mcu/OSC32_IN: track 6.60 -> 7.94 mm
- net +VSYS: track 0.00 -> 1.15 mm
- net Net-(U4-SS): track 0.00 -> 1.11 mm
- net /gsm/TXD: track 10.0 -> 10.7 mm
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- added copper zone on F.Cu, net /+VIN
- added copper zone on B.Cu, net /psu/+VIN_PROTECTED
- added copper zone on F.Cu, net /psu/+VIN_PROTECTED
- added copper zone on In2.Cu, net GND

Commit message: save
Parts:
- added C19: 10u, Capacitor_SMD:C_0805_2012Metric, B.Cu at (140.1, 79.9)
- moved C5 2.23 mm to (134.4, 72.7)
- moved C17 0.50 mm to (134.3, 72.8)
- moved C7 0.20 mm to (139.7, 81.7)
- moved C30 0.14 mm to (137.6, 87.9)
- moved C8 0.12 mm to (140.9, 77.0)
- moved C9 0.12 mm to (140.9, 75.4)
Connections:
- U1 pad 1: unconnected-(U1-VBAT-Pad1) -> Net-(U1-VBAT)
- U1 pad 14: unconnected-(U1-PA4-Pad14) -> /gsm/GSM_EN
- U1 pad 25: unconnected-(U1-PB12-Pad25) -> /gsm/GSM_DTR
- U1 pad 32: unconnected-(U1-PA11-Pad32) -> /mcu/PSU_CTRL
Routing:
- net /mcu/PSU_CTRL: track 0.00 -> 33.3 mm, vias 0 -> 2
- net /gsm/GSM_DTR: track 0.00 -> 28.5 mm, vias 0 -> 2
- net GND: track 0.91 -> 17.8 mm, vias 19 -> 33
- net /gsm/GSM_EN: track 0.00 -> 11.7 mm, vias 0 -> 2
- net Net-(U1-VBAT): track 0.00 -> 2.61 mm, vias 0 -> 1
- net /mcu/OCTOSPI1_NCS: track 15.0 -> 16.7 mm
- net +3V3: track 57.3 -> 56.1 mm
- net /gsm/GSM_PWRKEY: track 23.1 -> 24.3 mm
- net /gsm/GPS_RX: track 27.8 -> 28.9 mm
- net /mcu/RESET: track 17.9 -> 18.8 mm
- net /battery charger/CHARGER_STAT: track 17.5 -> 18.1 mm
- net /gsm/GSM_RESET: track 22.4 -> 21.8 mm
- net /gsm/GSM_LINE_BUF_EN: track 33.4 -> 32.8 mm

Commit message: edits
Parts:
- removed C12: 0.1u, Capacitor_SMD:C_0603_1608Metric
- removed Q1: SSM6N7002KFU, Package_TO_SOT_SMD:SOT-363_SC-70-6
- added C38: 0.1u, Capacitor_SMD:C_0603_1608Metric, F.Cu at (162.1, 81.2)
- added C43: 0.1u, Capacitor_SMD:C_0603_1608Metric, F.Cu at (162.0, 71.7)
- added U11: PUMH10,115, Package_TO_SOT_SMD:SOT-363_SC-70-6, F.Cu at (152.6, 77.5)
- U3: value 74LVC244APW,118 -> NXB0108PW
- moved U3 1.69 mm to (158.9, 76.4)
- moved C18 1.65 mm to (153.3, 72.5), turned to 90 degrees
- moved C11 0.96 mm to (142.3, 63.2), turned to 90 degrees
Connections:
- C19 pad 1: Net-(U1-VBAT) -> +3V3
- U1 pad 1: Net-(U1-VBAT) -> +3V3
- U1 pad 44: /gsm/GSM_LINE_BUF_EN -> /gsm/GSM_STATUS
- U1 pad 46: /gsm/GSM_STATUS -> /gsm/GSM_LINE_BUF_EN
- U3 pad 1: /gsm/GSM_LINE_BUF_EN -> /gsm/STATUS
- U3 pad 10: GND -> /gsm/GSM_LINE_BUF_EN
- U3 pad 11: /gsm/GSM_TX -> GND
- U3 pad 12: /gsm/GSM_RX -> /gsm/GPS_RX
- U3 pad 14: /gsm/GSM_DTR -> /gsm/GPS_TX
- U3 pad 15: /gsm/GPS_RX -> /gsm/GSM_TX
- U3 pad 16: /gsm/GPS_TX -> /gsm/GSM_RX
- U3 pad 17: /gsm/GSM_STATUS -> /gsm/GSM_DTR
- U3 pad 19: /gsm/GSM_LINE_BUF_EN -> +3V3
- U3 pad 2: /gsm/AP_RDY -> +2V8
- U3 pad 20: +3V3 -> /gsm/GSM_STATUS
- U3 pad 3: /gsm/STATUS -> /gsm/AP_RDY
- U3 pad 4: /gsm/U3_TXD -> /gsm/DTR
- U3 pad 5: /gsm/U3_RXD -> /gsm/RXD
- U3 pad 6: /gsm/DTR -> /gsm/TXD
- U3 pad 7: /gsm/RI -> /gsm/U3_TXD
- U3 pad 8: /gsm/RXD -> /gsm/RI
- U3 pad 9: /gsm/TXD -> /gsm/U3_RXD
Routing:
- net /gsm/GSM_LINE_BUF_EN: track 32.8 -> 25.7 mm
- net /gsm/GSM_STATUS: track 23.6 -> 28.7 mm
- net /gsm/U3_RXD: track 8.38 -> 3.82 mm
- net /gsm/GSM_TX: track 14.6 -> 19.1 mm
- net /gsm/STATUS: track 8.87 -> 4.98 mm
- net /gsm/GSM_RX: track 16.4 -> 20.2 mm
- net /gsm/AP_RDY: track 10.6 -> 7.74 mm
- net /gsm/U3_TXD: track 6.77 -> 4.04 mm
- net Net-(U1-VBAT): track 2.61 -> 0.00 mm, vias 1 -> 0
- net /gsm/GSM_DTR: track 28.5 -> 31.1 mm
- net /gsm/RXD: track 10.2 -> 12.5 mm
- net /gsm/GPS_RX: track 28.9 -> 27.4 mm
- net /gsm/GPS_TX: track 29.0 -> 27.6 mm
- net /gsm/TXD: track 10.7 -> 11.8 mm
- net /gsm/GSM_RI: track 17.4 -> 18.4 mm
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
Commit message: edits
Parts:
- removed U5: DF5A6.8JE,LM, Package_TO_SOT_SMD:Diodes_SOT-553
- added U12: DF6A6.8FUT, Package_TO_SOT_SMD:SOT-363_SC-70-6, F.Cu at (151.2, 64.2)
Routing:
- net +2V8: track 1.88 -> 13.4 mm, vias 0 -> 2
- net Net-(J2-I/O): track 6.54 -> 9.32 mm
- net Net-(J2-CLK): track 8.01 -> 10.2 mm
- net /gsm/SIM_VCC: track 9.32 -> 8.58 mm
- net Net-(J2-RST): track 5.90 -> 6.49 mm
- net GND: vias 60 -> 63

Commit message: save
Parts:
- added C42: 0.1u, Capacitor_SMD:C_0603_1608Metric, B.Cu at (130.7, 85.5)
- added U12: MC3479, Package_LGA:LGA-12_2x2mm_P0.5mm, B.Cu at (133.6, 84.3)
- renumbered C8 to C10, C9 to C11, C10 to C12, C38 to C13, C11 to C14, C43 to C15, C13 to C16, C14 to C17, C15 to C18, C18 to C19, C16 to C20, C20 to C21, C21 to C22, C22 to C23, C23 to C24, C24 to C25, C25 to C26, C26 to C27, C27 to C28, C28 to C29, C29 to C30, C30 to C31, C31 to C32, C32 to C33, C41 to C34, C33 to C35, C42 to C36, C35 to C37, C36 to C38, C37 to C39, C39 to C40, C40 to C41, C17 to C5, C5 to C6, C19 to C7, C6 to C8, C7 to C9, J3 to J1, J4 to J2, J1 to J3, J5 to J4, J2 to J5, Q2 to Q1, R13 to R1, R7 to R10, R8 to R11, R14 to R12, R9 to R13, R10 to R14, R11 to R16, R12 to R17, R4 to R2, R17 to R3, R16 to R4, R1 to R5, R2 to R6, R3 to R7, R5 to R8, R6 to R9, U9 to U11, U11 to U3, U3 to U4, U4 to U5, U12 to U6, U8 to U7, U6 to U8, U7 to U9, Y3 to Y1
Connections:
- net /mcu/I2C_SCL renamed /I2C_SCL
- net /mcu/I2C_SDA renamed /I2C_SDA
- U1 pad 29: unconnected-(U1-PA8-Pad29) -> /accelerometer/ACC_INT1
Routing:
- net /accelerometer/ACC_INT1: track 0.00 -> 9.39 mm, vias 0 -> 1
- net /I2C_SDA: track 18.7 -> 23.5 mm, vias 1 -> 2
- net /I2C_SCL: track 21.4 -> 25.3 mm, vias 1 -> 2
- net +3V3: track 55.5 -> 58.1 mm
- net /battery charger/CHARGER_INT: track 17.1 -> 19.6 mm
- net /battery charger/CHARGER_STAT: track 18.1 -> 18.7 mm
- net GND: vias 63 -> 62
