File: tracker/tracker.kicad_pcb (KiCad board)
At the start: 2 copper layers, 50.5 x 56.9 mm, 76 parts, among them J1 Conn_01x10, J2 SIM_Card, M1 BG96, Q1 SSM6N7002KFU, Q2 SSM6N7002KFU, Q3 SSM6N7002KFU, U1 STM32U545CEUx, U2 GD25QxxxEY, U3 74LVC244APW,118, U4 AP22800HB-7, U5 DF5A6.8JE,LM, U6 LMR51430, U7 AP61100Z6, U8 BQ25601, Y1 32.768KHz, Y2 8MHz

Commit message: first version
Parts:
- removed the C12 at (96.8, 85.8)
- removed the C17 at (149.0, 71.7)
- removed the C19 at (155.5, 50.7)
- removed the C38 at (186.6, 98.0)
- removed Q2, Q3: SSM6N7002KFU, Package_TO_SOT_SMD:SOT-363_SC-70-6
- removed the R13 at (190.2, 92.5)
- removed the R14 at (190.2, 94.5)
- removed the U5 at (148.9, 63.0)
- removed the U8 at (145.7, 89.0)
- added C13: 0.1u, Capacitor_SMD:C_0603_1608Metric, F.Cu at (162.1, 81.2)
- added C15: 0.1u, Capacitor_SMD:C_0603_1608Metric, F.Cu at (162.0, 71.7)
- added C36: 0.1u, Capacitor_SMD:C_0603_1608Metric, B.Cu at (153.5, 89.8)
- added C42: 0.1u, Capacitor_SMD:C_0603_1608Metric, B.Cu at (130.7, 85.5)
- added C5: 4.7u, Capacitor_SMD:C_0603_1608Metric, F.Cu at (134.3, 72.8)
- added C7: 10u, Capacitor_SMD:C_0805_2012Metric, B.Cu at (140.1, 79.9)
- added D1: 12V, Diode_SMD:D_SOD-323, F.Cu at (165.2, 95.3)
- added J2: Conn_01x01, My Footprints:pad_smd_1.5x3, F.Cu at (170.5, 93.2)
- added J3: Conn_01x05, Connector_JST:JST_PH_B5B-PH-SM4-TB_1x05-1MP_P2.00mm_Vertical, F.Cu at (127.8, 80.2)
- added J4: Conn_Coaxial, Connector_Coaxial:U.FL_Molex_MCRF_73412-0110_Vertical, B.Cu at (164.0, 46.4)
- added J6: Conn_01x02, Connector_JST:JST_XH_B2B-XH-A_1x02_P2.50mm_Vertical, B.Cu at (131.2, 92.0)
- added R1: 10K, Resistor_SMD:R_0603_1608Metric, F.Cu at (161.8, 95.5)
- added R12: 200K, Resistor_SMD:R_0402_1005Metric, B.Cu at (137.6, 92.6)
- added R15: TBD, Resistor_SMD:R_0402_1005Metric, B.Cu at (148.8, 94.5)
- added R2: 220K, Resistor_SMD:R_0603_1608Metric, F.Cu at (165.3, 93.5)
- added R3: 150K, Resistor_SMD:R_0603_1608Metric, F.Cu at (169.0, 87.8)
- added U10: PUMH10,115, Package_TO_SOT_SMD:SOT-363_SC-70-6, F.Cu at (133.5, 84.7)
- added U11: ~, My Footprints:BQ25622E, B.Cu at (148.9, 90.4)
- added U12: MC3479, Package_LGA:LGA-12_2x2mm_P0.5mm, B.Cu at (133.6, 84.3)
- added U4: NXB0108PW, Package_SO:TSSOP-20_4.4x6.5mm_P0.65mm, F.Cu at (158.9, 76.4)
- added U6: DF6A6.8FUT, Package_TO_SOT_SMD:SOT-363_SC-70-6, F.Cu at (151.2, 64.2)
- added U7: PUMH10,115, Package_TO_SOT_SMD:SOT-363_SC-70-6, F.Cu at (158.1, 83.5)
- C10: renamed from C8; footprint Capacitor_SMD:C_0402_1005Metric -> Capacitor_SMD:C_0603_1608Metric
- C11: renamed from C9; footprint Capacitor_SMD:C_0402_1005Metric -> Capacitor_SMD:C_0603_1608Metric
- C12: renamed from C10; footprint Capacitor_SMD:C_0402_1005Metric -> Capacitor_SMD:C_0603_1608Metric
- C14: renamed from C11; footprint Capacitor_SMD:C_0402_1005Metric -> Capacitor_SMD:C_0603_1608Metric
- C16: renamed from C13; footprint Capacitor_SMD:C_0402_1005Metric -> Capacitor_SMD:C_0603_1608Metric
- C17: renamed from C14; footprint Capacitor_SMD:C_0402_1005Metric -> Capacitor_SMD:C_0603_1608Metric
- C18: renamed from C15; moved to B.Cu
- C20: renamed from C16; moved to B.Cu
- C21: renamed from C20; footprint Capacitor_SMD:C_0402_1005Metric -> Capacitor_SMD:C_0603_1608Metric; moved to B.Cu
- C22: renamed from C21; footprint Capacitor_SMD:C_0402_1005Metric -> Capacitor_SMD:C_0603_1608Metric; moved to B.Cu
- C23: renamed from C22; footprint Capacitor_SMD:C_0402_1005Metric -> Capacitor_SMD:C_0603_1608Metric
- C30: renamed from C29; moved to B.Cu
- C31: renamed from C30; moved to B.Cu
- C32: renamed from C31; moved to B.Cu
- C33: renamed from C32; moved to B.Cu
- C34, L3, L4: moved to B.Cu
- C38: renamed from C36; moved to B.Cu
- C39: renamed from C37; moved to B.Cu
- C40: renamed from C39; moved to B.Cu
- C41: renamed from C40; moved to B.Cu
- C6: renamed from C5; footprint Capacitor_SMD:C_0402_1005Metric -> Capacitor_SMD:C_0603_1608Metric
- C8: renamed from C6; footprint Capacitor_SMD:C_0402_1005Metric -> Capacitor_SMD:C_0603_1608Metric
- C9: renamed from C7; footprint Capacitor_SMD:C_0402_1005Metric -> Capacitor_SMD:C_0603_1608Metric
- J1: value Conn_01x10 -> Conn_01x01; footprint Connector:Tag-Connect_TC2050-IDC-NL_2x05_P1.27mm_Vertical -> My Footprints:pad_smd_1.5x3
- Q1: value SSM6N7002KFU -> DMP2008UFG; footprint Package_TO_SOT_SMD:SOT-363_SC-70-6 -> Package_SON:Diodes_PowerDI3333-8
- R13: renamed from R9; moved to B.Cu
- R14: renamed from R10; moved to B.Cu
- R16: renamed from R11; moved to B.Cu
- R17: renamed from R12; moved to B.Cu
- R4: value 200K -> 10K; footprint Resistor_SMD:R_0402_1005Metric -> Resistor_SMD:R_0603_1608Metric
- U2: moved to F.Cu
- U3: value 74LVC244APW,118 -> PUMH10,115; footprint Package_SO:TSSOP-20_4.4x6.5mm_P0.65mm -> Package_TO_SOT_SMD:SOT-363_SC-70-6
- U9: renamed from U7; moved to B.Cu
- moved C29 69.5 mm to (157.0, 89.5)
- moved C4 58.0 mm to (148.0, 72.9), turned to 180 degrees
- moved C23 57.5 mm to (153.0, 60.1), turned to 90 degrees
- moved C3 54.4 mm to (148.0, 81.1), turned to 180 degrees
- moved J1 54.0 mm to (168.2, 93.2), turned to 90 degrees
- moved C2 51.8 mm to (145.9, 81.5)
- moved C1 50.7 mm to (145.9, 85.0), turned to 180 degrees
- moved L4 48.1 mm to (150.5, 86.3), turned to 90 degrees
- moved C41 45.2 mm to (143.9, 89.1), turned to 180 degrees
- moved C40 44.9 mm to (143.9, 87.0), turned to 180 degrees
- moved C38 43.6 mm to (150.1, 94.2), turned to -90 degrees
- moved R16 43.2 mm to (147.3, 93.1), turned to 180 degrees
- moved R17 43.1 mm to (147.3, 94.2)
- moved C39 42.8 mm to (143.9, 92.1), turned to 180 degrees
- moved C37 41.8 mm to (150.2, 90.4), turned to -90 degrees
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- renumbered C18 to C19, C23 to C24, C24 to C25, C25 to C26, C26 to C27, C27 to C28, C28 to C29, C33 to C35, C35 to C37, J2 to J5, R7 to R10, R8 to R11, R1 to R5, R2 to R6, R3 to R7, R5 to R8, R6 to R9, U4 to U5, U6 to U8
Connections:
- net Net-(AE1-A) renamed /gsm/ANT_GNSS
- C12 pad 1: Net-(U2-VCC) -> +3V3
- C24 pad 1: /psu/+VIN -> /psu/+VIN_PROTECTED
- C25 pad 1: /psu/+VIN -> /psu/+VIN_PROTECTED
- C30 pad 1: /low_voltage_psu/+VSYS -> +VSYS
- C31 pad 1: /low_voltage_psu/+3V3 -> +3V3
- C38 pad 1: Net-(U8-REGN) -> Net-(U11-REGN)
- C39 pad 1: Net-(C37-Pad1) -> /battery charger/+BAT
- C40 pad 1: /battery charger/+VSYS -> +VSYS
- C41 pad 1: /battery charger/+VSYS -> +VSYS
- J1 pad 1: +3V3 -> /+VIN
- J5 pad 2: Net-(J2-RST) -> Net-(J5-RST)
- J5 pad 3: Net-(J2-CLK) -> Net-(J5-CLK)
- L3 pad 2: /low_voltage_psu/+3V3 -> +3V3
- L4 pad 2: /battery charger/+VSYS -> +VSYS
- M1 pad 60: unconnected-(M1-ANT_MAIN-Pad60) -> /gsm/ANT_MAIN
- Q1 pad 1: GND -> /psu/+VIN_PROTECTED
- Q1 pad 2: /gsm/GSM_RESET -> /psu/+VIN_PROTECTED
- Q1 pad 3: /gsm/PWRKEY -> /psu/+VIN_PROTECTED
- Q1 pad 4: GND -> Net-(D1-A)
- Q1 pad 5: /gsm/GSM_PWRKEY -> /+VIN
- R13 pad 2: /low_voltage_psu/+3V3 -> +3V3
- R16 pad 1: Net-(U8-REGN) -> Net-(U11-TS_BIAS)
- R4 pad 1: +3V3 -> /mcu/VIN_MEAS
- R4 pad 2: /mcu/PSU_CTRL -> GND
- R5 pad 1: /mcu/I2C_SCL -> /I2C_SCL
- R6 pad 1: /mcu/I2C_SDA -> /I2C_SDA
- R8 pad 1: /psu/+VIN -> /psu/+VIN_PROTECTED
- RN1 pad 1: /gsm/SIM_CLK -> /gsm/SIM_RST
- RN1 pad 3: /gsm/SIM_RST -> /gsm/SIM_CLK
- RN1 pad 6: Net-(J2-RST) -> Net-(J5-CLK)
- RN1 pad 8: Net-(J2-CLK) -> Net-(J5-RST)
- U1 pad 1: unconnected-(U1-VBAT-Pad1) -> +3V3
- U1 pad 14: /mcu/OCTOSPI1_NCS -> /gsm/GSM_EN
- U1 pad 20: unconnected-(U1-PB2-Pad20) -> /mcu/VIN_MEAS
- U1 pad 22: unconnected-(U1-VCAP-Pad22) -> /mcu/VCAP
- U1 pad 25: unconnected-(U1-PB12-Pad25) -> /gsm/GSM_DTR
- U1 pad 26: unconnected-(U1-PB13-Pad26) -> /gsm/GSM_RESET
- U1 pad 28: unconnected-(U1-PB15-Pad28) -> /gsm/GSM_PWRKEY
- U1 pad 29: /gsm/GSM_STATUS -> /accelerometer/ACC_INT1
- U1 pad 32: unconnected-(U1-PA11-Pad32) -> /mcu/PSU_CTRL
- U1 pad 33: unconnected-(U1-PA12-Pad33) -> /mcu/OCTOSPI1_NCS
- U1 pad 34: unconnected-(U1-PA13-Pad34) -> /mcu/SWDIO
- U1 pad 37: unconnected-(U1-PA14-Pad37) -> /mcu/SWCLK
- U1 pad 38: unconnected-(U1-PA15-Pad38) -> /battery charger/POWER_CYCLE
- U1 pad 39: unconnected-(U1-PB3-Pad39) -> /battery charger/CHARGE_ENABLE
- U1 pad 40: unconnected-(U1-PB4-Pad40) -> /battery charger/CHARGER_INT
- U1 pad 41: unconnected-(U1-PB5-Pad41) -> /battery charger/CHARGER_STAT
- U1 pad 42: unconnected-(U1-PB6-Pad42) -> /I2C_SCL
- U1 pad 43: unconnected-(U1-PB7-Pad43) -> /I2C_SDA
- U1 pad 44: unconnected-(U1-PH3-Pad44) -> /gsm/GSM_STATUS
- U1 pad 45: unconnected-(U1-PB8-Pad45) -> /gsm/GSM_AP_READY
- U1 pad 46: unconnected-(U1-PB9-Pad46) -> /gsm/GSM_LINE_BUF_EN
- U2 pad 8: Net-(U2-VCC) -> +3V3
- U3 pad 1: (no net) -> GND
- U3 pad 2: /gsm/AP_RDY -> /gsm/GSM_RESET
- U3 pad 3: /gsm/STATUS -> /gsm/PWRKEY
- U3 pad 4: /gsm/U3_TXD -> GND
- U3 pad 5: /gsm/U3_RXD -> /gsm/GSM_PWRKEY
- U3 pad 6: /gsm/DTR -> /gsm/RESET
- U8 pad 3: /psu/+VIN -> /psu/+VIN_PROTECTED
- U9 pad 3: /low_voltage_psu/+VSYS -> +VSYS
- U9 pad 5: /low_voltage_psu/+VSYS -> /battery charger/CHARGER_PG
- U9 pad 6: /low_voltage_psu/+3V3 -> +3V3
- Y1 pad 1: /mcu/OSC32_OUT -> /mcu/OSC32_IN
- Y1 pad 2: /mcu/OSC32_IN -> unconnected-(Y1-Pad2)
- Y1 pad 3: (no net) -> unconnected-(Y1-Pad3)
- Y1 pad 4: (no net) -> /mcu/OSC32_OUT
Routing:
- net +3V3: track 0.00 -> 58.1 mm, vias 0 -> 16
- net /mcu/VIN_MEAS: track 0.00 -> 44.2 mm, vias 0 -> 2
- net /mcu/PSU_CTRL: track 0.00 -> 33.3 mm, vias 0 -> 2
- net /gsm/GSM_DTR: track 0.00 -> 30.9 mm, vias 0 -> 2
- net /gsm/GSM_STATUS: track 0.00 -> 28.7 mm, vias 0 -> 2
- net /gsm/GPS_TX: track 0.00 -> 27.6 mm, vias 0 -> 2
- net /gsm/GPS_RX: track 0.00 -> 27.6 mm, vias 0 -> 2
- net /gsm/GSM_AP_READY: track 0.00 -> 26.6 mm, vias 0 -> 2
- net /gsm/PWRKEY: track 0.00 -> 25.4 mm, vias 0 -> 1
- net /gsm/RESET: track 0.00 -> 25.0 mm, vias 0 -> 1
- net /gsm/GSM_LINE_BUF_EN: track 0.00 -> 24.6 mm, vias 0 -> 2
- net /mcu/OCTOSPI1_IO0: track 0.00 -> 24.3 mm
- net /gsm/GSM_PWRKEY: track 0.00 -> 24.3 mm, vias 0 -> 2
- net Net-(U11-~{CE}): track 0.00 -> 24.2 mm, vias 0 -> 1
- net /mcu/OCTOSPI1_IO2: track 0.00 -> 24.1 mm
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- added copper zone on B.Cu, net +3V3
- added copper zone on In1.Cu, net +3V3
- added copper zone on B.Cu, net +5V
- added copper zone on In1.Cu, net +5V
- added copper zone on B.Cu, net +VSYS
- added copper zone on F.Cu, net +VSYS
- added copper zone on In1.Cu, net +VSYS
- added copper zone on F.Cu, net /+VIN
- added copper zone on B.Cu, net /battery charger/+BAT
- added copper zone on In1.Cu, net /battery charger/+BAT
- added copper zone on B.Cu, net /battery charger/BQ_SW
- added copper zone on F.Cu, net /gsm/+GSM_SWITCHED
- added copper zone on B.Cu, net /gsm/+VBAT_GSM
- added copper zone on F.Cu, net /gsm/+VBAT_GSM
- added copper zone on B.Cu, net /psu/+VIN_PROTECTED
- added copper zone on F.Cu, net /psu/+VIN_PROTECTED
- added copper zone on B.Cu, net GND
- added copper zone on F.Cu, net GND
- added copper zone on In1.Cu, net GND
- added copper zone on In2.Cu, net GND
- added copper zone on B.Cu, net Net-(U8-SW)
- added copper zone on B.Cu, net Net-(U9-SW)
Other:
- board size 50.5 x 56.9 mm -> 49.4 x 53.4 mm
- copper layers 2 -> 4
