File: tracker/battery_charger.kicad_sch (KiCad schematic)
At the start: 17 parts, among them Q3 SSM6N7002KFU, U8 BQ25601

Commit message: save
Parts:
- removed C34: 10u, Capacitor_SMD:C_0805_2012Metric, symbol Device:C_Small
- removed Q3: SSM6N7002KFU, Package_TO_SOT_SMD:SOT-363_SC-70-6, symbol Device:Q_Dual_NMOS_S1G1D2S2G2D1
- removed R13: 37K, Resistor_SMD:R_0402_1005Metric, symbol Device:R_Small
- removed R14: 100K, Resistor_SMD:R_0402_1005Metric, symbol Device:R_Small
- removed U8: BQ25601, Package_DFN_QFN:Texas_RTW_WQFN-24-1EP_4x4mm_P0.5mm_EP2.7x2.7mm_ThermalVias, symbol Battery_Management:BQ25601
- added C41: 10u, Capacitor_SMD:C_0805_2012Metric, symbol Device:C_Small
- added C42: 0.1u, Capacitor_SMD:C_0603_1608Metric, symbol Device:C_Small
- added J6: Conn_01x02, Connector_JST:JST_XH_B2B-XH-A_1x02_P2.50mm_Vertical, symbol Connector_Generic:Conn_01x02
- added R15: TBD, Resistor_SMD:R_0402_1005Metric, symbol Device:R_Small
- added U10: PUMH10,115, Package_TO_SOT_SMD:SOT-363_SC-70-6, symbol My Libraries:PUMH10,115
- added U9: ~, My Footprints:BQ25622E, symbol My Libraries:BQ25622E
Connections:
- net +3V3: now also U10.2, U10.5
- net +5V: now also U9.18 (VBUS)
- net +VSYS: now also U9.9 (SYS)
- net BQ_SW: now also U9.16 (SW)
- net CHARGER_INT: now also U9.11 (~{INT})
- net CHARGER_PG: now also U9.3 (~{PG})
- net CHARGER_STAT: now also U9.10 (STAT)
- net CHARGE_ENABLE: now also U10.1
- net GND: now also C41.2, C42.2, J6.2 (Pin_2), R15.2, U9.15 (GND)
- net POWER_CYCLE: now also U10.4
- net at C35.2: now also U9.1 (BTST)
- net +BAT: now reaches C37.1
- net +BAT: now also J6.1 (Pin_1), U9.8 (BAT)
- net at C36.1: now also U9.2 (REGN); no longer R11.1
- net at R11.2, R12.1: now also U9.6 (TS)
- new net: U10.6, U9.14 (~{CE})
- new net: C41.1, C42.1, U9.17 (PMID)
- new net: R15.1, U9.4 (ILIM)
- new net: R11.1, U9.5 (TS_BIAS)
- new net: U10.3, U9.7 (~{QON})
- new net I2C_SCL: U9.13 (SCL)
- new net I2C_SDA: U9.12 (SDA)
Other:
- moved on the sheet: C31, C32, C33, C35, C36, C37, C38, C39, C40, L4, R11, R12

Commit message: save project
Parts:
- removed C38: 10u, Capacitor_SMD:C_0805_2012Metric, symbol Device:C_Small
Other:
- moved on the sheet: C39, C40
Changed lines of the file:
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@@
 	)
 	(junction
-		(at 208.28 43.18)
+		(at 199.39 43.18)
 		(diameter 0.9144)
 		(color 0 0 0 0)
@@
 	)
 	(junction
-		(at 198.12 43.18)
-		(diameter 0.9144)
-		(color 0 0 0 0)
-	)
-	(junction
 		(at 111.76 43.18)
 		(diameter 0.9144)
@@
 	)
 	(junction
-		(at 218.44 43.18)
+		(at 209.55 43.18)
 		(diameter 0.9144)
 		(color 0 0 0 0)
@@
 	(wire
 		(pts
-			(xy 190.5 43.18) (xy 198.12 43.18)
-		)
-		(stroke
-			(width 0)
-			(type solid)
-		)
-	)
-	(wire
-		(pts
-			(xy 198.12 43.18) (xy 208.28 43.18)
+			(xy 190.5 43.18) (xy 199.39 43.18)
 		)
 		(stroke
@@
 	(wire
 		(pts
-			(xy 208.28 43.18) (xy 218.44 43.18)
-		)
-		(stroke
-			(width 0)
-			(type solid)
-		)
-	)
-	(wire
-		(pts
-			(xy 218.44 43.18) (xy 228.6 43.18)
+			(xy 199.39 43.18) (xy 209.55 43.18)
+		)
+		(stroke
+			(width 0)
+			(type solid)
+		)
+	)
+	(wire
+		(pts
+			(xy 209.55 43.18) (xy 226.06 43.18)
 		)
 		(stroke
@@
 	(hierarchical_label "+VSYS"
 		(shape input)
-		(at 228.6 43.18 0)
+		(at 226.06 43.18 0)
 		(effects
 			(font
@@
 	(symbol
 		(lib_id "Device:C_Small")
-		(at 208.28 45.72 0)
+		(at 199.39 45.72 0)
 		(unit 1)
 		(exclude_from_sim no)
@@
 		(fields_autoplaced yes)
 		(property "Reference" "C39"
-			(at 210.82 45.0849 0)
+			(at 201.93 45.0849 0)
 			(effects
 				(font
@@
 		)
 		(property "Value" "10u"
-			(at 210.82 47.6249 0)
+			(at 201.93 47.6249 0)
 			(effects
 				(font
@@
 		)
 		(property "Footprint" "Capacitor_SMD:C_0805_2012Metric"
-			(at 208.28 45.72 0)
+			(at 199.39 45.72 0)
 			(effects
 				(font
@@
 		)
 		(property "Datasheet" "~"
-			(at 208.28 45.72 0)
+			(at 199.39 45.72 0)
 			(effects
 				(font
@@
 		)
 		(property "Description" "Unpolarized capacitor, small symbol"
-			(at 208.28 45.72 0)
+			(at 199.39 45.72 0)
 			(effects
 				(font
@@
 	(symbol
 		(lib_id "power:GND")
-		(at 218.44 48.26 0)
+		(at 209.55 48.26 0)
 		(unit 1)
 		(exclude_from_sim no)
@@
 		(dnp no)
 		(property "Reference" "#PWR066"
-			(at 218.44 54.61 0)
+			(at 209.55 54.61 0)
 			(effects
 				(font
@@
 		)
 		(property "Value" "GND"
-			(at 218.44 52.07 0)
+			(at 209.55 52.07 0)
 			(effects
 				(font
@@
 		)
 		(property "Footprint" ""
-			(at 218.44 48.26 0)
+			(at 209.55 48.26 0)
 			(effects
 				(font
@@
 		)
 		(property "Datasheet" ""
-			(at 218.44 48.26 0)
+			(at 209.55 48.26 0)
 			(effects
 				(font
@@
 		)
 		(property "Description" "Power symbol creates a global label with name \"GND\" , ground"
-			(at 218.44 48.26 0)
+			(at 209.55 48.26 0)
 			(effects
 				(font
@@
 	)
 	(symbol
-		(lib_id "Device:C_Small")
-		(at 198.12 45.72 0)
-		(unit 1)
-		(exclude_from_sim no)
-		(in_bom yes)
-		(on_board yes)
-		(dnp no)
-		(fields_autoplaced yes)
-		(property "Reference" "C38"
-			(at 200.66 45.0849 0)
-			(effects
-				(font
-					(size 1.27 1.27)
-				)
-				(justify left)
-			)
-		)
-		(property "Value" "10u"
-			(at 200.66 47.6249 0)
-			(effects
-				(font
-					(size 1.27 1.27)
-				)
-				(justify left)
-			)
-		)
-		(property "Footprint" "Capacitor_SMD:C_0805_2012Metric"
-			(at 198.12 45.72 0)
-			(effects
-				(font
-					(size 1.27 1.27)
-				)
-				(hide yes)
-			)
-		)
-		(property "Datasheet" "~"
-			(at 198.12 45.72 0)
-			(effects
-				(font
-					(size 1.27 1.27)
-				)
-				(hide yes)
-			)
-		)
-		(property "Description" "Unpolarized capacitor, small symbol"
-			(at 198.12 45.72 0)
-			(effects
-				(font
-					(size 1.27 1.27)
-				)
-				(hide yes)
-			)
-		)
-		(pin "1"
-		)
-		(pin "2"
-		)
-		(instances
-			(project "BK4000TG_V3"
-				(path "/12391f46-36fb-49a8-aa55-7542601826a6/c65676c7-aef7-4daf-8f47-0f811de4e8b5"
-					(reference "C22")
-					(unit 1)
-				)
-			)
-			(project "BK4000TG_V3"
-				(path "/4f1d18f5-7d2b-4d0b-8633-b1619d53124c/f6a238ba-2427-4db5-a4e9-0e2d7bd0deba"
-					(reference "C38")
-					(unit 1)
-				)
-			)
-		)
-	)
-	(symbol
 		(lib_id "power:GND")
 		(at 124.46 60.96 0)
@@
 	(symbol
 		(lib_id "power:GND")
-		(at 208.28 48.26 0)
+		(at 199.39 48.26 0)
 		(unit 1)
 		(exclude_from_sim no)
@@
 		(dnp no)
 		(property "Reference" "#PWR065"
-			(at 208.28 54.61 0)
+			(at 199.39 54.61 0)
 			(effects
 				(font
@@
 		)
 		(property "Value" "GND"
-			(at 208.28 52.07 0)
+			(at 199.39 52.07 0)
 			(effects
 				(font
@@
 		)
 		(property "Footprint" ""
-			(at 208.28 48.26 0)
+			(at 199.39 48.26 0)
 			(effects
 				(font
@@
 		)
 		(property "Datasheet" ""
-			(at 208.28 48.26 0)
+			(at 199.39 48.26 0)
 			(effects
 				(font
@@
 		)
 		(property "Description" "Power symbol creates a global label with name \"GND\" , ground"
-			(at 208.28 48.26 0)
+			(at 199.39 48.26 0)
 			(effects
 				(font
@@
 	(symbol
 		(lib_id "Device:C_Small")
-		(at 218.44 45.72 0)
+		(at 209.55 45.72 0)
 		(unit 1)
 		(exclude_from_sim no)
@@
 		(fields_autoplaced yes)
 		(property "Reference" "C40"
-			(at 220.98 45.0849 0)
+			(at 212.09 45.0849 0)
 			(effects
 				(font
@@
 		)
 		(property "Value" "10u"
-			(at 220.98 47.6249 0)
+			(at 212.09 47.6249 0)
 			(effects
 				(font
@@
 		)
 		(property "Footprint" "Capacitor_SMD:C_0805_2012Metric"
-			(at 218.44 45.72 0)
+			(at 209.55 45.72 0)
 			(effects
 				(font
@@
 		)
 		(property "Datasheet" "~"
-			(at 218.44 45.72 0)
+			(at 209.55 45.72 0)
 			(effects
 				(font
@@
 		)
 		(property "Description" "Unpolarized capacitor, small symbol"
-			(at 218.44 45.72 0)
+			(at 209.55 45.72 0)
 			(effects
 				(font
@@
 					(unit 1)
 				)
-			)
-		)
-	)
-	(symbol
-		(lib_id "power:GND")
-		(at 198.12 48.26 0)
-		(unit 1)
-		(exclude_from_sim no)
-		(in_bom yes)
-		(on_board yes)
-		(dnp no)
-		(property "Reference" "#PWR063"
-			(at 198.12 54.61 0)
-			(effects
-				(font
-					(size 1.27 1.27)
-				)
-				(hide yes)
-			)
-		)
-		(property "Value" "GND"
-			(at 198.12 52.07 0)
-			(effects
-				(font
-					(size 1.27 1.27)
-				)
-			)
-		)
-		(property "Footprint" ""
-			(at 198.12 48.26 0)
-			(effects
-				(font
-					(size 1.27 1.27)
-				)
-				(hide yes)
-			)
-		)
-		(property "Datasheet" ""
-			(at 198.12 48.26 0)
-			(effects
-				(font
-					(size 1.27 1.27)
-				)
-				(hide yes)
-			)
-		)
-		(property "Description" "Power symbol creates a global label with name \"GND\" , ground"
-			(at 198.12 48.26 0)
-			(effects
-				(font
-					(size 1.27 1.27)
-				)
-				(hide yes)
-			)
-		)
-		(pin "1"
-		)
-		(instances
-			(project "BK4000TG_V3"
-				(path "/12391f46-36fb-49a8-aa55-7542601826a6/c65676c7-aef7-4daf-8f47-0f811de4e8b5"
-					(reference "#PWR064")
-					(unit 1)
-				)
-			)
-			(project "BK4000TG_V3"
-				(path "/4f1d18f5-7d2b-4d0b-8633-b1619d53124c/f6a238ba-2427-4db5-a4e9-0e2d7bd0deba"
-					(reference "#PWR063")
-					(unit 1)
-				)

Commit message: save
Parts:
- renumbered C31 to C32, C32 to C33, C41 to C34, C33 to C35, C42 to C36, C35 to C37, C36 to C38, C37 to C39, C39 to C40, C40 to C41, R11 to R16, R12 to R17, U9 to U11
Changed lines of the file:
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@@
 		(on_board yes)
 		(dnp no)
-		(property "Reference" "#PWR059"
+		(property "Reference" "#PWR076"
 			(at 147.32 107.95 0)
 			(effects
@@
 			(project "BK4000TG_V3"
 				(path "/4f1d18f5-7d2b-4d0b-8633-b1619d53124c/f6a238ba-2427-4db5-a4e9-0e2d7bd0deba"
-					(reference "#PWR059")
+					(reference "#PWR076")
 					(unit 1)
 				)
@@
 		(dnp no)
 		(fields_autoplaced yes)
-		(property "Reference" "C35"
+		(property "Reference" "C37"
 			(at 167.64 45.0849 0)
 			(effects
@@
 			(project "BK4000TG_V3"
 				(path "/4f1d18f5-7d2b-4d0b-8633-b1619d53124c/f6a238ba-2427-4db5-a4e9-0e2d7bd0deba"
-					(reference "C35")
+					(reference "C37")
 					(unit 1)
 				)
@@
 		(on_board yes)
 		(dnp no)
-		(property "Reference" "#PWR057"
+		(property "Reference" "#PWR073"
 			(at 121.92 54.61 0)
 			(effects
@@
 			(project "BK4000TG_V3"
 				(path "/4f1d18f5-7d2b-4d0b-8633-b1619d53124c/f6a238ba-2427-4db5-a4e9-0e2d7bd0deba"
-					(reference "#PWR057")
+					(reference "#PWR073")
 					(unit 1)
 				)
@@
 		(on_board yes)
 		(dnp no)
-		(property "Reference" "#PWR061"
+		(property "Reference" "#PWR077"
 			(at 165.1 64.77 0)
 			(effects
@@
 			(project "BK4000TG_V3"
 				(path "/4f1d18f5-7d2b-4d0b-8633-b1619d53124c/f6a238ba-2427-4db5-a4e9-0e2d7bd0deba"
-					(reference "#PWR061")
+					(reference "#PWR077")
 					(unit 1)
 				)
@@
 		(on_board yes)
 		(dnp no)
-		(property "Reference" "#PWR074"
+		(property "Reference" "#PWR082"
 			(at 220.98 80.01 0)
 			(effects
@@
 			(project "tracker"
 				(path "/4f1d18f5-7d2b-4d0b-8633-b1619d53124c/f6a238ba-2427-4db5-a4e9-0e2d7bd0deba"
-					(reference "#PWR074")
+					(reference "#PWR082")
 					(unit 1)
 				)
@@
 		(dnp no)
 		(fields_autoplaced yes)
-		(property "Reference" "C37"
+		(property "Reference" "C39"
 			(at 190.5 73.0249 0)
 			(effects
@@
 			(project "BK4000TG_V3"
 				(path "/4f1d18f5-7d2b-4d0b-8633-b1619d53124c/f6a238ba-2427-4db5-a4e9-0e2d7bd0deba"
-					(reference "C37")
+					(reference "C39")
 					(unit 1)
 				)
@@
 		(dnp no)
 		(fields_autoplaced yes)
-		(property "Reference" "#FLG02"
+		(property "Reference" "#FLG06"
 			(at 215.9 69.215 0)
 			(effects
@@
 			(project "BK4000TG_V3"
 				(path "/4f1d18f5-7d2b-4d0b-8633-b1619d53124c/f6a238ba-2427-4db5-a4e9-0e2d7bd0deba"
-					(reference "#FLG02")
+					(reference "#FLG06")
 					(unit 1)
 				)
@@
 		(on_board yes)
 		(dnp no)
-		(property "Reference" "U9"
+		(property "Reference" "U11"
 			(at 147.574 38.862 0)
 			(effects
@@
 			(project ""
 				(path "/4f1d18f5-7d2b-4d0b-8633-b1619d53124c/f6a238ba-2427-4db5-a4e9-0e2d7bd0deba"
-					(reference "U9")
+					(reference "U11")
 					(unit 1)
 				)
@@
 		(on_board yes)
 		(dnp no)
-		(property "Reference" "#PWR062"
+		(property "Reference" "#PWR079"
 			(at 187.96 82.55 0)
 			(effects
@@
 			(project "BK4000TG_V3"
 				(path "/4f1d18f5-7d2b-4d0b-8633-b1619d53124c/f6a238ba-2427-4db5-a4e9-0e2d7bd0deba"
-					(reference "#PWR062")
+					(reference "#PWR079")
 					(unit 1)
 				)
@@
 		(dnp no)
 		(fields_autoplaced yes)
-		(property "Reference" "C31"
+		(property "Reference" "C32"
 			(at 101.6 45.0849 0)
 			(effects
@@
 			(project "BK4000TG_V3"
 				(path "/4f1d18f5-7d2b-4d0b-8633-b1619d53124c/f6a238ba-2427-4db5-a4e9-0e2d7bd0deba"
-					(reference "C31")
+					(reference "C32")
 					(unit 1)
 				)
@@
 		(dnp no)
 		(fields_autoplaced yes)
-		(property "Reference" "C39"
+		(property "Reference" "C40"
 			(at 201.93 45.0849 0)
 			(effects
@@
 			(project "BK4000TG_V3"
 				(path "/4f1d18f5-7d2b-4d0b-8633-b1619d53124c/f6a238ba-2427-4db5-a4e9-0e2d7bd0deba"
-					(reference "C39")
+					(reference "C40")
 					(unit 1)
 				)
@@
 		(dnp no)
 		(fields_autoplaced yes)
-		(property "Reference" "C41"
+		(property "Reference" "C34"
 			(at 118.11 57.7849 0)
 			(effects
@@
 			(project "tracker"
 				(path "/4f1d18f5-7d2b-4d0b-8633-b1619d53124c/f6a238ba-2427-4db5-a4e9-0e2d7bd0deba"
-					(reference "C41")
+					(reference "C34")
 					(unit 1)
 				)
@@
 		(on_board yes)
 		(dnp no)
-		(property "Reference" "#PWR066"
+		(property "Reference" "#PWR081"
 			(at 209.55 54.61 0)
 			(effects
@@
 			(project "BK4000TG_V3"
 				(path "/4f1d18f5-7d2b-4d0b-8633-b1619d53124c/f6a238ba-2427-4db5-a4e9-0e2d7bd0deba"
-					(reference "#PWR066")
+					(reference "#PWR081")
 					(unit 1)
 				)
@@
 		(dnp no)
 		(fields_autoplaced yes)
-		(property "Reference" "C32"
+		(property "Reference" "C33"
 			(at 114.3 45.0849 0)
 			(effects
@@
 			(project "BK4000TG_V3"
 				(path "/4f1d18f5-7d2b-4d0b-8633-b1619d53124c/f6a238ba-2427-4db5-a4e9-0e2d7bd0deba"
-					(reference "C32")
+					(reference "C33")
 					(unit 1)
 				)
@@
 		(on_board yes)
 		(dnp no)
-		(property "Reference" "#PWR069"
+		(property "Reference" "#PWR074"
 			(at 124.46 67.31 0)
 			(effects
@@
 			(project "tracker"
 				(path "/4f1d18f5-7d2b-4d0b-8633-b1619d53124c/f6a238ba-2427-4db5-a4e9-0e2d7bd0deba"
-					(reference "#PWR069")
+					(reference "#PWR074")
 					(unit 1)
 				)
@@
 		(on_board yes)
 		(dnp no)
-		(property "Reference" "#PWR068"
+		(property "Reference" "#PWR072"
 			(at 115.57 67.31 0)
 			(effects
@@
 			(project "tracker"
 				(path "/4f1d18f5-7d2b-4d0b-8633-b1619d53124c/f6a238ba-2427-4db5-a4e9-0e2d7bd0deba"
-					(reference "#PWR068")
+					(reference "#PWR072")
 					(unit 1)
 				)
@@
 		(dnp no)
 		(fields_autoplaced yes)
-		(property "Reference" "C36"
+		(property "Reference" "C38"
 			(at 167.64 55.2449 0)
 			(effects
@@
 			(project "BK4000TG_V3"
 				(path "/4f1d18f5-7d2b-4d0b-8633-b1619d53124c/f6a238ba-2427-4db5-a4e9-0e2d7bd0deba"
-					(reference "C36")
+					(reference "C38")
 					(unit 1)
 				)
@@
 		(on_board yes)
 		(dnp no)
-		(property "Reference" "#PWR065"
+		(property "Reference" "#PWR080"
 			(at 199.39 54.61 0)
 			(effects
@@
 			(project "BK4000TG_V3"
 				(path "/4f1d18f5-7d2b-4d0b-8633-b1619d53124c/f6a238ba-2427-4db5-a4e9-0e2d7bd0deba"
-					(reference "#PWR065")
+					(reference "#PWR080")
 					(unit 1)
 				)
@@
 		(dnp no)
 		(fields_autoplaced yes)
-		(property "Reference" "C40"
+		(property "Reference" "C41"
 			(at 212.09 45.0849 0)
 			(effects
@@
 			(project "BK4000TG_V3"
 				(path "/4f1d18f5-7d2b-4d0b-8633-b1619d53124c/f6a238ba-2427-4db5-a4e9-0e2d7bd0deba"
-					(reference "C40")
+					(reference "C41")
 					(unit 1)
 				)
@@
 		(dnp no)
 		(fields_autoplaced yes)
-		(property "Reference" "C42"
+		(property "Reference" "C36"
 			(at 127 57.7849 0)
 			(effects
@@
 			(project "tracker"
 				(path "/4f1d18f5-7d2b-4d0b-8633-b1619d53124c/f6a238ba-2427-4db5-a4e9-0e2d7bd0deba"
-					(reference "C42")
+					(reference "C36")
 					(unit 1)
 				)
@@
 		(dnp no)
 		(fields_autoplaced yes)
-		(property "Reference" "R11"
+		(property "Reference" "R16"
 			(at 172.72 77.4699 0)
 			(effects
@@
 			(project "BK4000TG_V3"
 				(path "/4f1d18f5-7d2b-4d0b-8633-b1619d53124c/f6a238ba-2427-4db5-a4e9-0e2d7bd0deba"
-					(reference "R11")
+					(reference "R16")
 					(unit 1)
 				)
@@
 		(dnp no)
 		(fields_autoplaced yes)
-		(property "Reference" "R12"
+		(property "Reference" "R17"
 			(at 172.72 87.6299 0)
 			(effects
@@
 			(project "BK4000TG_V3"
 				(path "/4f1d18f5-7d2b-4d0b-8633-b1619d53124c/f6a238ba-2427-4db5-a4e9-0e2d7bd0deba"
-					(reference "R12")
+					(reference "R17")
 					(unit 1)
 				)
@@
 		(on_board yes)
 		(dnp no)
-		(property "Reference" "#PWR054"
+		(property "Reference" "#PWR070"
 			(at 99.06 54.61 0)
 			(effects
@@
 			(project "BK4000TG_V3"
 				(path "/4f1d18f5-7d2b-4d0b-8633-b1619d53124c/f6a238ba-2427-4db5-a4e9-0e2d7bd0deba"
-					(reference "#PWR054")
+					(reference "#PWR070")
 					(unit 1)
 				)
@@
 		(on_board yes)
 		(dnp no)
-		(property "Reference" "#PWR052"
+		(property "Reference" "#PWR068"
 			(at 95.25 105.41 0)
 			(effects
@@
 			(project "BK4000TG_V3"
 				(path "/4f1d18f5-7d2b-4d0b-8633-b1619d53124c/f6a238ba-2427-4db5-a4e9-0e2d7bd0deba"
-					(reference "#PWR052")
+					(reference "#PWR068")
 					(unit 1)
 				)
@@
 		(on_board yes)
 		(dnp no)
-		(property "Reference" "#PWR055"
+		(property "Reference" "#PWR071"
 			(at 111.76 54.61 0)
 			(effects
@@
 			(project "BK4000TG_V3"
 				(path "/4f1d18f5-7d2b-4d0b-8633-b1619d53124c/f6a238ba-2427-4db5-a4e9-0e2d7bd0deba"
-					(reference "#PWR055")
+					(reference "#PWR071")
 					(unit 1)
 				)
@@
 		(on_board yes)
 		(dnp no)
-		(property "Reference" "#PWR056"
+		(property "Reference" "#PWR069"
 			(at 95.25 135.89 0)
 			(effects
@@
 			(project "tracker"
 				(path "/4f1d18f5-7d2b-4d0b-8633-b1619d53124c/f6a238ba-2427-4db5-a4e9-0e2d7bd0deba"
-					(reference "#PWR056")
+					(reference "#PWR069")
 					(unit 1)
 				)
@@
 		(on_board yes)
 		(dnp no)
-		(property "Reference" "#PWR060"
+		(property "Reference" "#PWR078"
 			(at 170.18 97.79 0)
 			(effects
@@
 			(project "BK4000TG_V3"
 				(path "/4f1d18f5-7d2b-4d0b-8633-b1619d53124c/f6a238ba-2427-4db5-a4e9-0e2d7bd0deba"
-					(reference "#PWR060")
+					(reference "#PWR078")
 					(unit 1)
 				)
@@
 		(dnp no)
 		(fields_autoplaced yes)
-		(property "Reference" "C33"
+		(property "Reference" "C35"
 			(at 124.46 45.0849 0)
 			(effects
@@
 			(project "BK4000TG_V3"
 				(path "/4f1d18f5-7d2b-4d0b-8633-b1619d53124c/f6a238ba-2427-4db5-a4e9-0e2d7bd0deba"
-					(reference "C33")
+					(reference "C35")
 					(unit 1)
 				)
@@
 		(on_board yes)
 		(dnp no)
-		(property "Reference" "#PWR070"
+		(property "Reference" "#PWR075"
 			(at 128.27 80.01 0)
 			(effects
@@
 			(project "tracker"
 				(path "/4f1d18f5-7d2b-4d0b-8633-b1619d53124c/f6a238ba-2427-4db5-a4e9-0e2d7bd0deba"
-					(reference "#PWR070")
-					(unit 1)
-				)
+					(reference "#PWR075")
+					(unit 1)
+				)
