File: tracker/battery_charger.kicad_sch (KiCad schematic)
At the start: 17 parts, among them J6 Conn_01x02, U10 PUMH10,115

Commit message: Edits
Other:
- moved on the sheet: U10A, U10B
Changed lines of the file:
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@@
 	(wire
 		(pts
-			(xy 119.38 88.9) (xy 134.62 88.9)
+			(xy 80.01 88.9) (xy 134.62 88.9)
 		)
 		(stroke
@@
 	(wire
 		(pts
-			(xy 78.74 147.32) (xy 87.63 147.32)
+			(xy 78.74 156.21) (xy 87.63 156.21)
 		)
 		(stroke
@@
 	(wire
 		(pts
-			(xy 119.38 91.44) (xy 134.62 91.44)
+			(xy 80.01 91.44) (xy 134.62 91.44)
 		)
 		(stroke
@@
 	(wire
 		(pts
-			(xy 124.46 116.84) (xy 100.33 116.84)
+			(xy 124.46 125.73) (xy 100.33 125.73)
 		)
 		(stroke
@@
 	(wire
 		(pts
-			(xy 124.46 96.52) (xy 124.46 116.84)
+			(xy 124.46 96.52) (xy 124.46 125.73)
 		)
 		(stroke
@@
 	(wire
 		(pts
-			(xy 80.01 116.84) (xy 87.63 116.84)
+			(xy 80.01 125.73) (xy 87.63 125.73)
 		)
 		(stroke
@@
 	(wire
 		(pts
-			(xy 119.38 93.98) (xy 134.62 93.98)
+			(xy 80.01 93.98) (xy 134.62 93.98)
 		)
 		(stroke
@@
 	(wire
 		(pts
-			(xy 162.56 93.98) (xy 162.56 147.32)
+			(xy 162.56 93.98) (xy 162.56 156.21)
 		)
 		(stroke
@@
 	(wire
 		(pts
-			(xy 162.56 147.32) (xy 100.33 147.32)
+			(xy 162.56 156.21) (xy 100.33 156.21)
 		)
 		(stroke
@@
 	(wire
 		(pts
-			(xy 119.38 86.36) (xy 134.62 86.36)
+			(xy 80.01 86.36) (xy 134.62 86.36)
 		)
 		(stroke
@@
 	(wire
 		(pts
-			(xy 119.38 83.82) (xy 134.62 83.82)
+			(xy 80.01 83.82) (xy 134.62 83.82)
 		)
 		(stroke
@@
 	(hierarchical_label "CHARGE_ENABLE"
 		(shape input)
-		(at 80.01 116.84 180)
+		(at 80.01 125.73 180)
 		(effects
 			(font
@@
 	(hierarchical_label "I2C_SDA"
 		(shape input)
-		(at 119.38 91.44 180)
+		(at 80.01 91.44 180)
 		(effects
 			(font
@@
 	(hierarchical_label "I2C_SCL"
 		(shape input)
-		(at 119.38 88.9 180)
+		(at 80.01 88.9 180)
 		(effects
 			(font
@@
 	(hierarchical_label "CHARGER_PG"
 		(shape input)
-		(at 119.38 86.36 180)
+		(at 80.01 86.36 180)
 		(effects
 			(font
@@
 	(hierarchical_label "CHARGER_STAT"
 		(shape input)
-		(at 119.38 83.82 180)
+		(at 80.01 83.82 180)
 		(effects
 			(font
@@
 	(hierarchical_label "CHARGER_INT"
 		(shape input)
-		(at 119.38 93.98 180)
+		(at 80.01 93.98 180)
 		(effects
 			(font
@@
 	(hierarchical_label "POWER_CYCLE"
 		(shape input)
-		(at 78.74 147.32 180)
+		(at 78.74 156.21 180)
 		(effects
 			(font
@@
 	(symbol
 		(lib_id "My Libraries:PUMH10,115")
-		(at 95.25 116.84 270)
+		(at 95.25 125.73 270)
 		(unit 1)
 		(exclude_from_sim no)
@@
 		(fields_autoplaced yes)
 		(property "Reference" "U10"
-			(at 94.0083 120.65 90)
+			(at 94.0083 129.54 90)
 			(effects
 				(font
@@
 		)
 		(property "Value" "PUMH10,115"
-			(at 94.0083 123.19 90)
+			(at 94.0083 132.08 90)
 			(effects
 				(font
@@
 		)
 		(property "Footprint" "Package_TO_SOT_SMD:SOT-363_SC-70-6"
-			(at 95.25 116.84 0)
+			(at 95.25 125.73 0)
 			(effects
 				(font
@@
 		)
 		(property "Datasheet" "https://assets.nexperia.com/documents/data-sheet/PUMH10.pdf"
-			(at 95.25 116.84 0)
+			(at 95.25 125.73 0)
 			(effects
 				(font
@@
 		)
 		(property "Description" "Dual NPN Transistor with internal resistors SOT-363"
-			(at 95.25 116.84 0)
+			(at 95.25 125.73 0)
 			(effects
 				(font
@@
 	(symbol
 		(lib_id "power:+3.3V")
-		(at 95.25 101.6 0)
+		(at 95.25 110.49 0)
 		(unit 1)
 		(exclude_from_sim no)
@@
 		(dnp no)
 		(property "Reference" "#PWR068"
-			(at 95.25 105.41 0)
+			(at 95.25 114.3 0)
 			(effects
 				(font
@@
 		)
 		(property "Value" "+3V3"
-			(at 95.25 97.79 0)
+			(at 95.25 106.68 0)
 			(effects
 				(font
@@
 		)
 		(property "Footprint" ""
-			(at 95.25 101.6 0)
+			(at 95.25 110.49 0)
 			(effects
 				(font
@@
 		)
 		(property "Datasheet" ""
-			(at 95.25 101.6 0)
+			(at 95.25 110.49 0)
 			(effects
 				(font
@@
 		)
 		(property "Description" "Power symbol creates a global label with name \"+3.3V\""
-			(at 95.25 101.6 0)
+			(at 95.25 110.49 0)
 			(effects
 				(font
@@
 	(symbol
 		(lib_id "power:+3.3V")
-		(at 95.25 132.08 0)
+		(at 95.25 140.97 0)
 		(unit 1)
 		(exclude_from_sim no)
@@
 		(dnp no)
 		(property "Reference" "#PWR069"
-			(at 95.25 135.89 0)
+			(at 95.25 144.78 0)
 			(effects
 				(font
@@
 		)
 		(property "Value" "+3V3"
-			(at 95.25 128.27 0)
+			(at 95.25 137.16 0)
 			(effects
 				(font
@@
 		)
 		(property "Footprint" ""
-			(at 95.25 132.08 0)
+			(at 95.25 140.97 0)
 			(effects
 				(font
@@
 		)
 		(property "Datasheet" ""
-			(at 95.25 132.08 0)
+			(at 95.25 140.97 0)
 			(effects
 				(font
@@
 		)
 		(property "Description" "Power symbol creates a global label with name \"+3.3V\""
-			(at 95.25 132.08 0)
+			(at 95.25 140.97 0)
 			(effects
 				(font
@@
 	(symbol
 		(lib_id "My Libraries:PUMH10,115")
-		(at 95.25 147.32 270)
+		(at 95.25 156.21 270)
 		(unit 2)
 		(exclude_from_sim no)
@@
 		(fields_autoplaced yes)
 		(property "Reference" "U10"
-			(at 94.0083 151.13 90)
+			(at 94.0083 160.02 90)
 			(effects
 				(font
@@
 		)
 		(property "Value" "PUMH10,115"
-			(at 94.0083 153.67 90)
+			(at 94.0083 162.56 90)
 			(effects
 				(font
@@
 		)
 		(property "Footprint" "Package_TO_SOT_SMD:SOT-363_SC-70-6"
-			(at 95.25 147.32 0)
+			(at 95.25 156.21 0)
 			(effects
 				(font
@@
 		)
 		(property "Datasheet" "https://assets.nexperia.com/documents/data-sheet/PUMH10.pdf"
-			(at 95.25 147.32 0)
+			(at 95.25 156.21 0)
 			(effects
 				(font
@@
 		)
 		(property "Description" "Dual NPN Transistor with internal resistors SOT-363"
-			(at 95.25 147.32 0)
-			(effects
-				(font
+			(at 95.25 156.21 0)
+			(effects
+				(font
