File: tracker/gsm.kicad_sch (KiCad schematic)
At the start: 22 parts, among them J2 SIM_Card, M1 BG96, Q1 SSM6N7002KFU, U3 74LVC244APW,118, U4 AP22800HB-7, U5 DF5A6.8JE,LM

Commit message: save
Parts:
- added J5: Conn_Coaxial, Connector_Coaxial:U.FL_Molex_MCRF_73412-0110_Vertical, symbol Connector:Conn_Coaxial
Connections:
- net GND: now also J5.2 (Ext)
- net GSM_LINE_BUF_EN: now also U3.1 (~{1OE}); no longer U3. (~{1OE})
- net SIM_CLK: now also RN1.3 (R3.1); no longer RN1.1 (R1.1)
- net SIM_RST: now also RN1.1 (R1.1); no longer RN1.3 (R3.1)
- net at J2.3 (CLK), U5.3 (IO2): now also RN1.6 (R3.2); no longer RN1.8 (R1.2)
- net at J2.2 (RST), U5.4 (IO3): now also RN1.8 (R1.2); no longer RN1.6 (R3.2)
- net ANT_GNSS: now reaches AE1.1 (A), M1.49 (ANT_GNSS)
- net ANT_MAIN: now reaches M1.60 (ANT_MAIN)
- net ANT_MAIN: now also J5.1 (In)
Changed lines of the file:
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@@
 		)
 	)
+	(label "ANT_MAIN"
+		(at 290.83 91.44 0)
+		(effects
+			(font
+				(size 1.27 1.27)
+			)
+			(justify left bottom)
+		)
+	)
 	(label "SIM_VCC"
 		(at 284.48 137.16 180)
@@
 		)
 	)
+	(label "ANT_GNSS"
+		(at 292.1 106.68 0)
+		(effects
+			(font
+				(size 1.27 1.27)
+			)
+			(justify left bottom)
+		)
+	)
 	(label "+VBAT_GSM"
 		(at 248.92 50.8 180)
@@
 			)
 		)
-		(pin ""
+		(pin "1"
 		)
 		(pin "10"
@@
 		(dnp no)
 		(property "Reference" "M1"
-			(at 264.16 97.79 0)
+			(at 263.144 97.79 0)
 			(effects
 				(font
@@
 	(symbol
 		(lib_id "Device:R_Pack04_Split")
-		(at 303.53 142.24 270)
+		(at 303.53 139.7 270)
 		(unit 1)
 		(exclude_from_sim no)
@@
 		(dnp no)
 		(property "Reference" "RN1"
-			(at 302.26 134.62 90)
+			(at 302.26 132.08 90)
 			(effects
 				(font
@@
 		)
 		(property "Value" "22R"
-			(at 303.53 139.7 90)
+			(at 303.53 137.16 90)
 			(effects
 				(font
@@
 		)
 		(property "Footprint" "Resistor_SMD:R_Array_Concave_4x0603"
-			(at 303.53 140.208 90)
+			(at 303.53 137.668 90)
 			(effects
 				(font
@@
 		)
 		(property "Datasheet" "~"
-			(at 303.53 142.24 0)
+			(at 303.53 139.7 0)
 			(effects
 				(font
@@
 		)
 		(property "Description" "4 resistor network, parallel topology, split"
-			(at 303.53 142.24 0)
+			(at 303.53 139.7 0)
 			(effects
 				(font
@@
 	)
 	(symbol
+		(lib_id "power:GND")
+		(at 312.42 96.52 0)
+		(unit 1)
+		(exclude_from_sim no)
+		(in_bom yes)
+		(on_board yes)
+		(dnp no)
+		(property "Reference" "#PWR073"
+			(at 312.42 102.87 0)
+			(effects
+				(font
+					(size 1.27 1.27)
+				)
+				(hide yes)
+			)
+		)
+		(property "Value" "GND"
+			(at 312.42 100.33 0)
+			(effects
+				(font
+					(size 1.27 1.27)
+				)
+			)
+		)
+		(property "Footprint" ""
+			(at 312.42 96.52 0)
+			(effects
+				(font
+					(size 1.27 1.27)
+				)
+				(hide yes)
+			)
+		)
+		(property "Datasheet" ""
+			(at 312.42 96.52 0)
+			(effects
+				(font
+					(size 1.27 1.27)
+				)
+				(hide yes)
+			)
+		)
+		(property "Description" "Power symbol creates a global label with name \"GND\" , ground"
+			(at 312.42 96.52 0)
+			(effects
+				(font
+					(size 1.27 1.27)
+				)
+				(hide yes)
+			)
+		)
+		(pin "1"
+		)
+		(instances
+			(project "tracker"
+				(path "/4f1d18f5-7d2b-4d0b-8633-b1619d53124c/0c625b57-2ba8-40e9-b547-0ed0363dd1ec"
+					(reference "#PWR073")
+					(unit 1)
+				)
+			)
+		)
+	)
+	(symbol
 		(lib_id "Device:R_Pack04_Split")
-		(at 303.53 139.7 270)
+		(at 303.53 142.24 270)
 		(unit 3)
 		(exclude_from_sim no)
@@
 		(fields_autoplaced yes)
 		(property "Reference" "RN1"
-			(at 303.53 134.62 90)
+			(at 303.53 137.16 90)
 			(effects
 				(font
@@
 		)
 		(property "Value" "22R"
-			(at 303.53 137.16 90)
+			(at 303.53 139.7 90)
 			(effects
 				(font
@@
 		)
 		(property "Footprint" "Resistor_SMD:R_Array_Concave_4x0603"
-			(at 303.53 137.668 90)
+			(at 303.53 140.208 90)
 			(effects
 				(font
@@
 		)
 		(property "Datasheet" "~"
-			(at 303.53 139.7 0)
+			(at 303.53 142.24 0)
 			(effects
 				(font
@@
 		)
 		(property "Description" "4 resistor network, parallel topology, split"
-			(at 303.53 139.7 0)
+			(at 303.53 142.24 0)
 			(effects
 				(font
@@
 					(unit 1)
 				)
+			)
+		)
+	)
+	(symbol
+		(lib_id "Connector:Conn_Coaxial")
+		(at 312.42 91.44 0)
+		(unit 1)
+		(exclude_from_sim no)
+		(in_bom yes)
+		(on_board yes)
+		(dnp no)
+		(fields_autoplaced yes)
+		(property "Reference" "J5"
+			(at 316.23 90.4631 0)
+			(effects
+				(font
+					(size 1.27 1.27)
+				)
+				(justify left)
+			)
+		)
+		(property "Value" "Conn_Coaxial"
+			(at 316.23 93.0031 0)
+			(effects
+				(font
+					(size 1.27 1.27)
+				)
+				(justify left)
+			)
+		)
+		(property "Footprint" "Connector_Coaxial:U.FL_Molex_MCRF_73412-0110_Vertical"
+			(at 312.42 91.44 0)
+			(effects
+				(font
+					(size 1.27 1.27)
+				)
+				(hide yes)
+			)
+		)
+		(property "Datasheet" "~"
+			(at 312.42 91.44 0)
+			(effects
+				(font
+					(size 1.27 1.27)
+				)
+				(hide yes)
+			)
+		)
+		(property "Description" "coaxial connector (BNC, SMA, SMB, SMC, Cinch/RCA, LEMO, ...)"
+			(at 312.42 91.44 0)
+			(effects
+				(font
+					(size 1.27 1.27)
+				)
+				(hide yes)
+			)
+		)
+		(pin "2"
+		)
+		(pin "1"
+		)
+		(instances
+			(project ""
+				(path "/4f1d18f5-7d2b-4d0b-8633-b1619d53124c/0c625b57-2ba8-40e9-b547-0ed0363dd1ec"
+					(reference "J5")
+					(unit 1)
+				)

Commit message: save project
Parts:
- removed C17, C19: 1u, Capacitor_SMD:C_0402_1005Metric, symbol Device:C_Small
- C12, C20, C21: footprint Capacitor_SMD:C_0402_1005Metric -> Capacitor_SMD:C_0603_1608Metric
Other:
- moved on the sheet: C15, C16

Commit message: save
Connections:
- no-connect marks 26 -> 29
Changed lines of the file:
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@@
+	)
+	(no_connect
+		(at 215.9 119.38)
 	)
 	(no_connect
@@
 	(no_connect
 		(at 226.06 106.68)
+	)
+	(no_connect
+		(at 205.74 165.1)
 	)
 	(no_connect
@@
 	)
 	(no_connect
+		(at 215.9 121.92)
+	)
+	(no_connect

Commit message: edits
Parts:
- removed C12: 0.1u, Capacitor_SMD:C_0603_1608Metric, symbol Device:C_Small
- removed Q1: SSM6N7002KFU, Package_TO_SOT_SMD:SOT-363_SC-70-6, symbol Device:Q_Dual_NMOS_S1G1D2S2G2D1
- removed U3: 74LVC244APW,118, Package_SO:TSSOP-20_4.4x6.5mm_P0.65mm, symbol My Libraries:74LVC244APW,118
- added C38, C43: 0.1u, Capacitor_SMD:C_0603_1608Metric, symbol Device:C_Small
- added U11: PUMH10,115, Package_TO_SOT_SMD:SOT-363_SC-70-6, symbol My Libraries:PUMH10,115
- added U3: NXB0108PW, Package_SO:TSSOP-20_4.4x6.5mm_P0.65mm, symbol My Libraries:NXB0108PW
Connections:
- net +2V8: now also C43.1, U3.2 (VCCA)
- net +3V3: now also C38.1, U3.19 (VCCB)
- net AP_RDY: now also U3.3 (A2)
- net DTR: now also U3.4 (A3)
- net GND: now also C38.2, C43.2, U11.1, U11.4, U3.11 (GND)
- net GPS_RX: now also U3.12 (B8)
- net GPS_TX: now also U3.14 (B6)
- net GSM_AP_READY: now also U3.18 (B2)
- net GSM_DTR: now also U3.17 (B3)
- net GSM_LINE_BUF_EN: now also U3.10 (OE)
- net GSM_PWRKEY: now also U11.5
- net GSM_RESET: now also U11.2
- net GSM_RI: now also U3.13 (B7)
- net GSM_RX: now also U3.16 (B4)
- net GSM_STATUS: now also U3.20 (B1)
- net GSM_TX: now also U3.15 (B5)
- net PWRKEY: now also U11.3
- net RESET: now also U11.6
- net RI: now also U3.8 (A7)
- net RXD: now also U3.5 (A4)
- net STATUS: now also U3.1 (A1)
- net TXD: now also U3.6 (A5)
- net U3_RXD: now also U3.9 (A8)
- net U3_TXD: now also U3.7 (A6)
- no-connect marks 29 -> 28
Other:
- note removed: "GSM to MCU Signals"
- note removed: "MCU to GSM Signals"

Commit message: edits
Parts:
- removed U5: DF5A6.8JE,LM, Package_TO_SOT_SMD:Diodes_SOT-553, symbol My Libraries:DF5A6.8JE,LM
- added U12: DF6A6.8FUT, Package_TO_SOT_SMD:SOT-363_SC-70-6, symbol My Libraries:DF6A6.8FUT
Connections:
- net GND: now also U12.3 (GND), U12.6 (GND)
- net SIM_VCC: now also U12.4 (IO3)
- net at J2.7 (I/O), RN1.7 (R2.2): now also U12.2 (IO2)
- net at J2.3 (CLK), RN1.6 (R3.2): now also U12.1 (IO1)
- net at J2.2 (RST), RN1.8 (R1.2): now also U12.5 (IO4)
Changed lines of the file:
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@@
-	)
-	(junction
-		(at 322.58 137.16)
-		(diameter 0.9144)
-		(color 0 0 0 0)
 	)
 	(junction
@@
 	)
 	(junction
+		(at 314.96 142.24)
+		(diameter 0)
+		(color 0 0 0 0)
+	)
+	(junction
 		(at 121.92 50.8)
 		(diameter 0.9144)
@@
 	)
 	(junction
+		(at 320.04 137.16)
+		(diameter 0)
+		(color 0 0 0 0)
+	)
+	(junction
 		(at 208.28 109.22)
 		(diameter 0.9144)
@@
 	)
 	(junction
+		(at 317.5 161.29)
+		(diameter 0)
+		(color 0 0 0 0)
+	)
+	(junction
 		(at 248.92 99.06)
+		(diameter 0)
+		(color 0 0 0 0)
+	)
+	(junction
+		(at 322.58 139.7)
 		(diameter 0)
 		(color 0 0 0 0)
@@
 	)
 	(junction
-		(at 320.04 139.7)
-		(diameter 0.9144)
-		(color 0 0 0 0)
-	)
-	(junction
 		(at 231.14 50.8)
 		(diameter 0)
@@
 	)
 	(junction
-		(at 314.96 144.78)
-		(diameter 0.9144)
-		(color 0 0 0 0)
-	)
-	(junction
-		(at 317.5 142.24)
-		(diameter 0.9144)
+		(at 317.5 144.78)
+		(diameter 0)
 		(color 0 0 0 0)
 	)
@@
 	(wire
 		(pts
-			(xy 317.5 142.24) (xy 317.5 149.86)
-		)
-		(stroke
-			(width 0)
-			(type solid)
-		)
-	)
-	(wire
-		(pts
 			(xy 205.74 142.24) (xy 226.06 142.24)
 		)
@@
 	(wire
 		(pts
+			(xy 320.04 160.02) (xy 320.04 161.29)
+		)
+		(stroke
+			(width 0)
+			(type default)
+		)
+	)
+	(wire
+		(pts
 			(xy 157.48 50.8) (xy 157.48 55.88)
 		)
@@
 	(wire
 		(pts
-			(xy 307.34 139.7) (xy 320.04 139.7)
-		)
-		(stroke
-			(width 0)
-			(type solid)
-		)
-	)
-	(wire
-		(pts
 			(xy 208.28 109.22) (xy 226.06 109.22)
 		)
@@
 	(wire
 		(pts
-			(xy 320.04 139.7) (xy 340.36 139.7)
+			(xy 307.34 139.7) (xy 322.58 139.7)
 		)
 		(stroke
@@
 	(wire
 		(pts
+			(xy 317.5 161.29) (xy 320.04 161.29)
+		)
+		(stroke
+			(width 0)
+			(type default)
+		)
+	)
+	(wire
+		(pts
 			(xy 105.41 120.65) (xy 105.41 134.62)
 		)
@@
 	(wire
 		(pts
-			(xy 314.96 144.78) (xy 314.96 149.86)
+			(xy 322.58 139.7) (xy 340.36 139.7)
 		)
 		(stroke
@@
 	(wire
 		(pts
-			(xy 317.5 142.24) (xy 340.36 142.24)
+			(xy 307.34 142.24) (xy 314.96 142.24)
 		)
 		(stroke
@@
 	(wire
 		(pts
-			(xy 271.78 137.16) (xy 322.58 137.16)
-		)
-		(stroke
-			(width 0)
-			(type solid)
-		)
-	)
-	(wire
-		(pts
-			(xy 322.58 137.16) (xy 325.12 137.16)
+			(xy 271.78 137.16) (xy 320.04 137.16)
+		)
+		(stroke
+			(width 0)
+			(type solid)
+		)
+	)
+	(wire
+		(pts
+			(xy 320.04 137.16) (xy 325.12 137.16)
 		)
 		(stroke
@@
 	(wire
 		(pts
-			(xy 322.58 137.16) (xy 322.58 149.86)
-		)
-		(stroke
-			(width 0)
-			(type solid)
-		)
-	)
-	(wire
-		(pts
 			(xy 205.74 132.08) (xy 226.06 132.08)
 		)
@@
 	(wire
 		(pts
+			(xy 317.5 144.78) (xy 317.5 149.86)
+		)
+		(stroke
+			(width 0)
+			(type default)
+		)
+	)
+	(wire
+		(pts
 			(xy 144.78 58.42) (xy 149.86 58.42)
 		)
@@
 	(wire
 		(pts
+			(xy 317.5 161.29) (xy 317.5 162.56)
+		)
+		(stroke
+			(width 0)
+			(type solid)
+		)
+	)
+	(wire
+		(pts
 			(xy 271.78 144.78) (xy 299.72 144.78)
 		)
@@
 	(wire
 		(pts
-			(xy 314.96 144.78) (xy 332.74 144.78)
-		)
-		(stroke
-			(width 0)
-			(type solid)
-		)
-	)
-	(wire
-		(pts
-			(xy 307.34 144.78) (xy 314.96 144.78)
+			(xy 307.34 144.78) (xy 317.5 144.78)
 		)
 		(stroke
@@
 	(wire
 		(pts
+			(xy 314.96 142.24) (xy 340.36 142.24)
+		)
+		(stroke
+			(width 0)
+			(type solid)
+		)
+	)
+	(wire
+		(pts
 			(xy 344.17 106.68) (xy 344.17 92.71)
 		)
@@
 	(wire
 		(pts
-			(xy 307.34 142.24) (xy 317.5 142.24)
-		)
-		(stroke
-			(width 0)
-			(type solid)
-		)
-	)
-	(wire
-		(pts
 			(xy 105.41 142.24) (xy 116.84 142.24)
 		)
@@
 	(wire
 		(pts
+			(xy 320.04 137.16) (xy 320.04 149.86)
+		)
+		(stroke
+			(width 0)
+			(type default)
+		)
+	)
+	(wire
+		(pts
 			(xy 105.41 152.4) (xy 116.84 152.4)
 		)
@@
 	(wire
 		(pts
+			(xy 317.5 144.78) (xy 332.74 144.78)
+		)
+		(stroke
+			(width 0)
+			(type solid)
+		)
+	)
+	(wire
+		(pts
 			(xy 105.41 119.38) (xy 105.41 120.65)
 		)
@@
 	(wire
 		(pts
-			(xy 317.5 160.02) (xy 317.5 162.56)
+			(xy 317.5 160.02) (xy 317.5 161.29)
 		)
 		(stroke
@@
 	(wire
 		(pts
+			(xy 322.58 139.7) (xy 322.58 149.86)
+		)
+		(stroke
+			(width 0)
+			(type default)
+		)
+	)
+	(wire
+		(pts
 			(xy 81.28 246.38) (xy 88.9 246.38)
 		)
@@
 	(wire
 		(pts
-			(xy 320.04 139.7) (xy 320.04 149.86)
-		)
-		(stroke
-			(width 0)
-			(type solid)
-		)
-	)
-	(wire
-		(pts
 			(xy 85.09 119.38) (xy 85.09 120.65)
 		)
@@
 			(width 0)
 			(type solid)
+		)
+	)
+	(wire
+		(pts
+			(xy 314.96 142.24) (xy 314.96 149.86)
+		)
+		(stroke
+			(width 0)
+			(type default)
 		)
 	)
@@
 	)
 	(symbol
-		(lib_id "My Libraries:DF5A6.8JE,LM")
+		(lib_id "My Libraries:DF6A6.8FUT")
 		(at 317.5 154.94 0)
 		(unit 1)
@@
 		(on_board yes)
 		(dnp no)
-		(property "Reference" "U5"
-			(at 326.39 154.3049 0)
+		(fields_autoplaced yes)
+		(property "Reference" "U12"
+			(at 326.39 153.6699 0)
 			(effects
 				(font
@@
 			)
 		)
-		(property "Value" "DF5A6.8JE,LM"
-			(at 318.77 159.3849 0)
+		(property "Value" "DF6A6.8FUT"
+			(at 326.39 156.2099 0)
 			(effects
 				(font
@@
 			)
 		)
-		(property "Footprint" "Package_TO_SOT_SMD:Diodes_SOT-553"
-			(at 320.04 144.78 0)
+		(property "Footprint" "Package_TO_SOT_SMD:SOT-363_SC-70-6"
+			(at 317.5 154.94 0)
 			(effects
 				(font
@@
 			)
 		)
-		(property "Datasheet" ""
-			(at 261.62 142.24 0)
+		(property "Datasheet" "https://www.onsemi.com/download/data-sheet/pdf/df6a6.8fut1-d.pdf"
+			(at 317.5 154.94 0)
 			(effects
 				(font
@@
 			)
 		)
-		(property "Description" "ESD Suppressor, 4 Channel, 5V 6.4V 45pF"
+		(property "Description" "Quad TVS array SC−88 5V"
 			(at 317.5 154.94 0)
 			(effects
@@
 			)
 		)
+		(pin "5"
+		)
 		(pin "2"
 		)
@@
 		(pin "4"
 		)
-		(pin "5"
+		(pin "6"
 		)
 		(instances
-			(project "BK4000TG_V3"
-				(path "/12391f46-36fb-49a8-aa55-7542601826a6/c3fd325a-0513-427d-85da-0b3fb6542889"
-					(reference "U4")
+			(project ""
+				(path "/4f1d18f5-7d2b-4d0b-8633-b1619d53124c/0c625b57-2ba8-40e9-b547-0ed0363dd1ec"
+					(reference "U12")
 					(unit 1)
 				)
-			)
-			(project "BK4000TG_V3"
-				(path "/4f1d18f5-7d2b-4d0b-8633-b1619d53124c/0c625b57-2ba8-40e9-b547-0ed0363dd1ec"
-					(reference "U5")
-					(unit 1)
-				)

Commit message: save
Parts:
- renumbered C38 to C13, C11 to C14, C43 to C15, C13 to C16, C14 to C17, C15 to C18, C18 to C19, C16 to C20, C20 to C21, C21 to C22, C22 to C23, J5 to J4, J2 to J5, R3 to R7, U11 to U3, U3 to U4, U4 to U5, U12 to U6

Commit message: edit silkscreen
Parts:
- C14, C16, C17, C23: footprint Capacitor_SMD:C_0402_1005Metric -> Capacitor_SMD:C_0603_1608Metric
Changed lines of the file:
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@@
 			)
 		)
-		(property "Footprint" "Capacitor_SMD:C_0402_1005Metric"
+		(property "Footprint" "Capacitor_SMD:C_0603_1608Metric"
 			(at 332.74 132.08 0)
 			(effects
@@
 			)
 		)
-		(property "Footprint" "Capacitor_SMD:C_0402_1005Metric"
+		(property "Footprint" "Capacitor_SMD:C_0603_1608Metric"
 			(at 157.48 58.42 0)
 			(effects
@@
 			)
 		)
-		(property "Footprint" "Capacitor_SMD:C_0402_1005Metric"
+		(property "Footprint" "Capacitor_SMD:C_0603_1608Metric"
 			(at 116.84 66.04 0)
 			(effects
@@
 			)
 		)
-		(property "Footprint" "Capacitor_SMD:C_0402_1005Metric"
+		(property "Footprint" "Capacitor_SMD:C_0603_1608Metric"
 			(at 109.22 53.34 0)
 			(effects

Commit message: Edits
Other:
- note added: "Level Translator"
- note added: "Module Power Switch"
- moved on the sheet: AE1, J4, U3A, U3B
Changed lines of the file:
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@@
 	(generator_version "9.0")
 	(paper "A3")
+	(rectangle
+		(start 81.28 35.56)
+		(end 180.34 81.28)
+		(stroke
+			(width 0)
+			(type dash)
+			(color 132 132 132 1)
+		)
+		(fill
+			(type none)
+		)
+	)
+	(rectangle
+		(start 58.42 109.22)
+		(end 142.24 172.72)
+		(stroke
+			(width 0)
+			(type dash)
+			(color 132 132 132 1)
+		)
+		(fill
+			(type none)
+		)
+	)
+	(text "Module Power Switch"
+		(exclude_from_sim no)
+		(at 93.726 79.248 0)
+		(effects
+			(font
+				(size 1.27 1.27)
+			)
+		)
+	)
+	(text "Level Translator"
+		(exclude_from_sim no)
+		(at 132.588 170.942 0)
+		(effects
+			(font
+				(size 1.27 1.27)
+			)
+		)
+	)
 	(junction
 		(at 200.66 50.8)
@@
 	(wire
 		(pts
-			(xy 143.51 246.38) (xy 151.13 246.38)
+			(xy 105.41 222.25) (xy 113.03 222.25)
 		)
 		(stroke
@@
 	(wire
 		(pts
-			(xy 143.51 248.92) (xy 143.51 246.38)
+			(xy 105.41 224.79) (xy 105.41 222.25)
 		)
 		(stroke
@@
 	(wire
 		(pts
-			(xy 81.28 248.92) (xy 81.28 246.38)
+			(xy 106.68 190.5) (xy 106.68 187.96)
 		)
 		(stroke
@@
 	(wire
 		(pts
-			(xy 125.73 254) (xy 128.27 254)
+			(xy 87.63 229.87) (xy 90.17 229.87)
 		)
 		(stroke
@@
 	(wire
 		(pts
-			(xy 60.96 254) (xy 66.04 254)
+			(xy 86.36 195.58) (xy 91.44 195.58)
 		)
 		(stroke
@@
 	(wire
 		(pts
-			(xy 271.78 104.14) (xy 287.02 104.14)
+			(xy 271.78 104.14) (xy 285.75 104.14)
 		)
 		(stroke
@@
 	(wire
 		(pts
-			(xy 287.02 91.44) (xy 307.34 91.44)
+			(xy 285.75 76.2) (xy 306.07 76.2)
 		)
 		(stroke
@@
 	(wire
 		(pts
-			(xy 287.02 104.14) (xy 287.02 91.44)
+			(xy 285.75 104.14) (xy 285.75 76.2)
 		)
 		(stroke
@@
 	(wire
 		(pts
-			(xy 344.17 106.68) (xy 344.17 92.71)
+			(xy 311.15 106.68) (xy 311.15 101.6)
 		)
 		(stroke
@@
 	(wire
 		(pts
-			(xy 271.78 106.68) (xy 344.17 106.68)
+			(xy 271.78 106.68) (xy 311.15 106.68)
 		)
 		(stroke
@@
 	(wire
 		(pts
-			(xy 81.28 246.38) (xy 88.9 246.38)
+			(xy 106.68 187.96) (xy 114.3 187.96)
 		)
 		(stroke
@@
 	)
 	(label "PWRKEY"
-		(at 151.13 246.38 180)
+		(at 113.03 222.25 180)
 		(effects
 			(font
@@
 	)
 	(label "ANT_MAIN"
-		(at 290.83 91.44 0)
+		(at 289.56 76.2 0)
 		(effects
 			(font
@@
 	)
 	(label "RESET"
-		(at 88.9 246.38 180)
+		(at 114.3 187.96 180)
 		(effects
 			(font
@@
 	(hierarchical_label "GSM_RESET"
 		(shape input)
-		(at 60.96 254 180)
+		(at 86.36 195.58 180)
 		(effects
 			(font
@@
 	(hierarchical_label "GSM_PWRKEY"
 		(shape input)
-		(at 125.73 254 180)
+		(at 87.63 229.87 180)
 		(effects
 			(font
@@
 	(symbol
 		(lib_id "My Libraries:PUMH10,115")
-		(at 143.51 254 0)
+		(at 105.41 229.87 0)
 		(unit 2)
 		(exclude_from_sim no)
@@
 		(fields_autoplaced yes)
 		(property "Reference" "U3"
-			(at 146.05 253.9716 0)
+			(at 107.95 229.8416 0)
 			(effects
 				(font
@@
 		)
 		(property "Value" "PUMH10,115"
-			(at 146.05 256.5116 0)
+			(at 107.95 232.3816 0)
 			(effects
 				(font
@@
 		)
 		(property "Footprint" "Package_TO_SOT_SMD:SOT-363_SC-70-6"
-			(at 143.51 254 0)
+			(at 105.41 229.87 0)
 			(effects
 				(font
@@
 		)
 		(property "Datasheet" "https://assets.nexperia.com/documents/data-sheet/PUMH10.pdf"
-			(at 143.51 254 0)
+			(at 105.41 229.87 0)
 			(effects
 				(font
@@
 		)
 		(property "Description" "Dual NPN Transistor with internal resistors SOT-363"
-			(at 143.51 254 0)
+			(at 105.41 229.87 0)
 			(effects
 				(font
@@
 	(symbol
 		(lib_id "My Libraries:PUMH10,115")
-		(at 81.28 254 0)
+		(at 106.68 195.58 0)
 		(unit 1)
 		(exclude_from_sim no)
@@
 		(fields_autoplaced yes)
 		(property "Reference" "U3"
-			(at 83.82 253.9716 0)
+			(at 109.22 195.5516 0)
 			(effects
 				(font
@@
 		)
 		(property "Value" "PUMH10,115"
-			(at 83.82 256.5116 0)
+			(at 109.22 198.0916 0)
 			(effects
 				(font
@@
 		)
 		(property "Footprint" "Package_TO_SOT_SMD:SOT-363_SC-70-6"
-			(at 81.28 254 0)
+			(at 106.68 195.58 0)
 			(effects
 				(font
@@
 		)
 		(property "Datasheet" "https://assets.nexperia.com/documents/data-sheet/PUMH10.pdf"
-			(at 81.28 254 0)
+			(at 106.68 195.58 0)
 			(effects
 				(font
@@
 		)
 		(property "Description" "Dual NPN Transistor with internal resistors SOT-363"
-			(at 81.28 254 0)
+			(at 106.68 195.58 0)
 			(effects
 				(font
@@
 	(symbol
 		(lib_id "power:GND")
-		(at 143.51 261.62 0)
+		(at 105.41 237.49 0)
 		(unit 1)
 		(exclude_from_sim no)
@@
 		(dnp no)
 		(property "Reference" "#PWR042"
-			(at 143.51 267.97 0)
+			(at 105.41 243.84 0)
 			(effects
 				(font
@@
 		)
 		(property "Value" "GND"
-			(at 143.51 265.938 0)
+			(at 105.41 241.808 0)
 			(effects
 				(font
@@
 		)
 		(property "Footprint" ""
-			(at 143.51 261.62 0)
+			(at 105.41 237.49 0)
 			(effects
 				(font
@@
 		)
 		(property "Datasheet" ""
-			(at 143.51 261.62 0)
+			(at 105.41 237.49 0)
 			(effects
 				(font
@@
 		)
 		(property "Description" "Power symbol creates a global label with name \"GND\" , ground"
-			(at 143.51 261.62 0)
+			(at 105.41 237.49 0)
 			(effects
 				(font
@@
 	(symbol
 		(lib_id "power:GND")
-		(at 81.28 261.62 0)
+		(at 106.68 203.2 0)
 		(unit 1)
 		(exclude_from_sim no)
@@
 		(dnp no)
 		(property "Reference" "#PWR033"
-			(at 81.28 267.97 0)
+			(at 106.68 209.55 0)
 			(effects
 				(font
@@
 		)
 		(property "Value" "GND"
-			(at 81.28 265.43 0)
+			(at 106.68 207.01 0)
 			(effects
 				(font
@@
 		)
 		(property "Footprint" ""
-			(at 81.28 261.62 0)
+			(at 106.68 203.2 0)
 			(effects
 				(font
@@
 		)
 		(property "Datasheet" ""
-			(at 81.28 261.62 0)
+			(at 106.68 203.2 0)
 			(effects
 				(font
@@
 		)
 		(property "Description" "Power symbol creates a global label with name \"GND\" , ground"
-			(at 81.28 261.62 0)
+			(at 106.68 203.2 0)
 			(effects
 				(font
@@
 	(symbol
 		(lib_id "power:GND")
-		(at 312.42 96.52 0)
+		(at 311.15 81.28 0)
 		(unit 1)
 		(exclude_from_sim no)
@@
 		(dnp no)
 		(property "Reference" "#PWR053"
-			(at 312.42 102.87 0)
+			(at 311.15 87.63 0)
 			(effects
 				(font
@@
 		)
 		(property "Value" "GND"
-			(at 312.42 100.33 0)
+			(at 311.15 85.09 0)
 			(effects
 				(font
@@
 		)
 		(property "Footprint" ""
-			(at 312.42 96.52 0)
+			(at 311.15 81.28 0)
 			(effects
 				(font
@@
 		)
 		(property "Datasheet" ""
-			(at 312.42 96.52 0)
+			(at 311.15 81.28 0)
 			(effects
 				(font
@@
 		)
 		(property "Description" "Power symbol creates a global label with name \"GND\" , ground"
-			(at 312.42 96.52 0)
+			(at 311.15 81.28 0)
 			(effects
 				(font
@@
 	(symbol
 		(lib_id "Device:Antenna")
-		(at 344.17 87.63 0)
+		(at 311.15 96.52 0)
 		(unit 1)
 		(exclude_from_sim no)
@@
 		(fields_autoplaced yes)
 		(property "Reference" "AE1"
-			(at 346.71 86.9949 0)
+			(at 313.69 95.8849 0)
 			(effects
 				(font
@@
 		)
 		(property "Value" "Antenna"
-			(at 346.71 89.5349 0)
+			(at 313.69 98.4249 0)
 			(effects
 				(font
@@
 		)
 		(property "Footprint" "My Footprints:APAE1575R1820ABDC1"
-			(at 344.17 87.63 0)
+			(at 311.15 96.52 0)
 			(effects
 				(font
@@
 		)
 		(property "Datasheet" "~"
-			(at 344.17 87.63 0)
+			(at 311.15 96.52 0)
 			(effects
 				(font
@@
 		)
 		(property "Description" "Antenna"
-			(at 344.17 87.63 0)
+			(at 311.15 96.52 0)
 			(effects
 				(font
@@
 	(symbol
 		(lib_id "Connector:Conn_Coaxial")
-		(at 312.42 91.44 0)
+		(at 311.15 76.2 0)
 		(unit 1)
 		(exclude_from_sim no)
@@
 		(fields_autoplaced yes)
 		(property "Reference" "J4"
-			(at 316.23 90.4631 0)
+			(at 314.96 75.2231 0)
 			(effects
 				(font
@@
 		)
 		(property "Value" "Conn_Coaxial"
-			(at 316.23 93.0031 0)
+			(at 314.96 77.7631 0)
 			(effects
 				(font
@@
 		)
 		(property "Footprint" "Connector_Coaxial:U.FL_Molex_MCRF_73412-0110_Vertical"
-			(at 312.42 91.44 0)
+			(at 311.15 76.2 0)
 			(effects
 				(font
@@
 		)
 		(property "Datasheet" "~"
-			(at 312.42 91.44 0)
+			(at 311.15 76.2 0)
 			(effects
 				(font
@@
 		)
 		(property "Description" "coaxial connector (BNC, SMA, SMB, SMC, Cinch/RCA, LEMO, ...)"
-			(at 312.42 91.44 0)
+			(at 311.15 76.2 0)
 			(effects
 				(font
