File: tracker/gsm.kicad_sch (KiCad schematic)
At the start: 22 parts, among them J2 SIM_Card, M1 BG96, Q1 SSM6N7002KFU, U3 74LVC244APW,118, U4 AP22800HB-7, U5 DF5A6.8JE,LM

Commit message: first version
Parts:
- removed C12: 0.1u, Capacitor_SMD:C_0402_1005Metric, symbol Device:C_Small
- removed C17, C19: 1u, Capacitor_SMD:C_0402_1005Metric, symbol Device:C_Small
- removed Q1: SSM6N7002KFU, Package_TO_SOT_SMD:SOT-363_SC-70-6, symbol Device:Q_Dual_NMOS_S1G1D2S2G2D1
- removed U3: 74LVC244APW,118, Package_SO:TSSOP-20_4.4x6.5mm_P0.65mm, symbol My Libraries:74LVC244APW,118
- removed U5: DF5A6.8JE,LM, Package_TO_SOT_SMD:Diodes_SOT-553, symbol My Libraries:DF5A6.8JE,LM
- added C13, C15: 0.1u, Capacitor_SMD:C_0603_1608Metric, symbol Device:C_Small
- added J4: Conn_Coaxial, Connector_Coaxial:U.FL_Molex_MCRF_73412-0110_Vertical, symbol Connector:Conn_Coaxial
- added U3: PUMH10,115, Package_TO_SOT_SMD:SOT-363_SC-70-6, symbol My Libraries:PUMH10,115
- added U4: NXB0108PW, Package_SO:TSSOP-20_4.4x6.5mm_P0.65mm, symbol My Libraries:NXB0108PW
- added U6: DF6A6.8FUT, Package_TO_SOT_SMD:SOT-363_SC-70-6, symbol My Libraries:DF6A6.8FUT
- C14: renamed from C11; footprint Capacitor_SMD:C_0402_1005Metric -> Capacitor_SMD:C_0603_1608Metric
- C16: renamed from C13; footprint Capacitor_SMD:C_0402_1005Metric -> Capacitor_SMD:C_0603_1608Metric
- C17: renamed from C14; footprint Capacitor_SMD:C_0402_1005Metric -> Capacitor_SMD:C_0603_1608Metric
- C21: renamed from C20; footprint Capacitor_SMD:C_0402_1005Metric -> Capacitor_SMD:C_0603_1608Metric
- C22: renamed from C21; footprint Capacitor_SMD:C_0402_1005Metric -> Capacitor_SMD:C_0603_1608Metric
- C23: renamed from C22; footprint Capacitor_SMD:C_0402_1005Metric -> Capacitor_SMD:C_0603_1608Metric
- renumbered C15 to C18, C18 to C19, C16 to C20, J2 to J5, R3 to R7, U4 to U5
Connections:
- net +2V8: now also C15.1, U4.2 (VCCA)
- net +3V3: now also C13.1, U4.19 (VCCB)
- net AP_RDY: now also U4.3 (A2)
- net DTR: now also U4.4 (A3)
- net GND: now also C13.2, C15.2, J4.2 (Ext), U3.1, U3.4, U4.11 (GND), U6.3 (GND), U6.6 (GND)
- net GPS_RX: now also U4.12 (B8)
- net GPS_TX: now also U4.14 (B6)
- net GSM_AP_READY: now also U4.18 (B2)
- net GSM_DTR: now also U4.17 (B3)
- net GSM_LINE_BUF_EN: now also U4.10 (OE)
- net GSM_PWRKEY: now also U3.5
- net GSM_RESET: now also U3.2
- net GSM_RI: now also U4.13 (B7)
- net GSM_RX: now also U4.16 (B4)
- net GSM_STATUS: now also U4.20 (B1)
- net GSM_TX: now also U4.15 (B5)
- net PWRKEY: now also U3.3
- net RESET: now also U3.6
- net RI: now also U4.8 (A7)
- net RXD: now also U4.5 (A4)
- net SIM_CLK: now also RN1.3 (R3.1); no longer RN1.1 (R1.1)
- net SIM_RST: now also RN1.1 (R1.1); no longer RN1.3 (R3.1)
- net SIM_VCC: now also U6.4 (IO3)
- net STATUS: now also U4.1 (A1)
- net TXD: now also U4.6 (A5)
- net U3_RXD: now also U4.9 (A8)
- net U3_TXD: now also U4.7 (A6)
- net at J5.7 (I/O), RN1.7 (R2.2): now also U6.2 (IO2)
- net at J5.3 (CLK): now also RN1.6 (R3.2), U6.1 (IO1); no longer RN1.8 (R1.2)
- net at J5.2 (RST): now also RN1.8 (R1.2), U6.5 (IO4); no longer RN1.6 (R3.2)
- net ANT_GNSS: now reaches AE1.1 (A), M1.49 (ANT_GNSS)
- net ANT_MAIN: now reaches M1.60 (ANT_MAIN)
- net ANT_MAIN: now also J4.1 (In)
- no-connect marks 26 -> 28
Other:
- note added: "Level Translator"
- note added: "Module Power Switch"
- note removed: "GSM to MCU Signals"
- note removed: "MCU to GSM Signals"
- moved on the sheet: AE1, C18, C20
