File: tracker/mcu.kicad_sch (KiCad schematic)
At the start: 17 parts, among them J1 Conn_01x10, U1 STM32U545CEUx, U2 GD25QxxxEY, Y1 32.768KHz, Y2 8MHz

Commit message: save
Parts:
- removed J1: Conn_01x10, Connector:Tag-Connect_TC2050-IDC-NL_2x05_P1.27mm_Vertical, symbol Connector_Generic:Conn_01x10
- removed Y1: 32.768KHz, Crystal:Crystal_SMD_SeikoEpson_MC146-4Pin_6.7x1.5mm, symbol Device:Crystal_Small
- added J1: Conn_01x05, Connector_JST:JST_PH_B5B-PH-SM4-TB_1x05-1MP_P2.00mm_Vertical, symbol Connector_Generic:Conn_01x05
- added Y3: 32.768KHz, Crystal:Crystal_SMD_SeikoEpson_MC146-4Pin_6.7x1.5mm, symbol Device:Crystal_GND23_Small
Connections:
- net +3V3: now also C10.1, U2.8 (VCC), J1.1 (Pin_1)
- net GND: now also J1.5 (Pin_5)
- net GSM_AP_READY: now also U1.45 (PB8)
- net GSM_PWRKEY: now also U1.21 (PB10)
- net GSM_STATUS: now also U1.46 (PB9); no longer U1.29 (PA8)
- net I2C_SCL: now also U1.42 (PB6)
- net I2C_SDA: now also U1.43 (PB7)
- net OCTOSPI1_NCS: now also U1.33 (PA12); no longer U1.14 (PA4)
- net OSC32_IN: now also Y3.1
- net OSC32_OUT: now also Y3.4
- net RESET: now also J1.4 (Pin_4)
- net SWCLK: now also U1.37 (PA14), J1.2 (Pin_2)
- net SWDIO: now also U1.34 (PA13), J1.3 (Pin_3)
- net GSM_RESET: now reaches U1.20 (PB2)
- net GSM_LINE_BUF_EN: now reaches U1.44 (PH3)
- no-connect marks 2 -> 0
Other:
- note removed: "FDCAN1_RX"
- note removed: "FDCAN1_TX"
- moved on the sheet: C8, C9

Commit message: save project
Parts:
- added C17: 4.7u, Capacitor_SMD:C_0603_1608Metric, symbol Device:C_Small
- C10, C5, C6, C7, C8, C9: footprint Capacitor_SMD:C_0402_1005Metric -> Capacitor_SMD:C_0603_1608Metric
Connections:
- net CHARGER_INT: now also U1.38 (PA15)
- net GND: now also C17.2
- net GSM_PWRKEY: now also U1.28 (PB15); no longer U1.21 (PB10)
- net GSM_RESET: now also U1.26 (PB13); no longer U1.20 (PB2)
- net VIN_MEAS: now also U1.20 (PB2)
- net VCAP: now reaches U1.22 (VCAP)
- net VCAP: now also C17.1
Other:
- note added: "ADC1_IN17"
- note removed: "ADC12_IN3"
Changed lines of the file:
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@@
 		)
 	)
-	(text "ADC12_IN3"
+	(text "ADC1_IN17"
 		(exclude_from_sim no)
-		(at 90.17 131.318 0)
+		(at 115.824 138.684 0)
 		(effects
 			(font
@@
 	(wire
 		(pts
+			(xy 195.58 146.05) (xy 210.82 146.05)
+		)
+		(stroke
+			(width 0)
+			(type default)
+		)
+	)
+	(wire
+		(pts
 			(xy 180.34 182.88) (xy 182.88 182.88)
 		)
@@
 	(wire
 		(pts
-			(xy 151.13 138.43) (xy 165.1 138.43)
+			(xy 144.78 153.67) (xy 165.1 153.67)
 		)
 		(stroke
@@
 	(wire
 		(pts
-			(xy 144.78 153.67) (xy 165.1 153.67)
+			(xy 185.42 74.93) (xy 201.93 74.93)
 		)
 		(stroke
@@
 	(wire
 		(pts
-			(xy 185.42 74.93) (xy 201.93 74.93)
+			(xy 149.86 173.99) (xy 165.1 173.99)
 		)
 		(stroke
@@
 	(wire
 		(pts
+			(xy 149.86 180.34) (xy 149.86 179.07)
+		)
+		(stroke
+			(width 0)
+			(type default)
+		)
+	)
+	(wire
+		(pts
 			(xy 331.47 50.8) (xy 350.52 50.8)
 		)
@@
 	(wire
 		(pts
+			(xy 144.78 163.83) (xy 165.1 163.83)
+		)
+		(stroke
+			(width 0)
+			(type default)
+		)
+	)
+	(wire
+		(pts
 			(xy 365.76 74.93) (xy 363.22 74.93)
 		)
@@
 	(wire
 		(pts
-			(xy 106.68 130.81) (xy 125.73 130.81)
+			(xy 132.08 138.43) (xy 165.1 138.43)
 		)
 		(stroke
@@
 	(wire
 		(pts
-			(xy 144.78 158.75) (xy 165.1 158.75)
+			(xy 144.78 168.91) (xy 165.1 168.91)
 		)
 		(stroke
@@
 		)
 	)
+	(label "VCAP"
+		(at 153.67 173.99 0)
+		(fields_autoplaced yes)
+		(effects
+			(font
+				(size 1.27 1.27)
+			)
+			(justify left bottom)
+		)
+		(property "swd" ""
+			(at 153.67 175.26 0)
+			(effects
+				(font
+					(size 1.27 1.27)
+					(italic yes)
+				)
+				(justify left)
+			)
+		)
+	)
 	(label "OSC32_IN"
 		(at 58.42 228.6 180)
@@
 	(hierarchical_label "GSM_RESET"
 		(shape input)
-		(at 151.13 138.43 180)
+		(at 144.78 163.83 180)
 		(effects
 			(font
@@
 	(hierarchical_label "CHARGER_INT"
 		(shape input)
-		(at 233.68 157.48 180)
+		(at 210.82 146.05 0)
 		(effects
 			(font
 				(size 1.27 1.27)
 			)
-			(justify right)
+			(justify left)
 		)
 	)
@@
 	(hierarchical_label "VIN_MEAS"
 		(shape input)
-		(at 106.68 130.81 180)
+		(at 132.08 138.43 180)
 		(effects
 			(font
@@
 	(hierarchical_label "GSM_PWRKEY"
 		(shape input)
-		(at 144.78 158.75 180)
+		(at 144.78 168.91 180)
 		(effects
 			(font
@@
 			)
 		)
-		(property "Footprint" "Capacitor_SMD:C_0402_1005Metric"
+		(property "Footprint" "Capacitor_SMD:C_0603_1608Metric"
 			(at 162.56 77.47 0)
 			(effects
@@
 			)
 		)
-		(property "Footprint" "Capacitor_SMD:C_0402_1005Metric"
+		(property "Footprint" "Capacitor_SMD:C_0603_1608Metric"
 			(at 368.3 36.83 0)
 			(effects
@@
 	(symbol
 		(lib_id "power:GND")
+		(at 149.86 180.34 0)
+		(mirror y)
+		(unit 1)
+		(exclude_from_sim no)
+		(in_bom yes)
+		(on_board yes)
+		(dnp no)
+		(property "Reference" "#PWR033"
+			(at 149.86 186.69 0)
+			(effects
+				(font
+					(size 1.27 1.27)
+				)
+				(hide yes)
+			)
+		)
+		(property "Value" "GND"
+			(at 149.86 184.15 0)
+			(effects
+				(font
+					(size 1.27 1.27)
+				)
+			)
+		)
+		(property "Footprint" ""
+			(at 149.86 180.34 0)
+			(effects
+				(font
+					(size 1.27 1.27)
+				)
+				(hide yes)
+			)
+		)
+		(property "Datasheet" ""
+			(at 149.86 180.34 0)
+			(effects
+				(font
+					(size 1.27 1.27)
+				)
+				(hide yes)
+			)
+		)
+		(property "Description" "Power symbol creates a global label with name \"GND\" , ground"
+			(at 149.86 180.34 0)
+			(effects
+				(font
+					(size 1.27 1.27)
+				)
+				(hide yes)
+			)
+		)
+		(pin "1"
+		)
+		(instances
+			(project "tracker"
+				(path "/4f1d18f5-7d2b-4d0b-8633-b1619d53124c/5edf3f23-50ab-4fd8-9879-f628dc9bcaf7"
+					(reference "#PWR033")
+					(unit 1)
+				)
+			)
+		)
+	)
+	(symbol
+		(lib_id "power:GND")
 		(at 368.3 39.37 0)
 		(mirror y)
@@
 	)
 	(symbol
+		(lib_id "Device:C_Small")
+		(at 149.86 176.53 0)
+		(unit 1)
+		(exclude_from_sim no)
+		(in_bom yes)
+		(on_board yes)
+		(dnp no)
+		(fields_autoplaced yes)
+		(property "Reference" "C17"
+			(at 152.4 175.8949 0)
+			(effects
+				(font
+					(size 1.27 1.27)
+				)
+				(justify left)
+			)
+		)
+		(property "Value" "4.7u"
+			(at 152.4 178.4349 0)
+			(effects
+				(font
+					(size 1.27 1.27)
+				)
+				(justify left)
+			)
+		)
+		(property "Footprint" "Capacitor_SMD:C_0603_1608Metric"
+			(at 149.86 176.53 0)
+			(effects
+				(font
+					(size 1.27 1.27)
+				)
+				(hide yes)
+			)
+		)
+		(property "Datasheet" "~"
+			(at 149.86 176.53 0)
+			(effects
+				(font
+					(size 1.27 1.27)
+				)
+				(hide yes)
+			)
+		)
+		(property "Description" "Unpolarized capacitor, small symbol"
+			(at 149.86 176.53 0)
+			(effects
+				(font
+					(size 1.27 1.27)
+				)
+				(hide yes)
+			)
+		)
+		(pin "1"
+		)
+		(pin "2"
+		)
+		(instances
+			(project "tracker"
+				(path "/4f1d18f5-7d2b-4d0b-8633-b1619d53124c/5edf3f23-50ab-4fd8-9879-f628dc9bcaf7"
+					(reference "C17")
+					(unit 1)
+				)
+			)
+		)
+	)
+	(symbol
 		(lib_id "power:GND")
 		(at 25.4 261.62 0)
@@
 			)
 		)
-		(property "Footprint" "Capacitor_SMD:C_0402_1005Metric"
+		(property "Footprint" "Capacitor_SMD:C_0603_1608Metric"
 			(at 152.4 77.47 0)
 			(effects
@@
 			)
 		)
-		(property "Footprint" "Capacitor_SMD:C_0402_1005Metric"
+		(property "Footprint" "Capacitor_SMD:C_0603_1608Metric"
 			(at 212.09 77.47 0)
 			(effects
@@
 			)
 		)
-		(property "Footprint" "Capacitor_SMD:C_0402_1005Metric"
+		(property "Footprint" "Capacitor_SMD:C_0603_1608Metric"
 			(at 201.93 77.47 0)
 			(effects
@@
 			)
 		)
-		(property "Footprint" "Capacitor_SMD:C_0402_1005Metric"
+		(property "Footprint" "Capacitor_SMD:C_0603_1608Metric"
 			(at 172.72 77.47 0)
 			(effects

Commit message: save project
Connections:
- net CHARGER_INT: now also U1.40 (PB4); no longer U1.38 (PA15)
- net CHARGE_ENABLE: now also U1.39 (PB3)
- net POWER_CYCLE: now also U1.38 (PA15)
Changed lines of the file:
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@@
+	(wire
+		(pts
+			(xy 132.08 143.51) (xy 165.1 143.51)
+		)
+		(stroke
+			(width 0)
+			(type default)
+		)
+	)
 	(wire
 		(pts
@@
 			(width 0)
 			(type solid)
+		)
+	)
+	(wire
+		(pts
+			(xy 132.08 140.97) (xy 165.1 140.97)
+		)
+		(stroke
+			(width 0)
+			(type default)
 		)
 	)
@@
 		)
 	)
-	(hierarchical_label "PA6{slash}ADC_IN6"
-		(shape input)
-		(at 285.75 172.72 180)
+	(hierarchical_label "4_20_RES_EN"
+		(shape input)
+		(at 252.73 182.88 0)
+		(effects
+			(font
+				(size 1.27 1.27)
+			)
+			(justify left)
+		)
+	)
+	(hierarchical_label "GSM_RI"
+		(shape input)
+		(at 215.9 113.03 0)
+		(effects
+			(font
+				(size 1.27 1.27)
+			)
+			(justify left)
+		)
+	)
+	(hierarchical_label "GSM_RESET"
+		(shape input)
+		(at 144.78 163.83 180)
 		(effects
 			(font
@@
 		)
 	)
-	(hierarchical_label "4_20_RES_EN"
-		(shape input)
-		(at 252.73 182.88 0)
+	(hierarchical_label "CHARGER_STAT"
+		(shape input)
+		(at 370.84 115.57 180)
+		(effects
+			(font
+				(size 1.27 1.27)
+			)
+			(justify right)
+		)
+	)
+	(hierarchical_label "CHARGER_INT"
+		(shape input)
+		(at 132.08 143.51 180)
+		(effects
+			(font
+				(size 1.27 1.27)
+			)
+			(justify right)
+		)
+	)
+	(hierarchical_label "LED4_ON"
+		(shape input)
+		(at 69.85 154.94 180)
+		(effects
+			(font
+				(size 1.27 1.27)
+			)
+			(justify right)
+		)
+	)
+	(hierarchical_label "POWER_CYCLE"
+		(shape input)
+		(at 210.82 146.05 0)
 		(effects
 			(font
@@
 		)
 	)
-	(hierarchical_label "GSM_RI"
-		(shape input)
-		(at 215.9 113.03 0)
+	(hierarchical_label "GSM_DTR"
+		(shape input)
+		(at 240.03 115.57 0)
 		(effects
 			(font
@@
 		)
 	)
-	(hierarchical_label "GSM_RESET"
-		(shape input)
-		(at 144.78 163.83 180)
+	(hierarchical_label "I2C_SDA"
+		(shape input)
+		(at 152.4 151.13 180)
 		(effects
 			(font
@@
 		)
 	)
-	(hierarchical_label "CHARGER_STAT"
-		(shape input)
-		(at 370.84 115.57 180)
+	(hierarchical_label "GSM_AP_READY"
+		(shape input)
+		(at 144.78 153.67 180)
 		(effects
 			(font
@@
 		)
 	)
-	(hierarchical_label "CHARGER_INT"
-		(shape input)
-		(at 210.82 146.05 0)
-		(effects
-			(font
-				(size 1.27 1.27)
-			)
-			(justify left)
-		)
-	)
-	(hierarchical_label "LED4_ON"
-		(shape input)
-		(at 69.85 154.94 180)
+	(hierarchical_label "LED2_ON"
+		(shape input)
+		(at 69.85 149.86 180)
 		(effects
 			(font
@@
 		)
 	)
-	(hierarchical_label "POWER_CYCLE"
-		(shape input)
-		(at 330.2 179.07 180)
+	(hierarchical_label "LED1_ON"
+		(shape input)
+		(at 69.85 147.32 180)
 		(effects
 			(font
@@
 		)
 	)
-	(hierarchical_label "GSM_DTR"
-		(shape input)
-		(at 240.03 115.57 0)
-		(effects
-			(font
-				(size 1.27 1.27)
-			)
-			(justify left)
-		)
-	)
-	(hierarchical_label "I2C_SDA"
-		(shape input)
-		(at 152.4 151.13 180)
-		(effects
-			(font
-				(size 1.27 1.27)
-			)
-			(justify right)
-		)
-	)
-	(hierarchical_label "GSM_AP_READY"
-		(shape input)
-		(at 144.78 153.67 180)
-		(effects
-			(font
-				(size 1.27 1.27)
-			)
-			(justify right)
-		)
-	)
-	(hierarchical_label "LED2_ON"
-		(shape input)
-		(at 69.85 149.86 180)
-		(effects
-			(font
-				(size 1.27 1.27)
-			)
-			(justify right)
-		)
-	)
-	(hierarchical_label "LED1_ON"
-		(shape input)
-		(at 69.85 147.32 180)
-		(effects
-			(font
-				(size 1.27 1.27)
-			)
-			(justify right)
-		)
-	)
 	(hierarchical_label "CHARGE_ENABLE"
 		(shape input)
-		(at 331.47 148.59 180)
-		(effects
-			(font
+		(at 132.08 140.97 180)
+		(effects
+			(font

Commit message: save
Connections:
- net CHARGER_STAT: now also U1.41 (PB5)
Changed lines of the file:
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@@
+	(wire
+		(pts
+			(xy 152.4 146.05) (xy 165.1 146.05)
+		)
+		(stroke
+			(width 0)
+			(type default)
+		)
+	)
 	(wire
 		(pts
@@
 	(hierarchical_label "CHARGER_STAT"
 		(shape input)
-		(at 370.84 115.57 180)
-		(effects
-			(font
+		(at 152.4 146.05 180)
+		(effects
+			(font

Commit message: save
Parts:
- added C19: 10u, Capacitor_SMD:C_0805_2012Metric, symbol Device:C_Small
Connections:
- net GND: now also C19.2
- net GSM_DTR: now also U1.25 (PB12)
- net PSU_CTRL: now also U1.32 (PA11)
- net at U1.1 (VBAT): now also C19.1
- net GSM_EN: now reaches U1.14 (PA4)
- no-connect marks 0 -> 7

Commit message: edits
Connections:
- net +3V3: now also C19.1, U1.1 (VBAT)
- net GSM_LINE_BUF_EN: now also U1.46 (PB9); no longer U1.44 (PH3)
- net GSM_STATUS: now also U1.44 (PH3); no longer U1.46 (PB9)
Changed lines of the file:
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@@
+	)
+	(junction
+		(at 157.48 90.17)
+		(diameter 0)
+		(color 0 0 0 0)
 	)
 	(junction
@@
 	(hierarchical_label "GSM_STATUS"
 		(shape input)
-		(at 144.78 156.21 180)
+		(at 149.86 118.11 180)
 		(effects
 			(font
@@
 	(hierarchical_label "GSM_LINE_BUF_EN"
 		(shape input)
-		(at 149.86 118.11 180)
+		(at 144.78 156.21 180)
 		(effects
 			(font
@@
 					(unit 1)
 				)
+			)
+		)
+	)
+	(symbol
+		(lib_id "power:+3.3V")
+		(at 157.48 90.17 0)
+		(mirror y)
+		(unit 1)
+		(exclude_from_sim no)
+		(in_bom yes)
+		(on_board yes)
+		(dnp no)
+		(property "Reference" "#PWR080"
+			(at 157.48 93.98 0)
+			(effects
+				(font
+					(size 1.27 1.27)
+				)
+				(hide yes)
+			)
+		)
+		(property "Value" "+3V3"
+			(at 157.48 86.36 0)
+			(effects
+				(font
+					(size 1.27 1.27)
+				)
+			)
+		)
+		(property "Footprint" ""
+			(at 157.48 90.17 0)
+			(effects
+				(font
+					(size 1.27 1.27)
+				)
+				(hide yes)
+			)
+		)
+		(property "Datasheet" ""
+			(at 157.48 90.17 0)
+			(effects
+				(font
+					(size 1.27 1.27)
+				)
+				(hide yes)
+			)
+		)
+		(property "Description" "Power symbol creates a global label with name \"+3.3V\""
+			(at 157.48 90.17 0)
+			(effects
+				(font
+					(size 1.27 1.27)
+				)
+				(hide yes)
+			)
+		)
+		(pin "1"
+		)
+		(instances
+			(project "tracker"
+				(path "/4f1d18f5-7d2b-4d0b-8633-b1619d53124c/5edf3f23-50ab-4fd8-9879-f628dc9bcaf7"
+					(reference "#PWR080")
+					(unit 1)
+				)

Commit message: save
Parts:
- renumbered C8 to C10, C9 to C11, C10 to C12, C17 to C5, C5 to C6, C19 to C7, C6 to C8, C7 to C9, J1 to J3, R1 to R5, R2 to R6, Y3 to Y1
Connections:
- net ACC_INT1: now reaches U1.29 (PA8)
- no-connect marks 7 -> 6

Commit message: Edits
Other:
- note added: "Crystal Oscillators"
- note added: "FLASH Memory"
- note added: "I2C Pull-up resistors"
- note added: "Programming/Debugging Port"
- moved on the sheet: C1, C10, C11, C12, C2, C3, C4, C5, C6, C7, C8, C9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
