File: tracker/mcu.kicad_sch (KiCad schematic)
At the start: 17 parts, among them J1 Conn_01x10, U1 STM32U545CEUx, U2 GD25QxxxEY, Y1 32.768KHz, Y2 8MHz

Commit message: first version
Parts:
- removed J1: Conn_01x10, Connector:Tag-Connect_TC2050-IDC-NL_2x05_P1.27mm_Vertical, symbol Connector_Generic:Conn_01x10
- removed Y1: 32.768KHz, Crystal:Crystal_SMD_SeikoEpson_MC146-4Pin_6.7x1.5mm, symbol Device:Crystal_Small
- added C5: 4.7u, Capacitor_SMD:C_0603_1608Metric, symbol Device:C_Small
- added C7: 10u, Capacitor_SMD:C_0805_2012Metric, symbol Device:C_Small
- added J3: Conn_01x05, Connector_JST:JST_PH_B5B-PH-SM4-TB_1x05-1MP_P2.00mm_Vertical, symbol Connector_Generic:Conn_01x05
- added Y1: 32.768KHz, Crystal:Crystal_SMD_SeikoEpson_MC146-4Pin_6.7x1.5mm, symbol Device:Crystal_GND23_Small
- C10: renamed from C8; footprint Capacitor_SMD:C_0402_1005Metric -> Capacitor_SMD:C_0603_1608Metric
- C11: renamed from C9; footprint Capacitor_SMD:C_0402_1005Metric -> Capacitor_SMD:C_0603_1608Metric
- C12: renamed from C10; footprint Capacitor_SMD:C_0402_1005Metric -> Capacitor_SMD:C_0603_1608Metric
- C6: renamed from C5; footprint Capacitor_SMD:C_0402_1005Metric -> Capacitor_SMD:C_0603_1608Metric
- C8: renamed from C6; footprint Capacitor_SMD:C_0402_1005Metric -> Capacitor_SMD:C_0603_1608Metric
- C9: renamed from C7; footprint Capacitor_SMD:C_0402_1005Metric -> Capacitor_SMD:C_0603_1608Metric
- renumbered R1 to R5, R2 to R6
Connections:
- net +3V3: now also C12.1, U1.1 (VBAT), U2.8 (VCC), C7.1, J3.1 (Pin_1)
- net CHARGER_INT: now also U1.40 (PB4)
- net CHARGER_STAT: now also U1.41 (PB5)
- net CHARGE_ENABLE: now also U1.39 (PB3)
- net GND: now also C5.2, C7.2, J3.5 (Pin_5)
- net GSM_AP_READY: now also U1.45 (PB8)
- net GSM_DTR: now also U1.25 (PB12)
- net GSM_PWRKEY: now also U1.28 (PB15)
- net GSM_STATUS: now also U1.44 (PH3); no longer U1.29 (PA8)
- net I2C_SCL: now also U1.42 (PB6)
- net I2C_SDA: now also U1.43 (PB7)
- net OCTOSPI1_NCS: now also U1.33 (PA12); no longer U1.14 (PA4)
- net OSC32_IN: now also Y1.1
- net OSC32_OUT: now also Y1.4
- net POWER_CYCLE: now also U1.38 (PA15)
- net PSU_CTRL: now also U1.32 (PA11)
- net RESET: now also J3.4 (Pin_4)
- net SWCLK: now also U1.37 (PA14), J3.2 (Pin_2)
- net SWDIO: now also U1.34 (PA13), J3.3 (Pin_3)
- net VIN_MEAS: now also U1.20 (PB2)
- net VCAP: now reaches U1.22 (VCAP)
- net VCAP: now also C5.1
- net GSM_RESET: now reaches U1.26 (PB13)
- net GSM_LINE_BUF_EN: now reaches U1.46 (PB9)
- new net ACC_INT1: U1.29 (PA8)
- new net GSM_EN: U1.14 (PA4)
- no-connect marks 2 -> 6
Other:
- note added: "ADC1_IN17"
- note added: "Crystal Oscillators"
- note added: "FLASH Memory"
- note added: "I2C Pull-up resistors"
- note added: "Programming/Debugging Port"
- note removed: "ADC12_IN3"
- note removed: "FDCAN1_RX"
- note removed: "FDCAN1_TX"
- moved on the sheet: C1, C10, C11, C12, C2, C3, C4, C6, C8, C9, R5, R6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
