File: tracker/psu.kicad_sch (KiCad schematic)
At the start: 14 parts, among them Q2 SSM6N7002KFU, U6 LMR51430

Commit message: save
Parts:
- removed Q2: SSM6N7002KFU, Package_TO_SOT_SMD:SOT-363_SC-70-6, symbol Device:Q_Dual_NMOS_S1G1D2S2G2D1
- removed R4: 200K, Resistor_SMD:R_0402_1005Metric, symbol Device:R_Small
- added U8: PUMH10,115, Package_TO_SOT_SMD:SOT-363_SC-70-6, symbol My Libraries:PUMH10,115
Connections:
- net +3V3: now also U8.2
- net PSU_CTRL: now also U8.1
- net at R5.2, R6.2, U6.5 (EN): now also U8.6
- net +VIN renamed +VIN_PROTECTED

Commit message: save
Parts:
- renumbered C23 to C24, C24 to C25, C25 to C26, C26 to C27, C27 to C28, C28 to C29, R7 to R10, R8 to R11, R5 to R8, R6 to R9, U8 to U7, U6 to U8
Changed lines of the file:
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@@
 		(on_board yes)
 		(dnp no)
-		(property "Reference" "#PWR045"
+		(property "Reference" "#PWR061"
 			(at 177.8 62.23 0)
 			(effects
@@
 			(project "BK4000TG_V3"
 				(path "/4f1d18f5-7d2b-4d0b-8633-b1619d53124c/0e6bc46e-b05d-4d53-a1b9-fade2e6c2182"
-					(reference "#PWR045")
+					(reference "#PWR061")
 					(unit 1)
 				)
@@
 		(dnp no)
 		(fields_autoplaced yes)
-		(property "Reference" "U6"
+		(property "Reference" "U8"
 			(at 134.62 38.1 0)
 			(effects
@@
 			(project "BK4000TG_V3"
 				(path "/4f1d18f5-7d2b-4d0b-8633-b1619d53124c/0e6bc46e-b05d-4d53-a1b9-fade2e6c2182"
-					(reference "U6")
+					(reference "U8")
 					(unit 1)
 				)
@@
 		(on_board yes)
 		(dnp no)
-		(property "Reference" "R6"
+		(property "Reference" "R9"
 			(at 113.03 60.3249 0)
 			(effects
@@
 			(project "BK4000TG_V3"
 				(path "/4f1d18f5-7d2b-4d0b-8633-b1619d53124c/0e6bc46e-b05d-4d53-a1b9-fade2e6c2182"
-					(reference "R6")
+					(reference "R9")
 					(unit 1)
 				)
@@
 		(dnp no)
 		(fields_autoplaced yes)
-		(property "Reference" "C23"
+		(property "Reference" "C24"
 			(at 86.36 47.6249 0)
 			(effects
@@
 			(project "BK4000TG_V3"
 				(path "/4f1d18f5-7d2b-4d0b-8633-b1619d53124c/0e6bc46e-b05d-4d53-a1b9-fade2e6c2182"
-					(reference "C23")
+					(reference "C24")
 					(unit 1)
 				)
@@
 		(on_board yes)
 		(dnp no)
-		(property "Reference" "#PWR047"
+		(property "Reference" "#PWR063"
 			(at 198.12 80.01 0)
 			(effects
@@
 			(project "BK4000TG_V3"
 				(path "/4f1d18f5-7d2b-4d0b-8633-b1619d53124c/0e6bc46e-b05d-4d53-a1b9-fade2e6c2182"
-					(reference "#PWR047")
+					(reference "#PWR063")
 					(unit 1)
 				)
@@
 		(on_board yes)
 		(dnp no)
-		(property "Reference" "R8"
+		(property "Reference" "R11"
 			(at 200.66 70.612 0)
 			(effects
@@
 			(project "BK4000TG_V3"
 				(path "/4f1d18f5-7d2b-4d0b-8633-b1619d53124c/0e6bc46e-b05d-4d53-a1b9-fade2e6c2182"
-					(reference "R8")
+					(reference "R11")
 					(unit 1)
 				)
@@
 		(on_board yes)
 		(dnp no)
-		(property "Reference" "#PWR043"
+		(property "Reference" "#PWR059"
 			(at 111.76 72.39 0)
 			(effects
@@
 			(project "BK4000TG_V3"
 				(path "/4f1d18f5-7d2b-4d0b-8633-b1619d53124c/0e6bc46e-b05d-4d53-a1b9-fade2e6c2182"
-					(reference "#PWR043")
+					(reference "#PWR059")
 					(unit 1)
 				)
@@
 		(dnp no)
 		(fields_autoplaced yes)
-		(property "Reference" "U8"
+		(property "Reference" "U7"
 			(at 121.9483 101.6 90)
 			(effects
@@
 			(project "tracker"
 				(path "/4f1d18f5-7d2b-4d0b-8633-b1619d53124c/0e6bc46e-b05d-4d53-a1b9-fade2e6c2182"
-					(reference "U8")
+					(reference "U7")
 					(unit 2)
 				)
@@
 		(dnp no)
 		(fields_autoplaced yes)
-		(property "Reference" "#PWR041"
+		(property "Reference" "#PWR057"
 			(at 86.36 86.36 0)
 			(effects
@@
 			(project "tracker"
 				(path "/4f1d18f5-7d2b-4d0b-8633-b1619d53124c/0e6bc46e-b05d-4d53-a1b9-fade2e6c2182"
-					(reference "#PWR041")
+					(reference "#PWR057")
 					(unit 1)
 				)
@@
 		(dnp no)
 		(fields_autoplaced yes)
-		(property "Reference" "C27"
+		(property "Reference" "C28"
 			(at 190.5 52.7049 0)
 			(effects
@@
 			(project "BK4000TG_V3"
 				(path "/4f1d18f5-7d2b-4d0b-8633-b1619d53124c/0e6bc46e-b05d-4d53-a1b9-fade2e6c2182"
-					(reference "C27")
+					(reference "C28")
 					(unit 1)
 				)
@@
 		(on_board yes)
 		(dnp no)
-		(property "Reference" "R5"
+		(property "Reference" "R8"
 			(at 113.03 50.1649 0)
 			(effects
@@
 			(project "BK4000TG_V3"
 				(path "/4f1d18f5-7d2b-4d0b-8633-b1619d53124c/0e6bc46e-b05d-4d53-a1b9-fade2e6c2182"
-					(reference "R5")
+					(reference "R8")
 					(unit 1)
 				)
@@
 		(dnp no)
 		(fields_autoplaced yes)
-		(property "Reference" "C24"
+		(property "Reference" "C25"
 			(at 96.52 47.6249 0)
 			(effects
@@
 			(project "BK4000TG_V3"
 				(path "/4f1d18f5-7d2b-4d0b-8633-b1619d53124c/0e6bc46e-b05d-4d53-a1b9-fade2e6c2182"
-					(reference "C24")
+					(reference "C25")
 					(unit 1)
 				)
@@
 		(on_board yes)
 		(dnp no)
-		(property "Reference" "#PWR042"
+		(property "Reference" "#PWR058"
 			(at 93.98 59.69 0)
 			(effects
@@
 			(project "BK4000TG_V3"
 				(path "/4f1d18f5-7d2b-4d0b-8633-b1619d53124c/0e6bc46e-b05d-4d53-a1b9-fade2e6c2182"
-					(reference "#PWR042")
+					(reference "#PWR058")
 					(unit 1)
 				)
@@
 		(on_board yes)
 		(dnp no)
-		(property "Reference" "C25"
+		(property "Reference" "C26"
 			(at 153.67 43.8149 0)
 			(effects
@@
 			(project "BK4000TG_V3"
 				(path "/4f1d18f5-7d2b-4d0b-8633-b1619d53124c/0e6bc46e-b05d-4d53-a1b9-fade2e6c2182"
-					(reference "C25")
+					(reference "C26")
 					(unit 1)
 				)
@@
 		(dnp no)
 		(fields_autoplaced yes)
-		(property "Reference" "C28"
+		(property "Reference" "C29"
 			(at 210.82 57.7849 0)
 			(effects
@@
 			(project "BK4000TG_V3"
 				(path "/4f1d18f5-7d2b-4d0b-8633-b1619d53124c/0e6bc46e-b05d-4d53-a1b9-fade2e6c2182"
-					(reference "C28")
+					(reference "C29")
 					(unit 1)
 				)
@@
 		(dnp no)
 		(fields_autoplaced yes)
-		(property "Reference" "C26"
+		(property "Reference" "C27"
 			(at 180.34 52.7049 0)
 			(effects
@@
 			(project "BK4000TG_V3"
 				(path "/4f1d18f5-7d2b-4d0b-8633-b1619d53124c/0e6bc46e-b05d-4d53-a1b9-fade2e6c2182"
-					(reference "C26")
+					(reference "C27")
 					(unit 1)
 				)
@@
 		(on_board yes)
 		(dnp no)
-		(property "Reference" "#PWR046"
+		(property "Reference" "#PWR062"
 			(at 187.96 62.23 0)
 			(effects
@@
 			(project "BK4000TG_V3"
 				(path "/4f1d18f5-7d2b-4d0b-8633-b1619d53124c/0e6bc46e-b05d-4d53-a1b9-fade2e6c2182"
-					(reference "#PWR046")
+					(reference "#PWR062")
 					(unit 1)
 				)
@@
 		(dnp no)
 		(fields_autoplaced yes)
-		(property "Reference" "U8"
+		(property "Reference" "U7"
 			(at 85.1183 101.6 90)
 			(effects
@@
 			(project "tracker"
 				(path "/4f1d18f5-7d2b-4d0b-8633-b1619d53124c/0e6bc46e-b05d-4d53-a1b9-fade2e6c2182"
-					(reference "U8")
+					(reference "U7")
 					(unit 1)
 				)
@@
 		(on_board yes)
 		(dnp no)
-		(property "Reference" "#PWR040"
+		(property "Reference" "#PWR056"
 			(at 83.82 59.69 0)
 			(effects
@@
 			(project "BK4000TG_V3"
 				(path "/4f1d18f5-7d2b-4d0b-8633-b1619d53124c/0e6bc46e-b05d-4d53-a1b9-fade2e6c2182"
-					(reference "#PWR040")
+					(reference "#PWR056")
 					(unit 1)
 				)
@@
 		(on_board yes)
 		(dnp no)
-		(property "Reference" "R7"
+		(property "Reference" "R10"
 			(at 199.39 57.15 0)
 			(effects
@@
 			(project "BK4000TG_V3"
 				(path "/4f1d18f5-7d2b-4d0b-8633-b1619d53124c/0e6bc46e-b05d-4d53-a1b9-fade2e6c2182"
-					(reference "R7")
+					(reference "R10")
 					(unit 1)
 				)
@@
 		(dnp no)
 		(fields_autoplaced yes)
-		(property "Reference" "#FLG01"
+		(property "Reference" "#FLG05"
 			(at 76.2 41.275 0)
 			(effects
@@
 			(project "BK4000TG_V3"
 				(path "/4f1d18f5-7d2b-4d0b-8633-b1619d53124c/0e6bc46e-b05d-4d53-a1b9-fade2e6c2182"
-					(reference "#FLG01")
+					(reference "#FLG05")
 					(unit 1)
 				)
@@
 		(on_board yes)
 		(dnp no)
-		(property "Reference" "#PWR044"
+		(property "Reference" "#PWR060"
 			(at 134.62 63.5 0)
 			(effects
@@
 			(project "BK4000TG_V3"
 				(path "/4f1d18f5-7d2b-4d0b-8633-b1619d53124c/0e6bc46e-b05d-4d53-a1b9-fade2e6c2182"
-					(reference "#PWR044")
-					(unit 1)
-				)
+					(reference "#PWR060")
+					(unit 1)
+				)

Commit message: Edits
Changed lines of the file:
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@@
 	(text "Freq: 500KHz"
 		(exclude_from_sim no)
-		(at 139.192 118.872 0)
+		(at 129.794 69.596 0)
 		(effects
 			(font
