File: tracker/psu.kicad_sch (KiCad schematic)
At the start: 14 parts, among them Q2 SSM6N7002KFU, U6 LMR51430

Commit message: first version
Parts:
- removed Q2: SSM6N7002KFU, Package_TO_SOT_SMD:SOT-363_SC-70-6, symbol Device:Q_Dual_NMOS_S1G1D2S2G2D1
- removed R4: 200K, Resistor_SMD:R_0402_1005Metric, symbol Device:R_Small
- added U7: PUMH10,115, Package_TO_SOT_SMD:SOT-363_SC-70-6, symbol My Libraries:PUMH10,115
- renumbered C23 to C24, C24 to C25, C25 to C26, C26 to C27, C27 to C28, C28 to C29, R7 to R10, R8 to R11, R5 to R8, R6 to R9, U6 to U8
Connections:
- net +3V3: now also U7.2
- net PSU_CTRL: now also U7.1
- net at R8.2, R9.2, U8.5 (EN): now also U7.6
- net +VIN renamed +VIN_PROTECTED
