File: tracker/tracker.kicad_sch (KiCad schematic)
At the start: 0 parts

Commit message: save
Parts:
- added D1: 12V, Diode_SMD:D_SOD-323, symbol Device:D_Zener_Small_Filled
- added J3, J4: Conn_01x01, My Footprints:pad_smd_1.5x3, symbol Connector_Generic:Conn_01x01
- added Q2: DMP2008UFG, Package_SON:Diodes_PowerDI3333-8, symbol My Libraries:DMP2008UFG
- added R13: 10K, Resistor_SMD:R_0603_1608Metric, symbol Device:R_Small
- added R4: 220K, Resistor_SMD:R_0603_1608Metric, symbol Device:R_Small
Connections:
- new net: D1.2 (A), Q2.4 (G), R13.1, R4.2
- new net +VIN: J3.1 (Pin_1), Q2.5 (D)
- new net GND: J4.1 (Pin_1), R13.2
- new net psu/+VIN_PROTECTED: D1.1 (K), Q2.1 (S), Q2.2 (S), Q2.3 (S), R4.1
Other:
- sheet battery charger ports: added I2C_SCL, I2C_SDA; removed BAT_LEVEL, CHARGER_SCL, CHARGER_SDA
- sheet gsm ports: added none; removed GSM_EN
- sheet low_voltage_psu ports: added LV_PSU_EN; removed none
- sheet mcu ports: added CHARGER_INT, CHARGER_PG, CHARGER_STAT, CHARGE_ENABLE, GSM_LINE_BUF_EN, GSM_RESET, I2C_SCL, I2C_SDA, POWER_CYCLE; removed none
- sheet psu ports: added +VIN_PROTECTED; removed +VIN

Commit message: save project
Parts:
- added R16: 10K, Resistor_SMD:R_0603_1608Metric, symbol Device:R_Small
- added R17: 150K, Resistor_SMD:R_0603_1608Metric, symbol Device:R_Small
Connections:
- net GND: now also R16.2
- net psu/+VIN_PROTECTED: now also R17.1
- new net mcu/VIN_MEAS: R16.1, R17.2
Other:
- sheet mcu ports: added VIN_MEAS; removed none
- moved on the sheet: D1, Q2, R13, R4

Commit message: save
Other:
- sheet gsm ports: added GSM_EN; removed none
- sheet mcu ports: added GSM_EN; removed CHARGER_PG

Commit message: save
Parts:
- renumbered J3 to J1, J4 to J2, Q2 to Q1, R13 to R1, R4 to R2, R17 to R3, R16 to R4
Other:
- added sheet accelerometer (accelerometer.kicad_sch)
- sheet mcu ports: added ACC_INT1; removed none

Commit message: Edits
Other:
- note added: "Polarity Protection"
- note added: "Voltage Measurement"
