File: tracker/tracker.kicad_sch (KiCad schematic)
At the start: 0 parts

Commit message: first version
Parts:
- added D1: 12V, Diode_SMD:D_SOD-323, symbol Device:D_Zener_Small_Filled
- added J1, J2: Conn_01x01, My Footprints:pad_smd_1.5x3, symbol Connector_Generic:Conn_01x01
- added Q1: DMP2008UFG, Package_SON:Diodes_PowerDI3333-8, symbol My Libraries:DMP2008UFG
- added R1, R4: 10K, Resistor_SMD:R_0603_1608Metric, symbol Device:R_Small
- added R2: 220K, Resistor_SMD:R_0603_1608Metric, symbol Device:R_Small
- added R3: 150K, Resistor_SMD:R_0603_1608Metric, symbol Device:R_Small
Connections:
- new net: D1.2 (A), Q1.4 (G), R1.1, R2.2
- new net +VIN: J1.1 (Pin_1), Q1.5 (D)
- new net GND: J2.1 (Pin_1), R1.2, R4.2
- new net mcu/VIN_MEAS: R3.2, R4.1
- new net psu/+VIN_PROTECTED: D1.1 (K), Q1.1 (S), Q1.2 (S), Q1.3 (S), R2.1, R3.1
Other:
- added sheet accelerometer (accelerometer.kicad_sch)
- sheet battery charger ports: added I2C_SCL, I2C_SDA; removed BAT_LEVEL, CHARGER_SCL, CHARGER_SDA
- sheet low_voltage_psu ports: added LV_PSU_EN; removed none
- sheet mcu ports: added ACC_INT1, CHARGER_INT, CHARGER_STAT, CHARGE_ENABLE, GSM_EN, GSM_LINE_BUF_EN, GSM_RESET, I2C_SCL, I2C_SDA, POWER_CYCLE, VIN_MEAS; removed none
- sheet psu ports: added +VIN_PROTECTED; removed +VIN
- note added: "Polarity Protection"
- note added: "Voltage Measurement"
