File: tracker/accelerometer.kicad_sch (KiCad schematic)
At the start: 2 parts, among them U10 MC3479

Commit message: first version
Parts:
- C42: renamed from C51; footprint Capacitor_SMD:C_0402_1005Metric -> Capacitor_SMD:C_0603_1608Metric
- renumbered U10 to U12
Connections:
- net ACC_SCL renamed I2C_SCL
- net ACC_SDA renamed I2C_SDA
Changed lines of the file:
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@@
 		)
 	)
-	(hierarchical_label "ACC_SCL"
+	(hierarchical_label "I2C_SCL"
 		(shape input)
 		(at 129.54 78.74 180)
@@
 		)
 	)
-	(hierarchical_label "ACC_SDA"
+	(hierarchical_label "I2C_SDA"
 		(shape input)
 		(at 129.54 86.36 180)
@@
 	)
 	(symbol
-		(lib_id "power:+3.3V")
+		(lib_id "power:+3V3")
 		(at 157.48 55.88 0)
 		(unit 1)
@@
 		(dnp no)
 		(fields_autoplaced yes)
-		(property "Reference" "#PWR0107"
+		(property "Reference" "#PWR083"
 			(at 157.48 59.69 0)
 			(effects
@@
 		)
 		(property "Value" "+3V3"
-			(at 157.48 52.07 0)
+			(at 157.48 50.8 0)
 			(effects
 				(font
@@
 			)
 		)
-		(property "Description" "Power symbol creates a global label with name \"+3.3V\""
+		(property "Description" "Power symbol creates a global label with name \"+3V3\""
 			(at 157.48 55.88 0)
 			(effects
@@
 		)
 		(instances
-			(project "BK4000TG_V3"
-				(path "/12391f46-36fb-49a8-aa55-7542601826a6/691b4bcc-a256-4f68-a61f-dc2fa4faca7e"
-					(reference "#PWR0107")
+			(project "tracker"
+				(path "/4f1d18f5-7d2b-4d0b-8633-b1619d53124c/68d45962-0216-4a92-bb54-eaef1d80ce8b"
+					(reference "#PWR083")
 					(unit 1)
 				)
@@
 		(on_board yes)
 		(dnp no)
-		(property "Reference" "#PWR0109"
+		(property "Reference" "#PWR085"
 			(at 165.1 72.39 0)
 			(effects
@@
 				)
 			)
+			(project "BK4000TG_V3"
+				(path "/4f1d18f5-7d2b-4d0b-8633-b1619d53124c/68d45962-0216-4a92-bb54-eaef1d80ce8b"
+					(reference "#PWR085")
+					(unit 1)
+				)
+			)
 		)
 	)
@@
 		(on_board yes)
 		(dnp no)
-		(property "Reference" "U10"
+		(property "Reference" "U12"
 			(at 144.78 69.85 0)
 			(effects
@@
 				)
 			)
+			(project "BK4000TG_V3"
+				(path "/4f1d18f5-7d2b-4d0b-8633-b1619d53124c/68d45962-0216-4a92-bb54-eaef1d80ce8b"
+					(reference "U12")
+					(unit 1)
+				)
+			)
 		)
 	)
@@
 		(on_board yes)
 		(dnp no)
-		(property "Reference" "C51"
+		(property "Reference" "C42"
 			(at 167.005 62.2299 0)
 			(effects
@@
 			)
 		)
-		(property "Footprint" "Capacitor_SMD:C_0402_1005Metric"
+		(property "Footprint" "Capacitor_SMD:C_0603_1608Metric"
 			(at 165.1 62.23 0)
 			(effects
@@
 				)
 			)
+			(project "BK4000TG_V3"
+				(path "/4f1d18f5-7d2b-4d0b-8633-b1619d53124c/68d45962-0216-4a92-bb54-eaef1d80ce8b"
+					(reference "C42")
+					(unit 1)
+				)
+			)
 		)
 	)
@@
 		(on_board yes)
 		(dnp no)
-		(property "Reference" "#PWR0108"
+		(property "Reference" "#PWR084"
 			(at 157.48 102.87 0)
 			(effects
@@
 					(unit 1)
 				)
+			)
+			(project "BK4000TG_V3"
+				(path "/4f1d18f5-7d2b-4d0b-8633-b1619d53124c/68d45962-0216-4a92-bb54-eaef1d80ce8b"
+					(reference "#PWR084")
+					(unit 1)
+				)
