File: design_files/accelerometer.kicad_sch (KiCad schematic)
At the start: 2 parts, among them U12 MC3479

Commit message: Edits
Connections:
- net +3V3: now also U12.2 (CSN), U12.3 (DOUT_A6)
- net I2C_SDA: now also U12.4 (DIN_SDA); no longer U12.2 (CSN)
- no-connect marks 3 -> 1
Other:
- note added: "7-bit Device ID: 0x6C (0b1101100) 8-bit Address - Write: 0xD8 8-bit Address - Read: 0xD9"
Changed lines of the file:
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@@
 	(generator_version "9.0")
 	(paper "A4")
+	(rectangle
+		(start 86.36 96.52)
+		(end 132.08 109.22)
+		(stroke
+			(width 0)
+			(type dash)
+			(color 132 132 132 1)
+		)
+		(fill
+			(type none)
+		)
+	)
+	(text "7-bit Device ID: 0x6C (0b1101100)\n8-bit Address - Write: 0xD8\n8-bit Address - Read: 0xD9"
+		(exclude_from_sim no)
+		(at 88.392 103.632 0)
+		(effects
+			(font
+				(size 1.5 1.5)
+			)
+			(justify left)
+		)
+	)
 	(junction
 		(at 157.48 93.98)
@@
 	)
 	(junction
+		(at 137.16 83.82)
+		(diameter 0)
+		(color 0 0 0 0)
+	)
+	(junction
+		(at 157.48 64.77)
+		(diameter 0)
+		(color 0 0 0 0)
+	)
+	(junction
 		(at 157.48 58.42)
 		(diameter 0.9144)
@@
 	)
 	(no_connect
-		(at 142.24 81.28)
-	)
-	(no_connect
-		(at 142.24 83.82)
-	)
-	(no_connect
 		(at 172.72 83.82)
 	)
@@
 	(wire
 		(pts
+			(xy 137.16 86.36) (xy 137.16 83.82)
+		)
+		(stroke
+			(width 0)
+			(type default)
+		)
+	)
+	(wire
+		(pts
+			(xy 137.16 83.82) (xy 142.24 83.82)
+		)
+		(stroke
+			(width 0)
+			(type default)
+		)
+	)
+	(wire
+		(pts
+			(xy 142.24 86.36) (xy 137.16 86.36)
+		)
+		(stroke
+			(width 0)
+			(type default)
+		)
+	)
+	(wire
+		(pts
 			(xy 165.1 64.77) (xy 165.1 66.04)
 		)
@@
 	(wire
 		(pts
-			(xy 157.48 71.12) (xy 157.48 58.42)
+			(xy 157.48 71.12) (xy 157.48 64.77)
 		)
 		(stroke
@@
 	(wire
 		(pts
+			(xy 137.16 83.82) (xy 137.16 64.77)
+		)
+		(stroke
+			(width 0)
+			(type default)
+		)
+	)
+	(wire
+		(pts
 			(xy 157.48 93.98) (xy 157.48 96.52)
 		)
@@
 	(wire
 		(pts
+			(xy 157.48 64.77) (xy 157.48 58.42)
+		)
+		(stroke
+			(width 0)
+			(type solid)
+		)
+	)
+	(wire
+		(pts
 			(xy 172.72 81.28) (xy 180.34 81.28)
 		)
@@
 	(wire
 		(pts
-			(xy 129.54 86.36) (xy 142.24 86.36)
-		)
-		(stroke
-			(width 0)
-			(type solid)
+			(xy 129.54 81.28) (xy 142.24 81.28)
+		)
+		(stroke
+			(width 0)
+			(type solid)
+		)
+	)
+	(wire
+		(pts
+			(xy 137.16 64.77) (xy 157.48 64.77)
+		)
+		(stroke
+			(width 0)
+			(type default)
 		)
 	)
@@
 	(hierarchical_label "I2C_SDA"
 		(shape input)
-		(at 129.54 86.36 180)
-		(effects
-			(font
+		(at 129.54 81.28 180)
+		(effects
+			(font
