File: design_files/gsm.kicad_sch (KiCad schematic)
At the start: 22 parts, among them J4 Conn_Coaxial, J5 SIM_Card, M1 BG96, U3 PUMH10,115, U4 NXB0108PW, U5 AP22800HB-7, U6 DF6A6.8FUT

Commit message: First review.
Connections:
- net +GSM_SWITCHED: now also R7.1
- net GND: no longer R7.2
- net at U5.6 (DIS): now also R7.2; no longer R7.1
Other:
- moved on the sheet: C17, R7
Changed lines of the file:
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@@
 	)
 	(junction
-		(at 157.48 50.8)
-		(diameter 0.9144)
-		(color 0 0 0 0)
-	)
-	(junction
 		(at 210.82 50.8)
 		(diameter 0)
@@
 	)
 	(junction
+		(at 158.75 50.8)
+		(diameter 0)
+		(color 0 0 0 0)
+	)
+	(junction
 		(at 231.14 50.8)
 		(diameter 0)
@@
 	)
 	(junction
+		(at 149.86 53.34)
+		(diameter 0)
+		(color 0 0 0 0)
+	)
+	(junction
 		(at 105.41 120.65)
 		(diameter 0)
@@
 	(wire
 		(pts
-			(xy 157.48 50.8) (xy 157.48 55.88)
+			(xy 158.75 50.8) (xy 158.75 55.88)
 		)
 		(stroke
@@
 	(wire
 		(pts
+			(xy 149.86 53.34) (xy 152.4 53.34)
+		)
+		(stroke
+			(width 0)
+			(type solid)
+		)
+	)
+	(wire
+		(pts
 			(xy 87.63 229.87) (xy 90.17 229.87)
 		)
@@
 	(wire
 		(pts
+			(xy 158.75 50.8) (xy 165.1 50.8)
+		)
+		(stroke
+			(width 0)
+			(type solid)
+		)
+	)
+	(wire
+		(pts
 			(xy 271.78 104.14) (xy 285.75 104.14)
 		)
@@
 	(wire
 		(pts
-			(xy 157.48 60.96) (xy 157.48 68.58)
+			(xy 158.75 60.96) (xy 158.75 68.58)
 		)
 		(stroke
@@
 	(wire
 		(pts
-			(xy 144.78 53.34) (xy 152.4 53.34)
+			(xy 144.78 53.34) (xy 149.86 53.34)
 		)
 		(stroke
@@
 	(wire
 		(pts
-			(xy 149.86 63.5) (xy 149.86 68.58)
-		)
-		(stroke
-			(width 0)
-			(type solid)
-		)
-	)
-	(wire
-		(pts
 			(xy 210.82 50.8) (xy 220.98 50.8)
 		)
@@
 	(wire
 		(pts
-			(xy 152.4 50.8) (xy 157.48 50.8)
-		)
-		(stroke
-			(width 0)
-			(type solid)
-		)
-	)
-	(wire
-		(pts
-			(xy 157.48 50.8) (xy 165.1 50.8)
+			(xy 152.4 50.8) (xy 158.75 50.8)
 		)
 		(stroke
@@
 	(symbol
 		(lib_id "power:GND")
-		(at 149.86 68.58 0)
-		(unit 1)
-		(exclude_from_sim no)
-		(in_bom yes)
-		(on_board yes)
-		(dnp no)
-		(property "Reference" "#PWR043"
-			(at 149.86 74.93 0)
-			(effects
-				(font
-					(size 1.27 1.27)
-				)
-				(hide yes)
-			)
-		)
-		(property "Value" "GND"
-			(at 149.86 72.39 0)
-			(effects
-				(font
-					(size 1.27 1.27)
-				)
-			)
-		)
-		(property "Footprint" ""
-			(at 149.86 68.58 0)
-			(effects
-				(font
-					(size 1.27 1.27)
-				)
-				(hide yes)
-			)
-		)
-		(property "Datasheet" ""
-			(at 149.86 68.58 0)
-			(effects
-				(font
-					(size 1.27 1.27)
-				)
-				(hide yes)
-			)
-		)
-		(property "Description" "Power symbol creates a global label with name \"GND\" , ground"
-			(at 149.86 68.58 0)
-			(effects
-				(font
-					(size 1.27 1.27)
-				)
-				(hide yes)
-			)
-		)
-		(pin "1"
-		)
-		(instances
-			(project "BK4000TG_V3"
-				(path "/12391f46-36fb-49a8-aa55-7542601826a6/c3fd325a-0513-427d-85da-0b3fb6542889"
-					(reference "#PWR035")
-					(unit 1)
-				)
-			)
-			(project "BK4000TG_V3"
-				(path "/4f1d18f5-7d2b-4d0b-8633-b1619d53124c/0c625b57-2ba8-40e9-b547-0ed0363dd1ec"
-					(reference "#PWR043")
-					(unit 1)
-				)
-			)
-		)
-	)
-	(symbol
-		(lib_id "power:GND")
 		(at 210.82 55.88 0)
 		(unit 1)
@@
 	(symbol
 		(lib_id "Device:C_Small")
-		(at 157.48 58.42 0)
+		(at 158.75 58.42 0)
 		(unit 1)
 		(exclude_from_sim no)
@@
 		(fields_autoplaced yes)
 		(property "Reference" "C17"
-			(at 160.02 57.7849 0)
+			(at 161.29 57.7849 0)
 			(effects
 				(font
@@
 		)
 		(property "Value" "0.1u"
-			(at 160.02 60.3249 0)
+			(at 161.29 60.3249 0)
 			(effects
 				(font
@@
 		)
 		(property "Footprint" "Capacitor_SMD:C_0603_1608Metric"
-			(at 157.48 58.42 0)
+			(at 158.75 58.42 0)
 			(effects
 				(font
@@
 		)
 		(property "Datasheet" "~"
-			(at 157.48 58.42 0)
+			(at 158.75 58.42 0)
 			(effects
 				(font
@@
 		)
 		(property "Description" "Unpolarized capacitor, small symbol"
-			(at 157.48 58.42 0)
+			(at 158.75 58.42 0)
 			(effects
 				(font
@@
 	(symbol
 		(lib_id "power:GND")
-		(at 157.48 68.58 0)
+		(at 158.75 68.58 0)
 		(unit 1)
 		(exclude_from_sim no)
@@
 		(dnp no)
 		(property "Reference" "#PWR044"
-			(at 157.48 74.93 0)
+			(at 158.75 74.93 0)
 			(effects
 				(font
@@
 		)
 		(property "Value" "GND"
-			(at 157.48 72.39 0)
+			(at 158.75 72.39 0)
 			(effects
 				(font
@@
 		)
 		(property "Footprint" ""
-			(at 157.48 68.58 0)
+			(at 158.75 68.58 0)
 			(effects
 				(font
@@
 		)
 		(property "Datasheet" ""
-			(at 157.48 68.58 0)
+			(at 158.75 68.58 0)
 			(effects
 				(font
@@
 		)
 		(property "Description" "Power symbol creates a global label with name \"GND\" , ground"
-			(at 157.48 68.58 0)
+			(at 158.75 68.58 0)
 			(effects
 				(font
@@
 	(symbol
 		(lib_id "Device:R_Small")
-		(at 149.86 60.96 0)
+		(at 149.86 55.88 0)
 		(unit 1)
 		(exclude_from_sim no)
@@
 		(on_board yes)
 		(dnp no)
-		(fields_autoplaced yes)
 		(property "Reference" "R7"
-			(at 152.4 60.3249 0)
+			(at 151.13 55.372 0)
 			(effects
 				(font
@@
 		)
 		(property "Value" "10K"
-			(at 152.4 62.8649 0)
+			(at 151.13 57.912 0)
 			(effects
 				(font
@@
 		)
 		(property "Footprint" "Resistor_SMD:R_0402_1005Metric"
-			(at 149.86 60.96 0)
+			(at 149.86 55.88 0)
 			(effects
 				(font
@@
 		)
 		(property "Datasheet" "~"
-			(at 149.86 60.96 0)
+			(at 149.86 55.88 0)
 			(effects
 				(font
@@
 		)
 		(property "Description" "Resistor, small symbol"
-			(at 149.86 60.96 0)
+			(at 149.86 55.88 0)
 			(effects
 				(font
