File: R2/design_files/gsm.kicad_sch (KiCad schematic)
At the start: 24 parts, among them J4 Conn_Coaxial, J5 SIM_Card, M1 BG96, U3 PUMH10,115, U4 NXB0108PW, U5 AP22800HB-7, U6 DF6A6.8FUT

Commit message: Refactor code structure for improved readability and maintainability
Parts:
- AE1: footprint My Footprints:APAE1575R1820ABDC1 -> My_Footprints:APAE1575R1820ABDC1
- M1: footprint My Footprints:LGA_BG96 -> My_Footprints:LGA_BG96; symbol My Libraries:BG96 -> My_Libraries:BG96
- U3: symbol My Libraries:PUMH10,115 -> My_Libraries:PUMH10,115
- U4: symbol My Libraries:NXB0108PW -> My_Libraries:NXB0108PW
- U5: footprint My Footprints:UDFN2116-8_Diodes -> My_Footprints:UDFN2116-8_Diodes; symbol My Libraries:AP22800HB-7 -> My_Libraries:AP22800HB-7
- U6: symbol My Libraries:DF6A6.8FUT -> My_Libraries:DF6A6.8FUT
Connections:
- net +VBAT_GSM: now also M1.[32,33] (VBAT_BB), M1.[52,53] (VBAT_RF); no longer M1.32 (VBAT_BB), M1.33 (VBAT_BB), M1.52 (VBAT_RF), M1.53 (VBAT_RF)
- net GND: now also M1.[3,31,48,50,54,55,58,59,61,62,67,68,69,70,71,72,73,74,79,80,81,82,89,90,91,100,101,102] (GND); no longer M1.100 (GND), M1.101 (GND), M1.102 (GND), M1.3 (GND), M1.31 (GND), M1.48 (GND), M1.50 (GND), M1.54 (GND), M1.55 (GND), M1.58 (GND), M1.59 (GND), M1.61 (GND), M1.62 (GND), M1.67 (GND), M1.68 (GND), M1.69 (GND), M1.70 (GND), M1.71 (GND), M1.72 (GND), M1.73 (GND), M1.74 (GND), M1.79 (GND), M1.80 (GND), M1.81 (GND), M1.82 (GND), M1.89 (GND), M1.90 (GND), M1.91 (GND)
