File: R2/design_files/battery_charger.kicad_sch (KiCad schematic)
At the start: 18 parts, among them J6 Conn_01x02, U10 PUMH10,115, U11 BQ25622E

Commit message: Refactor code structure for improved readability and maintainability
Parts:
- added R23: 10K, Resistor_SMD:R_0402_1005Metric, symbol Device:R_Small
- L4: footprint My Footprints:Inductor_TYA252012 -> My_Footprints:Inductor_TYA252012
- U10: symbol My Libraries:PUMH10,115 -> My_Libraries:PUMH10,115
- U11: footprint My Footprints:BQ25622E -> My_Footprints:BQ25622E
Connections:
- net +VSYS: now also R23.1
- net at U10.6, U11.14 (~{CE}): now also R23.2

Commit message: Refactor code structure for improved readability and maintainability
Connections:
- net CHARGER_PG: no longer names the net of U11.3 (~{PG})
- no-connect marks 0 -> 1
