File: R2/design_files/tracker.kicad_pcb (KiCad board)
At the start: 4 copper layers, 49.4 x 53.4 mm, 96 parts, among them J1 Conn_01x01, J2 Conn_01x01, J3 Conn_01x05, J4 Conn_Coaxial, J5 SIM_Card, J6 Conn_01x02, M1 BG96, Q1 DMP2008UFG, U1 STM32U545CEUx, U10 PUMH10,115, U12 MC3479, U13 PUMH10,115, U2 GD25QxxxEY, U3 PUMH10,115, U4 NXB0108PW, U5 AP22800HB-7, U6 DF6A6.8FUT, U7 PUMH10,115, U8 LMR51430, U9 AP61100Z6, Y1 32.768KHz, Y2 8MHz

Commit message: Refactor code structure for improved readability and maintainability
Parts:
- AE1: footprint My Footprints:APAE1575R1820ABDC1 -> My_Footprints:APAE1575R1820ABDC1
- J1, J2: footprint My Footprints:pad_smd_1.5x3 -> My_Footprints:pad_smd_1.5x3
- L3: footprint My Footprints:L_0806_2016Metric_TAIYO_YUDEN_SMD -> My_Footprints:L_0806_2016Metric_TAIYO_YUDEN_SMD
- L4: footprint My Footprints:Inductor_TYA252012 -> My_Footprints:Inductor_TYA252012
- M1: footprint My Footprints:LGA_BG96 -> My_Footprints:LGA_BG96
- U11: footprint My Footprints:BQ25622E -> My_Footprints:BQ25622E
- U5: footprint My Footprints:UDFN2116-8_Diodes -> My_Footprints:UDFN2116-8_Diodes
Changed lines of the file:
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@@
 		)
 	)
-	(footprint "My Footprints:pad_smd_1.5x3"
+	(footprint "My_Footprints:pad_smd_1.5x3"
 		(layer "F.Cu")
 		(at 170.494054 93.25 90)
@@
 		)
 	)
-	(footprint "My Footprints:pad_smd_1.5x3"
+	(footprint "My_Footprints:pad_smd_1.5x3"
 		(layer "F.Cu")
 		(at 168.17 93.24 90)
@@
 		)
 	)
-	(footprint "My Footprints:UDFN2116-8_Diodes"
+	(footprint "My_Footprints:UDFN2116-8_Diodes"
 		(layer "F.Cu")
 		(at 144.155 64.345 -90)
@@
 		)
 	)
-	(footprint "My Footprints:L_0806_2016Metric_TAIYO_YUDEN_SMD"
+	(footprint "My_Footprints:L_0806_2016Metric_TAIYO_YUDEN_SMD"
 		(layer "B.Cu")
 		(at 136.995 90.33 90)
@@
 		)
 	)
-	(footprint "My Footprints:BQ25622E"
+	(footprint "My_Footprints:BQ25622E"
 		(layer "B.Cu")
 		(at 150.095 90.74 90)
@@
 		)
 	)
-	(footprint "My Footprints:LGA_BG96"
+	(footprint "My_Footprints:LGA_BG96"
 		(layer "B.Cu")
 		(at 158.787 62.602 180)
@@
 		)
 	)
-	(footprint "My Footprints:Inductor_TYA252012"
+	(footprint "My_Footprints:Inductor_TYA252012"
 		(layer "B.Cu")
 		(at 151.7626 86.7 90)
@@
 		)
 	)
-	(footprint "My Footprints:APAE1575R1820ABDC1"
+	(footprint "My_Footprints:APAE1575R1820ABDC1"
 		(layer "B.Cu")
 		(at 134.49 54.01 180)

Commit message: Enhance design settings in tracker.kicad_pro
- Added options to disable default application for footprint barcodes, dimensions, fields, shapes, and text.
- Expanded zone settings with additional parameters including border display style, corner radius, fill mode, and thermal relief specifications.
- Introduced new warnings for footprint symbol field mismatches and missing tuning profiles.
- Updated track settings to include options for centered tracks on vias and tuning profile track geometries.
Parts:
- added R23: 10K, Resistor_SMD:R_0402_1005Metric, F.Cu at (151.5, 87.2)
- U11: value ~ -> BQ25622E
Routing:
- net +VSYS: track 2.29 -> 7.10 mm
- net Net-(U11-~{CE}): track 25.5 -> 27.3 mm

Commit message: Refactor code structure for improved readability and maintainability
Parts:
- removed R21: 10K, Resistor_SMD:R_0402_1005Metric
- removed U13: PUMH10,115, Package_TO_SOT_SMD:SOT-363_SC-70-6
- removed Y2: 8MHz, Crystal:Crystal_SMD_0603-4Pin_6.0x3.5mm
- added Y3: 8MHz, Crystal:Crystal_SMD_SeikoEpson_FA238-4Pin_3.2x2.5mm, F.Cu at (146.9, 77.0)
- U11: value BQ25622E -> Untitled_1
- moved R9 2.87 mm to (159.7, 93.4), turned to 0 degrees
- moved C3 2.06 mm to (147.2, 79.8), turned to 0 degrees
- moved C4 2.00 mm to (146.5, 74.2)
- moved RN1 0.16 mm to (150.1, 60.6)
Connections:
- U11 pad 3: /battery charger/CHARGER_PG -> unconnected-(U11-~{PG}-Pad3)
Routing:
- net /battery charger/CHARGER_PG: track 17.8 -> 0.00 mm, vias 1 -> 0
- net Net-(U9-EN): track 5.85 -> 2.54 mm, vias 1 -> 0
- net GND: track 19.4 -> 22.3 mm, vias 317 -> 321
- net /mcu/OSC_OUT: track 9.90 -> 7.20 mm
- net Net-(J5-I/O): track 9.32 -> 12.0 mm
- net Net-(J5-CLK): track 8.95 -> 10.8 mm
- net /gsm/PWRKEY: track 25.4 -> 26.8 mm
- net /gsm/GSM_PWRKEY: track 24.3 -> 25.5 mm
- net /mcu/OSC_IN: track 9.98 -> 9.10 mm
- net +VSYS: track 7.10 -> 6.39 mm
Other:
- board text added: "BK Telematics TraceLink R2"
- board text removed: "BK Telematics TraceLink R1"
