File: R1/design_files/accelerometer.kicad_sch (KiCad schematic)
At the start: 2 parts, among them U12 MC3479

Commit message: Refactor code structure for improved readability and maintainability
Parts:
- U12: symbol My Libraries:MC3479 -> My_Libraries:MC3479
Changed lines of the file:
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@@
 	)
 	(symbol
-		(lib_id "My Libraries:MC3479")
+		(lib_id "My_Libraries:MC3479")
 		(at 157.48 81.28 0)
 		(unit 1)
