File: R1/design_files/battery_charger.kicad_sch (KiCad schematic)
At the start: 18 parts, among them J6 Conn_01x02, U10 PUMH10,115

Commit message: Refactor code structure for improved readability and maintainability
Parts:
- L4: footprint My Footprints:Inductor_TYA252012 -> My_Footprints:Inductor_TYA252012
- U10: symbol My Libraries:PUMH10,115 -> My_Libraries:PUMH10,115
- U11: footprint My Footprints:BQ25622E -> My_Footprints:BQ25622E; symbol My Libraries:BQ25622E -> My_Libraries:BQ25622E
Changed lines of the file:
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@@
 	)
 	(symbol
-		(lib_id "My Libraries:BQ25622E")
+		(lib_id "My_Libraries:BQ25622E")
 		(at 147.32 60.96 0)
 		(unit 1)
@@
 			)
 		)
-		(property "Footprint" "My Footprints:BQ25622E"
+		(property "Footprint" "My_Footprints:BQ25622E"
 			(at 147.32 60.96 0)
 			(effects
@@
 	)
 	(symbol
-		(lib_id "My Libraries:PUMH10,115")
+		(lib_id "My_Libraries:PUMH10,115")
 		(at 95.25 125.73 270)
 		(unit 1)
@@
 			)
 		)
-		(property "Footprint" "My Footprints:Inductor_TYA252012"
+		(property "Footprint" "My_Footprints:Inductor_TYA252012"
 			(at 184.15 43.18 0)
 			(effects
@@
 	)
 	(symbol
-		(lib_id "My Libraries:PUMH10,115")
+		(lib_id "My_Libraries:PUMH10,115")
 		(at 95.25 156.21 270)
 		(unit 2)
