File: R1/design_files/gsm.kicad_sch (KiCad schematic)
At the start: 22 parts, among them J4 Conn_Coaxial, J5 SIM_Card, M1 BG96, U3 PUMH10,115, U4 NXB0108PW, U5 AP22800HB-7, U6 DF6A6.8FUT

Commit message: Refactor code structure for improved readability and maintainability
Parts:
- AE1: footprint My Footprints:APAE1575R1820ABDC1 -> My_Footprints:APAE1575R1820ABDC1
- M1: footprint My Footprints:LGA_BG96 -> My_Footprints:LGA_BG96; symbol My Libraries:BG96 -> My_Libraries:BG96
- U3: symbol My Libraries:PUMH10,115 -> My_Libraries:PUMH10,115
- U4: symbol My Libraries:NXB0108PW -> My_Libraries:NXB0108PW
- U5: footprint My Footprints:UDFN2116-8_Diodes -> My_Footprints:UDFN2116-8_Diodes; symbol My Libraries:AP22800HB-7 -> My_Libraries:AP22800HB-7
- U6: symbol My Libraries:DF6A6.8FUT -> My_Libraries:DF6A6.8FUT
Changed lines of the file:
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@@
 	)
 	(symbol
-		(lib_id "My Libraries:PUMH10,115")
+		(lib_id "My_Libraries:PUMH10,115")
 		(at 105.41 229.87 0)
 		(unit 2)
@@
 	)
 	(symbol
-		(lib_id "My Libraries:DF6A6.8FUT")
+		(lib_id "My_Libraries:DF6A6.8FUT")
 		(at 317.5 154.94 0)
 		(unit 1)
@@
 	)
 	(symbol
-		(lib_id "My Libraries:+2V8")
+		(lib_id "My_Libraries:+2V8")
 		(at 208.28 106.68 0)
 		(unit 1)
@@
 	)
 	(symbol
-		(lib_id "My Libraries:PUMH10,115")
+		(lib_id "My_Libraries:PUMH10,115")
 		(at 106.68 195.58 0)
 		(unit 1)
@@
 	)
 	(symbol
-		(lib_id "My Libraries:+2V8")
+		(lib_id "My_Libraries:+2V8")
 		(at 105.41 119.38 0)
 		(unit 1)
@@
 	)
 	(symbol
-		(lib_id "My Libraries:BG96")
+		(lib_id "My_Libraries:BG96")
 		(at 248.92 124.46 0)
 		(unit 1)
@@
 			)
 		)
-		(property "Footprint" "My Footprints:LGA_BG96"
+		(property "Footprint" "My_Footprints:LGA_BG96"
 			(at 203.2 124.46 0)
 			(effects
@@
 	)
 	(symbol
-		(lib_id "My Libraries:AP22800HB-7")
+		(lib_id "My_Libraries:AP22800HB-7")
 		(at 134.62 55.88 0)
 		(unit 1)
@@
 			)
 		)
-		(property "Footprint" "My Footprints:UDFN2116-8_Diodes"
+		(property "Footprint" "My_Footprints:UDFN2116-8_Diodes"
 			(at 133.35 45.72 0)
 			(effects
@@
 	)
 	(symbol
-		(lib_id "My Libraries:NXB0108PW")
+		(lib_id "My_Libraries:NXB0108PW")
 		(at 95.25 144.78 0)
 		(mirror y)
@@
 	)
 	(symbol
-		(lib_id "My Libraries:+VSYS")
+		(lib_id "My_Libraries:+VSYS")
 		(at 106.68 48.26 0)
 		(unit 1)
@@
 			)
 		)
-		(property "Footprint" "My Footprints:APAE1575R1820ABDC1"
+		(property "Footprint" "My_Footprints:APAE1575R1820ABDC1"
 			(at 311.15 96.52 0)
 			(effects
