File: R1/design_files/low_voltage_psu.kicad_sch (KiCad schematic)
At the start: 7 parts, among them U9 AP61100Z6

Commit message: Refactor code structure for improved readability and maintainability
Parts:
- L3: footprint My Footprints:L_0806_2016Metric_TAIYO_YUDEN_SMD -> My_Footprints:L_0806_2016Metric_TAIYO_YUDEN_SMD
- U9: symbol My Libraries:AP61100Z6 -> My_Libraries:AP61100Z6
Changed lines of the file:
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@@
 	)
 	(symbol
-		(lib_id "My Libraries:AP61100Z6")
+		(lib_id "My_Libraries:AP61100Z6")
 		(at 135.89 71.12 0)
 		(unit 1)
@@
 			)
 		)
-		(property "Footprint" "My Footprints:L_0806_2016Metric_TAIYO_YUDEN_SMD"
+		(property "Footprint" "My_Footprints:L_0806_2016Metric_TAIYO_YUDEN_SMD"
 			(at 149.86 68.58 0)
 			(effects
