File: R1/design_files/psu.kicad_sch (KiCad schematic)
At the start: 13 parts, among them U7 PUMH10,115, U8 LMR51430

Commit message: Refactor code structure for improved readability and maintainability
Parts:
- U7: symbol My Libraries:PUMH10,115 -> My_Libraries:PUMH10,115
Changed lines of the file:
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@@
 	)
 	(symbol
-		(lib_id "My Libraries:PUMH10,115")
+		(lib_id "My_Libraries:PUMH10,115")
 		(at 123.19 97.79 270)
 		(unit 2)
@@
 	)
 	(symbol
-		(lib_id "My Libraries:PUMH10,115")
+		(lib_id "My_Libraries:PUMH10,115")
 		(at 86.36 97.79 270)
 		(unit 1)
