File: R1/design_files/tracker.kicad_pcb (KiCad board)
At the start: 4 copper layers, 49.4 x 53.4 mm, 92 parts, among them J1 Conn_01x01, J2 Conn_01x01, J3 Conn_01x05, J4 Conn_Coaxial, J5 SIM_Card, J6 Conn_01x02, M1 BG96, Q1 DMP2008UFG, U1 STM32U545CEUx, U10 PUMH10,115, U12 MC3479, U2 GD25QxxxEY, U3 PUMH10,115, U4 NXB0108PW, U5 AP22800HB-7, U6 DF6A6.8FUT, U7 PUMH10,115, U8 LMR51430, U9 AP61100Z6, Y1 32.768KHz, Y2 8MHz

Commit message: Refactor code structure for improved readability and maintainability
Parts:
- AE1: footprint My Footprints:APAE1575R1820ABDC1 -> My_Footprints:APAE1575R1820ABDC1
- J1, J2: footprint My Footprints:pad_smd_1.5x3 -> My_Footprints:pad_smd_1.5x3
- L3: footprint My Footprints:L_0806_2016Metric_TAIYO_YUDEN_SMD -> My_Footprints:L_0806_2016Metric_TAIYO_YUDEN_SMD
- L4: footprint My Footprints:Inductor_TYA252012 -> My_Footprints:Inductor_TYA252012
- M1: footprint My Footprints:LGA_BG96 -> My_Footprints:LGA_BG96
- U11: footprint My Footprints:BQ25622E -> My_Footprints:BQ25622E
- U5: footprint My Footprints:UDFN2116-8_Diodes -> My_Footprints:UDFN2116-8_Diodes
Changed lines of the file:
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@@
 		)
 	)
-	(footprint "My Footprints:pad_smd_1.5x3"
+	(footprint "My_Footprints:pad_smd_1.5x3"
 		(layer "F.Cu")
 		(at 170.494054 93.25 90)
@@
 		)
 	)
-	(footprint "My Footprints:pad_smd_1.5x3"
+	(footprint "My_Footprints:pad_smd_1.5x3"
 		(layer "F.Cu")
 		(at 168.17 93.24 90)
@@
 		)
 	)
-	(footprint "My Footprints:UDFN2116-8_Diodes"
+	(footprint "My_Footprints:UDFN2116-8_Diodes"
 		(layer "F.Cu")
 		(at 144.155 64.345 -90)
@@
 		)
 	)
-	(footprint "My Footprints:L_0806_2016Metric_TAIYO_YUDEN_SMD"
+	(footprint "My_Footprints:L_0806_2016Metric_TAIYO_YUDEN_SMD"
 		(layer "B.Cu")
 		(at 135.57 90.28 90)
@@
 		)
 	)
-	(footprint "My Footprints:BQ25622E"
+	(footprint "My_Footprints:BQ25622E"
 		(layer "B.Cu")
 		(at 148.87 90.445 90)
@@
 		)
 	)
-	(footprint "My Footprints:LGA_BG96"
+	(footprint "My_Footprints:LGA_BG96"
 		(layer "B.Cu")
 		(at 158.787 62.602 180)
@@
 		)
 	)
-	(footprint "My Footprints:Inductor_TYA252012"
+	(footprint "My_Footprints:Inductor_TYA252012"
 		(layer "B.Cu")
 		(at 150.5126 86.3 90)
@@
 		)
 	)
-	(footprint "My Footprints:APAE1575R1820ABDC1"
+	(footprint "My_Footprints:APAE1575R1820ABDC1"
 		(layer "B.Cu")
 		(at 134.49 54.01 180)
