File: R1/design_files/tracker.kicad_sch (KiCad schematic)
At the start: 8 parts, among them J1 Conn_01x01, J2 Conn_01x01, Q1 DMP2008UFG

Commit message: Refactor code structure for improved readability and maintainability
Parts:
- J1, J2: footprint My Footprints:pad_smd_1.5x3 -> My_Footprints:pad_smd_1.5x3
- Q1: symbol My Libraries:DMP2008UFG -> My_Libraries:DMP2008UFG
Changed lines of the file:
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@@
 	)
 	(symbol
-		(lib_id "My Libraries:DMP2008UFG")
+		(lib_id "My_Libraries:DMP2008UFG")
 		(at 50.8 52.07 90)
 		(unit 1)
@@
 			)
 		)
-		(property "Footprint" "My Footprints:pad_smd_1.5x3"
+		(property "Footprint" "My_Footprints:pad_smd_1.5x3"
 			(at 26.67 52.07 0)
 			(effects
@@
 	)
 	(symbol
-		(lib_id "My Libraries:+VSYS")
+		(lib_id "My_Libraries:+VSYS")
 		(at 142.24 184.15 0)
 		(unit 1)
@@
 	)
 	(symbol
-		(lib_id "My Libraries:+VSYS")
+		(lib_id "My_Libraries:+VSYS")
 		(at 102.87 142.24 0)
 		(unit 1)
@@
 			)
 		)
-		(property "Footprint" "My Footprints:pad_smd_1.5x3"
+		(property "Footprint" "My_Footprints:pad_smd_1.5x3"
 			(at 26.67 55.88 0)
 			(effects
@@
 	)
 	(symbol
-		(lib_id "My Libraries:+VSYS")
+		(lib_id "My_Libraries:+VSYS")
 		(at 143.51 88.9 0)
 		(unit 1)
